Commit message: manual merge of co-design-new-urdf

File: repair_urdf/urdf/repair.urdf.xacro (robot description, xacro)
@@ -3,6 +3,4 @@
 <xacro:include filename="$(find repair_urdf)/urdf/repair_arm.urdf.xacro"/>
 <link name="world"/>
-<link name="base_link">
-</link>
 <joint name="base_joint" type="fixed">
     <origin xyz="0 0 0.5" rpy="0 0 0"/>
@@ -10,19 +8,21 @@
     <child link="base_link"/>
 </joint>
-<link name="r_arm_mount_frame">
+<link name="base_link">
 </link>
-<joint name="r_arm_mount_joint" type="fixed">
-    <origin xyz="0 -0.2 0" rpy="${PI_2} ${PI} 0"/>
+<joint name="base_2rmountjoint" type="fixed">
+    <origin xyz="0 -0.2 0.0" rpy="0 0 0"/>
     <parent link="base_link"/>
     <child link="r_arm_mount_frame"/>
 </joint>
-<xacro:repair_arm base_link="r_arm_mount_frame" id="1"/>
-<link name="l_arm_mount_frame">
-</link>
-<joint name="l_arm_mount_joint" type="fixed">
-    <origin xyz="0 0.2 0" rpy="${-PI_2} 0 0"/>
+<joint name="base_2lmountjoint" type="fixed">
+    <origin xyz="0 0.2 0.0" rpy="0 0 0"/>
     <parent link="base_link"/>
     <child link="l_arm_mount_frame"/>
 </joint>
-<xacro:repair_arm base_link="l_arm_mount_frame" id="2"/>
+<link name="r_arm_mount_frame">
+</link>
+<link name="l_arm_mount_frame">
+</link>
+<xacro:repair_arm base_link="r_arm_mount_frame" id="1" is_sliding_wrist="0"/>
+<xacro:repair_arm base_link="l_arm_mount_frame" id="2" is_sliding_wrist="0"/>
 </robot>

File: repair_urdf/urdf/repair_arm.urdf.xacro (robot description, xacro)
@@ -5,7 +5,16 @@
 <xacro:property name="mid_tau_max" value="200.0" />
 <xacro:property name="sm_tau_max" value="200.0" />
-<xacro:macro name="repair_arm" params="id base_link" >
+<xacro:macro name="repair_arm" params="id base_link is_sliding_wrist" >
+<!-- id: 1 for right arm, everything else is considered left arm -->
+<!-- base_link: name of base link a the single arm -->
+<!-- is_sliding_wrist: whether to add a sliding joint along the axis of wrist's second d.o.f.
+    (true -> yes), everything else -> no -->
 <joint name="arm_${id}_joint_1" type="revolute">
-    <origin xyz="0 0 0" rpy="0 0 0"/>
+    <xacro:if value="${id == 1}">
+        <origin xyz="0 0 0" rpy="${PI_2} 0 0"/>
+    </xacro:if>
+    <xacro:unless value="${id == 1}">
+        <origin xyz="0 0 0" rpy="${-PI_2} 0 0"/>
+    </xacro:unless>
     <parent link="${base_link}"/>
     <child link="arm_${id}_link_1"/>
@@ -13,13 +22,77 @@
     <limit lower="${-150.0 * DEG2RAD}" upper="${150.0 * DEG2RAD}" effort="${big_tau_max}" velocity="10.0"/>
 </joint>
+<link name="arm_${id}_link_1">
+    <inertial>
+        <mass value="0.1"/>
+        <inertia ixx="0.0001" ixy="0" ixz="0" iyy="0.0001" iyz="0" izz="0.0001"/>
+        <origin xyz="0 0 0"/>
+    </inertial>
+    <xacro:if value="${id == 1}">
+        <collision name="arm_${id}_link_1_collision">
+            <geometry>
+                <mesh filename="package://repair_urdf/meshes/link_1.stl" scale="${mmTom} ${mmTom} ${mmTom}"/>
+            </geometry>
+            <material name="dark"/>
+        </collision>
+        <visual name="arm_${id}_link_1_visual">
+            <geometry>
+                <mesh filename="package://repair_urdf/meshes/link_1.stl" scale="${mmTom} ${mmTom} ${mmTom}"/>
+            </geometry>
+            <material name="dark"/>
+        </visual>
+    </xacro:if>
+    <xacro:unless value="${id == 1}">
+        <collision name="arm_${id}_link_1_collision">
+            <geometry>
+                <mesh filename="package://repair_urdf/meshes/link_1_mirror.stl" scale="${mmTom} ${mmTom} ${mmTom}"/>
+            </geometry>
+            <material name="dark"/>
+        </collision>
+        <visual name="arm_${id}_link_1_visual">
+            <geometry>
+                <mesh filename="package://repair_urdf/meshes/link_1_mirror.stl" scale="${mmTom} ${mmTom} ${mmTom}"/>
+            </geometry>
+            <material name="dark"/>
+        </visual>
+    </xacro:unless>
+</link>
 <joint name="arm_${id}_joint_2" type="revolute">
-    <origin xyz="${7.0 * mmTom} 0 0" rpy="0 ${-PI_2} ${PI}"/>
+    <xacro:if value="${id == 1}">
+        <origin xyz="${38.5 * mmTom} ${-23.0 *mmTom} 0" rpy="0 ${-PI_2} ${-PI}"/>
+    </xacro:if>
+    <xacro:unless value="${id == 1}">
+        <origin xyz="${38.5 * mmTom} ${23.0 *mmTom} 0" rpy="0 ${-PI_2} ${-PI}"/>
+    </xacro:unless>
     <parent link="arm_${id}_link_1"/>
     <child link="arm_${id}_link_2"/>
     <axis xyz="0 0 1"/>
-    <limit lower="${-90.0 * DEG2RAD}" upper="${90.0 * DEG2RAD}" effort="${big_tau_max}" velocity="10.0"/>
-</joint>
+    <limit lower="${-80.0 * DEG2RAD}" upper="${125.0 * DEG2RAD}" effort="${big_tau_max}" velocity="10.0"/>
+</joint>
+<link name="arm_${id}_link_2">
+    <inertial>
+        <mass value="0.1"/>
+        <inertia ixx="0.0001" ixy="0" ixz="0" iyy="0.0001" iyz="0" izz="0.0001"/>
+        <origin xyz="0 0 0"/>
+    </inertial>
+    <collision name="arm_${id}_link_2_collision">
+        <geometry>
+            <mesh filename="package://repair_urdf/meshes/link_2.stl" scale="${mmTom} ${mmTom} ${mmTom}"/>
+        </geometry>
+        <material name="dark"/>
+    </collision>
+    <visual name="arm_${id}_link_2_visual">
+        <geometry>
+            <mesh filename="package://repair_urdf/meshes/link_2.stl" scale="${mmTom} ${mmTom} ${mmTom}"/>
+        </geometry>
+        <material name="dark"/>
+    </visual>
+</link>
 <joint name="arm_${id}_joint_3" type="revolute">
-    <origin xyz="0 0 0" rpy="0 ${-PI_2} ${PI}"/>
+    <xacro:if value="${id == 1}">
+        <origin xyz="${5 * mmTom} 0 0" rpy="0 ${PI_2} 0"/>
+    </xacro:if>
+        <origin xyz="${5 * mmTom} 0 0" rpy="0 ${-PI_2} ${-PI}"/>
+    <xacro:if value="${id == 1}">
+    </xacro:if>
     <parent link="arm_${id}_link_2"/>
     <child link="arm_${id}_link_3"/>
@@ -27,13 +100,51 @@
     <limit lower="${-150.0 * DEG2RAD}" upper="${150.0 * DEG2RAD}" effort="${big_tau_max}" velocity="10.0"/>
 </joint>
+<link name="arm_${id}_link_3">
+    <inertial>
+        <mass value="0.1"/>
+        <inertia ixx="0.0001" ixy="0" ixz="0" iyy="0.0001" iyz="0" izz="0.0001"/>
+        <origin xyz="0 0 0"/>
+    </inertial>
+    <collision name="arm_${id}_link_3_collision">
+        <geometry>
+            <mesh filename="package://repair_urdf/meshes/link_3.stl" scale="${mmTom} ${mmTom} ${mmTom}"/>
+        </geometry>
+        <material name="dark"/>
+    </collision>
+    <visual name="arm_${id}_link_3_visual">
+        <geometry>
+            <mesh filename="package://repair_urdf/meshes/link_3.stl" scale="${mmTom} ${mmTom} ${mmTom}"/>
+        </geometry>
+        <material name="dark"/>
+    </visual>
+</link>
 <joint name="arm_${id}_joint_4" type="revolute">
-    <origin xyz="0 ${22.5000 * mmTom} ${360.150 * mmTom}" rpy="0 ${-PI_2} ${PI}"/>
+    <origin xyz="0 ${22.5000 * mmTom} ${360.150 * mmTom}" rpy="0 ${-PI_2} ${-PI}"/>
     <parent link="arm_${id}_link_3"/>
     <child link="arm_${id}_link_4"/>
     <axis xyz="0 0 1"/>
-    <limit lower="${-150.0 * DEG2RAD}" upper="${50.0 * DEG2RAD}" effort="${big_tau_max}" velocity="10.0"/>
-</joint>
+    <limit lower="${-150.0 * DEG2RAD}" upper="${120.0 * DEG2RAD}" effort="${big_tau_max}" velocity="10.0"/>
+</joint>
+<link name="arm_${id}_link_4">
+    <inertial>
+        <mass value="0.1"/>
+        <inertia ixx="0.0001" ixy="0" ixz="0" iyy="0.0001" iyz="0" izz="0.0001"/>
+        <origin xyz="0 0 0"/>
+    </inertial>
+    <collision name="arm_${id}_link_4_collision">
+        <geometry>
+            <mesh filename="package://repair_urdf/meshes/link_4.stl" scale="${mmTom} ${mmTom} ${mmTom}"/>
+        </geometry>
+        <material name="dark"/>
+    </collision>
+    <visual name="arm_${id}_link_4_visual">
+        <geometry>
+            <mesh filename="package://repair_urdf/meshes/link_4.stl" scale="${mmTom} ${mmTom} ${mmTom}"/>
+        </geometry>
+        <material name="dark"/>
+    </visual>
+</link>
 <joint name="arm_${id}_joint_5" type="revolute">
-    <origin xyz="0 0 0" rpy="0 ${-PI_2} ${PI}"/>
+    <origin xyz="${5 * mmTom} 0 0" rpy="${-PI_2} 0 ${-PI_2}"/>
     <parent link="arm_${id}_link_4"/>
     <child link="arm_${id}_link_5"/>
@@ -41,13 +152,76 @@
     <limit lower="${-150.0 * DEG2RAD}" upper="${150.0 * DEG2RAD}" effort="${big_tau_max}" velocity="10.0"/>
 </joint>
-<joint name="arm_${id}_joint_6" type="revolute">
-    <origin xyz="0 0 ${321.000 * mmTom}" rpy="0 ${-PI_2} ${PI}"/>
-    <parent link="arm_${id}_link_5"/>
-    <child link="arm_${id}_link_6"/>
-    <axis xyz="0 0 1"/>
-    <limit lower="${-150.0 * DEG2RAD}" upper="${150.0 * DEG2RAD}" effort="${big_tau_max}" velocity="10.0"/>
-</joint>
+<link name="arm_${id}_link_5">
+    <inertial>
+        <mass value="0.1"/>
+        <inertia ixx="0.0001" ixy="0" ixz="0" iyy="0.0001" iyz="0" izz="0.0001"/>
+        <origin xyz="0 0 0"/>
+    </inertial>
+    <collision name="arm_${id}_link_5_collision">
+        <geometry>
+            <mesh filename="package://repair_urdf/meshes/link_5.stl" scale="${mmTom} ${mmTom} ${mmTom}"/>
+        </geometry>
+        <material name="dark"/>
+    </collision>
+    <visual name="arm_${id}_link_5_visual">
+        <geometry>
+            <mesh filename="package://repair_urdf/meshes/link_5.stl" scale="${mmTom} ${mmTom} ${mmTom}"/>
+        </geometry>
+        <material name="dark"/>
+    </visual>
+</link>
+<xacro:if value="${is_sliding_wrist != True}">
+    <joint name="arm_${id}_joint_6" type="revolute">
+        <origin xyz="0 0 ${321.000 * mmTom}" rpy="0 ${-PI_2} 0"/>
+        <parent link="arm_${id}_link_5"/>
+        <child link="arm_${id}_link_6"/>
+        <axis xyz="0 0 1"/>
+        <limit lower="${-150.0 * DEG2RAD}" upper="${150.0 * DEG2RAD}" effort="${big_tau_max}" velocity="10.0"/>
+    </joint>
+</xacro:if>
+<xacro:unless value="${is_sliding_wrist != True}">
+    <joint name="arm_${id}_joint_6" type="revolute">
+        <origin xyz="0 0 ${321.000 * mmTom}" rpy="0 ${-PI_2} 0"/>
+        <parent link="arm_${id}_link_5"/>
+        <child link="dummy_sliding_wrist${id}_link"/>
+        <axis xyz="0 0 1"/>
+        <limit lower="${-150.0 * DEG2RAD}" upper="${150.0 * DEG2RAD}" effort="${big_tau_max}" velocity="10.0"/>
+    </joint>
+    <link name="dummy_sliding_wrist${id}_link">
+    </link>
+    <joint name="dummy_sliding_wrist${id}_joint" type="prismatic">
+        <origin xyz="0.0 0.0 0.0" rpy="0 0 0"/>
+        <parent link="dummy_sliding_wrist${id}_link"/>
+        <child link="arm_${id}_link_6"/>
+        <axis xyz="0 0 -1"/>
+        <limit lower="${sliding_wrist_deltaz_lb}" upper= "${sliding_wrist_deltaz_ub}" effort="1000.0" velocity="20.0"/>
+    </joint>
+</xacro:unless>
+<link name="arm_${id}_link_6">
+    <inertial>
+        <mass value="0.1"/>
+        <inertia ixx="0.0001" ixy="0" ixz="0" iyy="0.0001" iyz="0" izz="0.0001"/>
+        <origin xyz="0 0 0"/>
+    </inertial>
+    <collision name="arm_${id}_link_6_collision">
+        <geometry>
+            <mesh filename="package://repair_urdf/meshes/link_6.stl" scale="${mmTom} ${mmTom} ${mmTom}"/>
+        </geometry>
+        <material name="dark"/>
+    </collision>
+    <visual name="arm_${id}_link_6_visual">
+        <geometry>
+            <mesh filename="package://repair_urdf/meshes/link_6.stl" scale="${mmTom} ${mmTom} ${mmTom}"/>
+        </geometry>
+        <material name="dark"/>
+    </visual>
+</link>
 <joint name="arm_${id}_joint_7" type="revolute">
-    <origin xyz="${180.000 * mmTom} 0 0" rpy="0 ${-PI_2} ${PI}"/>
+    <xacro:if value="${id == 1}">
+        <origin xyz="${180.000 * mmTom} 0 0" rpy="${PI_2} 0 ${PI_2}"/>
+    </xacro:if>
+    <xacro:unless value="${id == 1}">
+        <origin xyz="${180.000 * mmTom} 0 0" rpy="${-PI_2} 0 ${-PI_2}"/>
+    </xacro:unless>
     <parent link="arm_${id}_link_6"/>
     <child link="arm_${id}_link_7"/>
@@ -55,4 +229,23 @@
     <limit lower="${-150.0 * DEG2RAD}" upper="${150.0 * DEG2RAD}" effort="${big_tau_max}" velocity="10.0"/>
 </joint>
+<link name="arm_${id}_link_7">
+    <inertial>
+        <mass value="0.1"/>
+        <inertia ixx="0.0001" ixy="0" ixz="0" iyy="0.0001" iyz="0" izz="0.0001"/>
+        <origin xyz="0 0 0"/>
+    </inertial>
+    <collision name="arm_${id}_link_7_collision">
+        <geometry>
+            <mesh filename="package://repair_urdf/meshes/link_7.stl" scale="${mmTom} ${mmTom} ${mmTom}"/>
+        </geometry>
+        <material name="dark"/>
+    </collision>
+    <visual name="arm_${id}_link_7_visual">
+        <geometry>
+            <mesh filename="package://repair_urdf/meshes/link_7.stl" scale="${mmTom} ${mmTom} ${mmTom}"/>
+        </geometry>
+        <material name="dark"/>
+    </visual>
+</link>
 <joint name="arm_${id}_tcp_joint" type="fixed">
     <origin xyz="0 0 0" rpy="0 0 0"/>
@@ -60,137 +253,4 @@
     <child link="arm_${id}_tcp"/>
 </joint>
-<link name="arm_${id}_link_1">
-    <inertial>
-        <mass value="0.1"/>
-        <inertia ixx="0.0001" ixy="0" ixz="0" iyy="0.0001" iyz="0" izz="0.0001"/>
-        <origin xyz="0 0 0"/>
-    </inertial>
-    <collision name="arm_${id}_link_1_collision">
-        <geometry>
-            <mesh filename="package://repair_urdf/meshes/link_1.stl" scale="${mmTom} ${mmTom} ${mmTom}"/>
-        </geometry>
-        <material name="dark"/>
-    </collision>
-    <visual name="arm_${id}_link_1_visual">
-        <geometry>
-            <mesh filename="package://repair_urdf/meshes/link_1.stl" scale="${mmTom} ${mmTom} ${mmTom}"/>
-        </geometry>
-        <material name="dark"/>
-    </visual>
-</link>
-<link name="arm_${id}_link_2">
-    <inertial>
-        <mass value="0.1"/>
-        <inertia ixx="0.0001" ixy="0" ixz="0" iyy="0.0001" iyz="0" izz="0.0001"/>
-        <origin xyz="0 0 0"/>
-    </inertial>
-    <collision name="arm_${id}_link_2_collision">
-        <geometry>
-            <mesh filename="package://repair_urdf/meshes/link_2.stl" scale="${mmTom} ${mmTom} ${mmTom}"/>
-        </geometry>
-        <material name="dark"/>
-    </collision>
-    <visual name="arm_${id}_link_2_visual">
-        <geometry>
-            <mesh filename="package://repair_urdf/meshes/link_2.stl" scale="${mmTom} ${mmTom} ${mmTom}"/>
-        </geometry>
-        <material name="dark"/>
-    </visual>
-</link>
-<link name="arm_${id}_link_3">
-    <inertial>
-        <mass value="0.1"/>
-        <inertia ixx="0.0001" ixy="0" ixz="0" iyy="0.0001" iyz="0" izz="0.0001"/>
-        <origin xyz="0 0 0"/>
-    </inertial>
-    <collision name="arm_${id}_link_3_collision">
-        <geometry>
-            <mesh filename="package://repair_urdf/meshes/link_3.stl" scale="${mmTom} ${mmTom} ${mmTom}"/>
-        </geometry>
-        <material name="dark"/>
-    </collision>
-    <visual name="arm_${id}_link_3_visual">
-        <geometry>
-            <mesh filename="package://repair_urdf/meshes/link_3.stl" scale="${mmTom} ${mmTom} ${mmTom}"/>
-        </geometry>
-        <material name="dark"/>
-    </visual>
-</link>
-<link name="arm_${id}_link_4">
-    <inertial>
-        <mass value="0.1"/>
-        <inertia ixx="0.0001" ixy="0" ixz="0" iyy="0.0001" iyz="0" izz="0.0001"/>
-        <origin xyz="0 0 0"/>
-    </inertial>
-    <collision name="arm_${id}_link_4_collision">
-        <geometry>
-            <mesh filename="package://repair_urdf/meshes/link_4.stl" scale="${mmTom} ${mmTom} ${mmTom}"/>
-        </geometry>
-        <material name="dark"/>
-    </collision>
-    <visual name="arm_${id}_link_4_visual">
-        <geometry>
-            <mesh filename="package://repair_urdf/meshes/link_4.stl" scale="${mmTom} ${mmTom} ${mmTom}"/>
-        </geometry>
-        <material name="dark"/>
-    </visual>
-</link>
-<link name="arm_${id}_link_5">
-    <inertial>
-        <mass value="0.1"/>
-        <inertia ixx="0.0001" ixy="0" ixz="0" iyy="0.0001" iyz="0" izz="0.0001"/>
-        <origin xyz="0 0 0"/>
-    </inertial>
-    <collision name="arm_${id}_link_5_collision">
-        <geometry>
-            <mesh filename="package://repair_urdf/meshes/link_5.stl" scale="${mmTom} ${mmTom} ${mmTom}"/>
-        </geometry>
-        <material name="dark"/>
-    </collision>
-    <visual name="arm_${id}_link_5_visual">
-        <geometry>
-            <mesh filename="package://repair_urdf/meshes/link_5.stl" scale="${mmTom} ${mmTom} ${mmTom}"/>
-        </geometry>
-        <material name="dark"/>
-    </visual>
-</link>
-<link name="arm_${id}_link_6">
-    <inertial>
-        <mass value="0.1"/>
-        <inertia ixx="0.0001" ixy="0" ixz="0" iyy="0.0001" iyz="0" izz="0.0001"/>
-        <origin xyz="0 0 0"/>
-    </inertial>
-    <collision name="arm_${id}_link_6_collision">
-        <geometry>
-            <mesh filename="package://repair_urdf/meshes/link_6.stl" scale="${mmTom} ${mmTom} ${mmTom}"/>
-        </geometry>
-        <material name="dark"/>
-    </collision>
-    <visual name="arm_${id}_link_6_visual">
-        <geometry>
-            <mesh filename="package://repair_urdf/meshes/link_6.stl" scale="${mmTom} ${mmTom} ${mmTom}"/>
-        </geometry>
-        <material name="dark"/>
-    </visual>
-</link>
-<link name="arm_${id}_link_7">
-    <inertial>
-        <mass value="0.1"/>
-        <inertia ixx="0.0001" ixy="0" ixz="0" iyy="0.0001" iyz="0" izz="0.0001"/>
-        <origin xyz="0 0 0"/>
-    </inertial>
-    <collision name="arm_${id}_link_7_collision">
-        <geometry>
-            <mesh filename="package://repair_urdf/meshes/link_7.stl" scale="${mmTom} ${mmTom} ${mmTom}"/>
-        </geometry>
-        <material name="dark"/>
-    </collision>
-    <visual name="arm_${id}_link_7_visual">
-        <geometry>
-            <mesh filename="package://repair_urdf/meshes/link_7.stl" scale="${mmTom} ${mmTom} ${mmTom}"/>
-        </geometry>
-        <material name="dark"/>
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
File: repair_urdf/urdf/repair_full.urdf.xacro (robot description, xacro)
@@ -3,4 +3,5 @@
 <xacro:include filename="$(find repair_urdf)/urdf/repair_arm.urdf.xacro"/>
 <xacro:include filename="$(find repair_urdf)/urdf/repair_cage.urdf.xacro"/>
+<xacro:arg name="is_sliding_wrist" default="false" />
 <joint name="x_joint" type="prismatic">
     <origin xyz="0.0 0.0 0.0" rpy="0.0 0.0 0.0"/>
@@ -23,11 +24,20 @@
 </link>
 <joint name="r_arm_mount_joint" type="prismatic">
-    <origin xyz="0.0 0.0 0.0" rpy="${-PI_2} 0 ${PI}"/>
+    <origin xyz="0.0 0.0 0.0" rpy="0 0 0"/>
     <parent link="base_link"/>
     <child link="dummy_r"/>
-    <axis xyz="0 0 1"/>
+    <axis xyz="0 -1 0"/>
+    <limit lower="${shoulder_width_lb}" upper= "${shoulder_width_ub}" effort="1000.0" velocity="20.0"/>
+</joint>
+<joint name="l_arm_mount_joint" type="prismatic">
+    <origin xyz="0.0 0.0 0.0" rpy="0 0 0"/>
+    <parent link="base_link"/>
+    <child link="dummy_l"/>
+    <axis xyz="0 1 0"/>
     <limit lower="${shoulder_width_lb}" upper= "${shoulder_width_ub}" effort="1000.0" velocity="20.0"/>
 </joint>
 <link name="dummy_r">
+</link>
+<link name="dummy_l">
 </link>
 <joint name="roll_r" type="revolute">
@@ -35,19 +45,7 @@
     <parent link="dummy_r"/>
     <child link="r_arm_mount_frame"/>
-    <axis xyz="-1 0 0"/>
+    <axis xyz="1 0 0"/>
     <limit lower="${shoulder_roll_lb}" upper="${shoulder_roll_ub}" effort="0.0" velocity="0.0"/>
 </joint>
-<link name="r_arm_mount_frame">
-</link>
-<xacro:repair_arm base_link="r_arm_mount_frame" id="1"/>
-<joint name="l_arm_mount_joint" type="prismatic">
-    <origin xyz="0.0 0.0 0.0" rpy="${-PI_2} 0 0"/>
-    <parent link="base_link"/>
-    <child link="dummy_l"/>
-    <axis xyz="0 0 1"/>
-    <limit lower="${shoulder_width_lb}" upper= "${shoulder_width_ub}" effort="1000.0" velocity="20.0"/>
-</joint>
-<link name="dummy_l">
-</link>
 <joint name="roll_l" type="revolute">
     <origin xyz="0.0 0.0 0.0" rpy="0.0 0.0 0.0"/>
@@ -57,6 +55,9 @@
     <limit lower="${shoulder_roll_lb}" upper="${shoulder_roll_ub}" effort="0.0" velocity="0.0"/>
 </joint>
+<link name="r_arm_mount_frame">
+</link>
 <link name="l_arm_mount_frame">
 </link>
-<xacro:repair_arm base_link="l_arm_mount_frame" id="2"/>
+<xacro:repair_arm base_link="r_arm_mount_frame" id="1" is_sliding_wrist="$(arg is_sliding_wrist)"/>
+<xacro:repair_arm base_link="l_arm_mount_frame" id="2" is_sliding_wrist="$(arg is_sliding_wrist)"/>
 </robot>

File: repair_urdf/urdf/utils.urdf.xacro (robot description, xacro)
@@ -15,4 +15,6 @@
 <xacro:property name="shoulder_roll_lb" value="-${PI}" />
 <xacro:property name="shoulder_roll_ub" value="${PI}" />
+<xacro:property name="sliding_wrist_deltaz_lb" value="0" />
+<xacro:property name="sliding_wrist_deltaz_ub" value="0.05" />
 <!-- color -->
 <material name="darkblue">
