Commit message: positiion tracking ok

File: repair_urdf/urdf/repair_full.urdf.xacro (robot description, xacro)
@@ -17,5 +17,5 @@
     <child link="base_link"/>
     <axis xyz="0 0 1"/>
-    <limit lower="${z_joint_limit_margin}" upper= "${cage_height - z_joint_limit_margin}" effort="1000.0" velocity="20.0"/>
+    <limit lower="${z_joint_lb}" upper= "${cage_height - z_joint_limit_margin}" effort="1000.0" velocity="20.0"/>
 </joint>
 <!-- RePAIR assembly (two arms) -->

File: repair_urdf/urdf/utils.urdf.xacro (robot description, xacro)
@@ -10,4 +10,5 @@
 <xacro:property name="x_joint_limit_margin" value="0.1" />
 <xacro:property name="z_joint_limit_margin" value="0.1" />
+<xacro:property name="z_joint_lb" value="0.5" />
 <xacro:property name="shoulder_width_lb" value="0.25" />
 <xacro:property name="shoulder_width_ub" value="0.6" />

Commit message: updated urdf parameters and simple postprocessing

File: repair_urdf/urdf/repair_full.urdf.xacro (robot description, xacro)
@@ -18,5 +18,5 @@
     <child link="base_link"/>
     <axis xyz="0 0 1"/>
-    <limit lower="${z_joint_lb}" upper= "${cage_height - z_joint_limit_margin}" effort="1000.0" velocity="20.0"/>
+    <limit lower="${z_joint_lb}" upper= "2" effort="1000.0" velocity="20.0"/>
 </joint>
 <!-- RePAIR assembly (two arms) -->

File: repair_urdf/urdf/utils.urdf.xacro (robot description, xacro)
@@ -7,12 +7,13 @@
 <xacro:property name="PI" value="3.14159265359" />
 <xacro:property name="PI_2" value="1.57079632679" />
+<xacro:property name="PI_4" value="0.7853981633974483" />
 <xacro:property name="DEG2RAD" value="${PI/180.0}" />
 <xacro:property name="x_joint_limit_margin" value="0.1" />
 <xacro:property name="z_joint_limit_margin" value="0.1" />
 <xacro:property name="z_joint_lb" value="0.5" />
-<xacro:property name="shoulder_width_lb" value="0.2" /> <!-- wrt shoulder center -->
+<xacro:property name="shoulder_width_lb" value="0.25" /> <!-- wrt shoulder center -->
 <xacro:property name="shoulder_width_ub" value="0.5" />
-<xacro:property name="shoulder_roll_lb" value="-${PI_2}" />
-<xacro:property name="shoulder_roll_ub" value="${PI_2}" />
+<xacro:property name="shoulder_roll_lb" value="-${PI_2 + PI_4}" />
+<xacro:property name="shoulder_roll_ub" value="${PI_2 + PI_4}" />
 <xacro:property name="sliding_wrist_deltaz_lb" value="0" />
 <xacro:property name="sliding_wrist_deltaz_ub" value="0.05" />
