Commit message: added collision yaml parser

File: repair_urdf/urdf/repair_arm_coll.urdf.xacro (robot description, xacro)
@@ -10,5 +10,5 @@
             <origin xyz="0 0 0" rpy="0 0 0"/>
             <geometry>
-                <sphere radius="${coll_radii_link1}"/>
+                <sphere radius="${coll_radius_link1}"/>
             </geometry>
             <material name="darkred"/>
@@ -24,5 +24,5 @@
             <origin xyz="0 0 0" rpy="0 0 0"/>
             <geometry>
-                <sphere radius="${coll_radii_link2}"/>
+                <sphere radius="${coll_radius_link2}"/>
             </geometry>
             <material name="darkred"/>
@@ -38,5 +38,5 @@
             <origin xyz="0 0 0" rpy="0 0 0"/>
             <geometry>
-                <sphere radius="${coll_radii_link3}"/>
+                <sphere radius="${coll_radius_link3}"/>
             </geometry>
             <material name="darkred"/>
@@ -52,5 +52,5 @@
             <origin xyz="0 0 0" rpy="0 0 0"/>
             <geometry>
-                <sphere radius="${coll_radii_link4}"/>
+                <sphere radius="${coll_radius_link4}"/>
             </geometry>
             <material name="darkred"/>
@@ -65,5 +65,5 @@
     <visual name="arm_${id}_link5_coll_visual">
             <geometry>
-                <sphere radius="${coll_radii_link5}"/>
+                <sphere radius="${coll_radius_link5}"/>
             </geometry>
             <material name="darkred"/>
@@ -78,5 +78,5 @@
     <visual name="arm_${id}_link6_coll_visual">
             <geometry>
-                <sphere radius="${coll_radii_link6}"/>
+                <sphere radius="${coll_radius_link6}"/>
             </geometry>
             <material name="darkred"/>
@@ -91,5 +91,5 @@
         <visual name="arm_${id}_link7_coll_visual">
                 <geometry>
-                    <sphere radius="${coll_radii_link7}"/>
+                    <sphere radius="${coll_radius_link7}"/>
                 </geometry>
                 <material name="darkred"/>

File: repair_urdf/urdf/repair_arm_coll_params.urdf.xacro (robot description, xacro)
@@ -4,11 +4,11 @@
 <xacro:property name="yaml_file" value="$(find repair_urdf)/config/arm_coll.yaml" />
 <xacro:property name="coll_props" value="${xacro.load_yaml(yaml_file)}"/>
-<xacro:property name="coll_radii_link1" value="${coll_props['link1_coll']['coll_radii']}" />
-<xacro:property name="coll_radii_link2" value="${coll_props['link2_coll']['coll_radii']}" />
-<xacro:property name="coll_radii_link3" value="${coll_props['link3_coll']['coll_radii']}" />
-<xacro:property name="coll_radii_link4" value="${coll_props['link4_coll']['coll_radii']}" />
-<xacro:property name="coll_radii_link5" value="${coll_props['link5_coll']['coll_radii']}" />
-<xacro:property name="coll_radii_link6" value="${coll_props['link6_coll']['coll_radii']}" />
-<xacro:property name="coll_radii_link7" value="${coll_props['link7_coll']['coll_radii']}" />
+<xacro:property name="coll_radius_link1" value="${coll_props['link1_coll']['coll_radius']}" />
+<xacro:property name="coll_radius_link2" value="${coll_props['link2_coll']['coll_radius']}" />
+<xacro:property name="coll_radius_link3" value="${coll_props['link3_coll']['coll_radius']}" />
+<xacro:property name="coll_radius_link4" value="${coll_props['link4_coll']['coll_radius']}" />
+<xacro:property name="coll_radius_link5" value="${coll_props['link5_coll']['coll_radius']}" />
+<xacro:property name="coll_radius_link6" value="${coll_props['link6_coll']['coll_radius']}" />
+<xacro:property name="coll_radius_link7" value="${coll_props['link7_coll']['coll_radius']}" />
 <xacro:property name="link1_coll_offset_x" value="0.0" />
 <xacro:property name="link1_coll_offset_y" value="0.0" />

Commit message: added dofs for link5 coll adaptation

File: repair_urdf/urdf/repair_arm_coll.urdf.xacro (robot description, xacro)
@@ -57,8 +57,10 @@
     </visual>
 </link>
-<joint name="arm_${id}_link_5_coll_joint" type="fixed">
+<joint name="arm_${id}_link_5_coll_joint" type="prismatic">
     <origin xyz="${link5_coll_offset_x} ${link5_coll_offset_y} ${link5_coll_offset_z}" rpy="0 0 0"/>
     <parent link="arm_${id}_link_5"/>
     <child link="arm_${id}_link5_coll"/>
+    <limit lower="${0}" upper="${sliding_wrist_deltaz_ub}" effort="${big_tau_max}" velocity="10.0"/>
+    <axis xyz="1 0 0"/>
 </joint>
 <link name="arm_${id}_link5_coll">

File: repair_urdf/urdf/repair_arm_coll_params.urdf.xacro (robot description, xacro)
@@ -23,7 +23,7 @@
 <xacro:property name="link4_coll_offset_y" value="0.0" />
 <xacro:property name="link4_coll_offset_z" value="0.0" />
-<xacro:property name="link5_coll_offset_x" value="-0.075" />
+<xacro:property name="link5_coll_offset_x" value="-0.1" />
 <xacro:property name="link5_coll_offset_y" value="0.0" />
-<xacro:property name="link5_coll_offset_z" value="0.3" />
+<xacro:property name="link5_coll_offset_z" value="0.321" />
 <xacro:property name="link6_coll_offset_x" value="0.0" />
 <xacro:property name="link6_coll_offset_y" value="0.0" />

File: repair_urdf/urdf/utils.urdf.xacro (robot description, xacro)
@@ -7,4 +7,5 @@
 <xacro:property name="PI" value="3.14159265359" />
 <xacro:property name="PI_2" value="1.57079632679" />
+<xacro:property name="PI_3" value="1.047197551196598" />
 <xacro:property name="PI_4" value="0.7853981633974483" />
 <xacro:property name="DEG2RAD" value="${PI/180.0}" />
@@ -14,5 +15,5 @@
 <xacro:property name="shoulder_width_lb" value="0.21" /> <!-- wrt shoulder center -->
 <xacro:property name="shoulder_width_ub" value="0.5" />
-<xacro:property name="shoulder_roll_lb" value="-${PI_2}" />
+<xacro:property name="shoulder_roll_lb" value="-${PI_3}" />
 <xacro:property name="shoulder_roll_ub" value="${PI_2}" />
 <xacro:property name="sliding_wrist_deltaz_lb" value="0" />
