Commit message: full URDF with additional dofs

File: repair_urdf/urdf/utils.urdf.xacro (robot description, xacro)
@@ -8,4 +8,10 @@
 <xacro:property name="PI_2" value="1.57079632679" />
 <xacro:property name="DEG2RAD" value="${PI/180.0}" />
+<xacro:property name="x_joint_limit_margin" value="0.1" />
+<xacro:property name="z_joint_limit_margin" value="0.1" />
+<xacro:property name="shoulder_width_lb" value="0.25" />
+<xacro:property name="shoulder_width_ub" value="0.6" />
+<xacro:property name="shoulder_roll_lb" value="-${PI/4}" />
+<xacro:property name="shoulder_roll_ub" value="${PI/4}" />
 <!-- color -->
 <material name="darkblue">

Commit message: huge improvements

File: repair_urdf/urdf/utils.urdf.xacro (robot description, xacro)
@@ -12,7 +12,7 @@
 <xacro:property name="z_joint_lb" value="0.5" />
 <xacro:property name="shoulder_width_lb" value="0.25" />
-<xacro:property name="shoulder_width_ub" value="0.6" />
-<xacro:property name="shoulder_roll_lb" value="-${PI/4}" />
-<xacro:property name="shoulder_roll_ub" value="${PI/4}" />
+<xacro:property name="shoulder_width_ub" value="0.8" />
+<xacro:property name="shoulder_roll_lb" value="-${PI}" />
+<xacro:property name="shoulder_roll_ub" value="${PI}" />
 <!-- color -->
 <material name="darkblue">

Commit message: small changes

File: repair_urdf/urdf/utils.urdf.xacro (robot description, xacro)
@@ -12,5 +12,5 @@
 <xacro:property name="z_joint_lb" value="0.5" />
 <xacro:property name="shoulder_width_lb" value="0.25" />
-<xacro:property name="shoulder_width_ub" value="0.8" />
+<xacro:property name="shoulder_width_ub" value="0.5" />
 <xacro:property name="shoulder_roll_lb" value="-${PI}" />
 <xacro:property name="shoulder_roll_ub" value="${PI}" />

Commit message: changed shoulder lower bound and task relaxation

File: repair_urdf/urdf/utils.urdf.xacro (robot description, xacro)
@@ -11,5 +11,5 @@
 <xacro:property name="z_joint_limit_margin" value="0.1" />
 <xacro:property name="z_joint_lb" value="0.5" />
-<xacro:property name="shoulder_width_lb" value="0.25" />
+<xacro:property name="shoulder_width_lb" value="0.2" /> <!-- wrt shoulder center -->
 <xacro:property name="shoulder_width_ub" value="0.5" />
 <xacro:property name="shoulder_roll_lb" value="-${PI}" />

Commit message: restricted shoulder roll mounting angle

File: repair_urdf/urdf/utils.urdf.xacro (robot description, xacro)
@@ -13,6 +13,6 @@
 <xacro:property name="shoulder_width_lb" value="0.2" /> <!-- wrt shoulder center -->
 <xacro:property name="shoulder_width_ub" value="0.5" />
-<xacro:property name="shoulder_roll_lb" value="-${PI}" />
-<xacro:property name="shoulder_roll_ub" value="${PI}" />
+<xacro:property name="shoulder_roll_lb" value="-${PI_2}" />
+<xacro:property name="shoulder_roll_ub" value="${PI_2}" />
 <xacro:property name="sliding_wrist_deltaz_lb" value="0" />
 <xacro:property name="sliding_wrist_deltaz_ub" value="0.05" />

Commit message: task generator class name change

File: repair_urdf/urdf/utils.urdf.xacro (robot description, xacro)
@@ -19,5 +19,5 @@
 <xacro:property name="sliding_wrist_deltaz_ub" value="0.05" />
 <xacro:property name="softhand_mount_angle" value="${PI_4}" />
-<xacro:property name="object_size" value="0.08" />
+<xacro:property name="object_size" value="0.01" />
 <!-- color -->
 <material name="darkblue">

Commit message: fixed missing squared collision radii in collision handler

File: repair_urdf/urdf/utils.urdf.xacro (robot description, xacro)
@@ -11,5 +11,5 @@
 <xacro:property name="x_joint_limit_margin" value="0.1" />
 <xacro:property name="z_joint_limit_margin" value="0.1" />
-<xacro:property name="z_joint_lb" value="0.0" />
+<xacro:property name="z_joint_lb" value="0.5" />
 <xacro:property name="shoulder_width_lb" value="0.25" /> <!-- wrt shoulder center -->
 <xacro:property name="shoulder_width_ub" value="0.5" />

Commit message: qwertgyhj

File: repair_urdf/urdf/utils.urdf.xacro (robot description, xacro)
@@ -14,6 +14,6 @@
 <xacro:property name="shoulder_width_lb" value="0.25" /> <!-- wrt shoulder center -->
 <xacro:property name="shoulder_width_ub" value="0.5" />
-<xacro:property name="shoulder_roll_lb" value="-${PI_2 + PI_4}" />
-<xacro:property name="shoulder_roll_ub" value="${PI_2 + PI_4}" />
+<xacro:property name="shoulder_roll_lb" value="-${PI_2}" />
+<xacro:property name="shoulder_roll_ub" value="${PI_2}" />
 <xacro:property name="sliding_wrist_deltaz_lb" value="0" />
 <xacro:property name="sliding_wrist_deltaz_ub" value="0.05" />

Commit message: modified some parameters

File: repair_urdf/urdf/utils.urdf.xacro (robot description, xacro)
@@ -11,5 +11,5 @@
 <xacro:property name="x_joint_limit_margin" value="0.1" />
 <xacro:property name="z_joint_limit_margin" value="0.1" />
-<xacro:property name="z_joint_lb" value="0.5" />
+<xacro:property name="z_joint_lb" value="0.3" />
 <xacro:property name="shoulder_width_lb" value="0.25" /> <!-- wrt shoulder center -->
 <xacro:property name="shoulder_width_ub" value="0.5" />
@@ -17,5 +17,5 @@
 <xacro:property name="shoulder_roll_ub" value="${PI_2}" />
 <xacro:property name="sliding_wrist_deltaz_lb" value="0" />
-<xacro:property name="sliding_wrist_deltaz_ub" value="0.05" />
+<xacro:property name="sliding_wrist_deltaz_ub" value="0.1" />
 <xacro:property name="softhand_mount_angle" value="${PI_4}" />
 <xacro:property name="object_size" value="0.02" />

Commit message: update

File: repair_urdf/urdf/utils.urdf.xacro (robot description, xacro)
@@ -12,5 +12,5 @@
 <xacro:property name="z_joint_limit_margin" value="0.1" />
 <xacro:property name="z_joint_lb" value="0.3" />
-<xacro:property name="shoulder_width_lb" value="0.25" /> <!-- wrt shoulder center -->
+<xacro:property name="shoulder_width_lb" value="0.21" /> <!-- wrt shoulder center -->
 <xacro:property name="shoulder_width_ub" value="0.5" />
 <xacro:property name="shoulder_roll_lb" value="-${PI_2}" />

Commit message: relaxed upper bound on wrist offset to see what comes out

File: repair_urdf/urdf/utils.urdf.xacro (robot description, xacro)
@@ -23,5 +23,6 @@
 <xacro:property name="shoulder_roll_ub" value="${PI_2}" />
 <xacro:property name="sliding_wrist_deltaz_lb" value="0" />
-<xacro:property name="sliding_wrist_deltaz_ub" value="0.1" />
+<xacro:property name="sliding_wrist_deltaz_ub" value="0.5" />
+<!-- <xacro:property name="sliding_wrist_deltaz_ub" value="0.1" /> -->
 <xacro:property name="softhand_mount_angle" value="${PI_4}" />
 <xacro:property name="object_size" value="0.02" />

Commit message: restored wrist offset angle

File: repair_urdf/urdf/utils.urdf.xacro (robot description, xacro)
@@ -23,6 +23,5 @@
 <xacro:property name="shoulder_roll_ub" value="${PI_2}" />
 <xacro:property name="sliding_wrist_deltaz_lb" value="0" />
-<xacro:property name="sliding_wrist_deltaz_ub" value="0.5" />
-<!-- <xacro:property name="sliding_wrist_deltaz_ub" value="0.1" /> -->
+<xacro:property name="sliding_wrist_deltaz_ub" value="0.1" />
 <xacro:property name="softhand_mount_angle" value="${PI_4}" />
 <xacro:property name="object_size" value="0.02" />

Commit message: added wrist attractor cost term

File: repair_urdf/urdf/utils.urdf.xacro (robot description, xacro)
@@ -23,5 +23,5 @@
 <xacro:property name="shoulder_roll_ub" value="${PI_2}" />
 <xacro:property name="sliding_wrist_deltaz_lb" value="0" />
-<xacro:property name="sliding_wrist_deltaz_ub" value="0.1" />
+<xacro:property name="sliding_wrist_deltaz_ub" value="0.01" />
 <xacro:property name="softhand_mount_angle" value="${PI_4}" />
 <xacro:property name="object_size" value="0.02" />
