Commit message: added dummy inertias to allow gazebo parsing

File: repair_urdf/urdf/repair_cage.urdf.xacro (robot description, xacro)
@@ -309,12 +309,5 @@
   </joint>
   <link name="working_surface_link">
-    <!-- dummy intertia to make Gazebo urdf2sdf converter work -->
-    <inertial>
-      <mass value="1.0" />
-      <origin xyz="0 0 0" />
-      <inertia ixx="0.1" ixy="0"  ixz="0"
-               iyy="0.1" iyz="0"
-               izz="0.01" />
-    </inertial>
+    <xacro:fake_inertial/>
   </link>
 </robot>

File: repair_urdf/urdf/repair_full.urdf.xacro (robot description, xacro)
@@ -8,21 +8,15 @@
 <xacro:arg name="show_coll" default="false" />
 <xacro:arg name="load_sol" default="false" />
-<joint name="x_joint" type="prismatic">
-    <origin xyz="0.0 0.0 0.0" rpy="0.0 0.0 0.0"/>
-    <parent link="working_surface_link"/>
-    <child link="dummy_link"/>
-    <axis xyz="1 0 0"/>
-    <limit lower="${- cage_depth/2 + x_joint_limit_margin}" upper= "${cage_depth/2 - x_joint_limit_margin}" effort="1000.0" velocity="20.0"/>
-</joint>
-<link name="dummy_link">
-    <inertial>
-      <mass value="1.0" />
-      <origin xyz="0 0 0" />
-      <inertia ixx="0.1" ixy="0"  ixz="0"
-               iyy="0.1" iyz="0"
-               izz="0.01" />
-    </inertial>
-</link>
 <xacro:if value="$(arg load_sol)">
+    <joint name="x_joint" type="prismatic">
+        <origin xyz="0.0 0.0 0.0" rpy="0.0 0.0 0.0"/>
+        <parent link="working_surface_link"/>
+        <child link="dummy_link"/>
+        <axis xyz="1 0 0"/>
+        <limit lower="${- cage_depth/2 + x_joint_limit_margin}" upper= "${cage_depth/2 - x_joint_limit_margin}" effort="1000.0" velocity="20.0"/>
+    </joint>
+    <link name="dummy_link">
+    </link>
+    <!-- RePAIR assembly (two arms) -->
     <joint name="z_joint" type="fixed">
         <origin xyz="0.0 0.0 ${mount_h}" rpy="0.0 0.0 0.0"/>
@@ -30,18 +24,6 @@
         <child link="base_link"/>
     </joint>
-</xacro:if>
-<xacro:unless value="$(arg load_sol)">
-    <joint name="z_joint" type="prismatic">
-        <origin xyz="0.0 0.0 0.0" rpy="0.0 0.0 0.0"/>
-        <parent link="dummy_link"/>
-        <child link="base_link"/>
-        <axis xyz="0 0 1"/>
-        <limit lower="${z_joint_lb}" upper= "2" effort="1000.0" velocity="20.0"/>
-    </joint>
-</xacro:unless>
-<!-- RePAIR assembly (two arms) -->
-<link name="base_link">
-</link>
-<xacro:if value="$(arg load_sol)">
+    <link name="base_link">
+    </link>
     <joint name="r_arm_mount_joint" type="fixed">
         <origin xyz="0.0 ${-should_w} 0.0" rpy="0 0 0"/>
@@ -54,6 +36,49 @@
         <child link="dummy_l"/>
     </joint>
+    <link name="dummy_r">
+    </link>
+    <link name="dummy_l">
+    </link>
+    <joint name="roll_r" type="fixed">
+        <origin xyz="0 0.0 0.0" rpy="${roll_mount} 0.0 0.0"/>
+        <parent link="dummy_r"/>
+        <child link="r_arm_mount_frame"/>
+    </joint>
+    <joint name="roll_l" type="fixed">
+        <origin xyz="0 0.0 0.0" rpy="${-roll_mount} 0.0 0.0"/>
+        <parent link="dummy_l"/>
+        <child link="l_arm_mount_frame"/>
+    </joint>
+    <link name="r_arm_mount_frame">
+        <xacro:fake_inertial/>
+    </link>
+    <link name="l_arm_mount_frame">
+        <xacro:fake_inertial/>
+    </link>
 </xacro:if>
 <xacro:unless value="$(arg load_sol)">
+    <joint name="x_joint" type="prismatic">
+        <origin xyz="0.0 0.0 0.0" rpy="0.0 0.0 0.0"/>
+        <parent link="working_surface_link"/>
+        <child link="dummy_link"/>
+        <axis xyz="1 0 0"/>
+        <limit lower="${- cage_depth/2 + x_joint_limit_margin}" upper= "${cage_depth/2 - x_joint_limit_margin}" effort="1000.0" velocity="20.0"/>
+    </joint>
+    <link name="dummy_link">
+    </link>
+    <joint name="z_joint" type="prismatic">
+        <origin xyz="0.0 0.0 0.0" rpy="0.0 0.0 0.0"/>
+        <parent link="dummy_link"/>
+        <child link="base_link"/>
+        <axis xyz="0 0 1"/>
+        <limit lower="${z_joint_lb}" upper= "2" effort="1000.0" velocity="20.0"/>
+    </joint>
+    <!-- RePAIR assembly (two arms) -->
+    <link name="base_link">
+    </link>
+    <link name="dummy_r">
+    </link>
+    <link name="dummy_l">
+    </link>
     <joint name="r_arm_mount_joint" type="prismatic">
         <origin xyz="0.0 0.0 0.0" rpy="0 0 0"/>
@@ -70,22 +95,4 @@
         <limit lower="${shoulder_width_lb}" upper= "${shoulder_width_ub}" effort="1000.0" velocity="20.0"/>
     </joint>
-</xacro:unless>
-<link name="dummy_r">
-</link>
-<link name="dummy_l">
-</link>
-<xacro:if value="$(arg load_sol)">
-    <joint name="roll_r" type="fixed">
-        <origin xyz="0 0.0 0.0" rpy="${roll_mount} 0.0 0.0"/>
-        <parent link="dummy_r"/>
-        <child link="r_arm_mount_frame"/>
-    </joint>
-    <joint name="roll_l" type="fixed">
-        <origin xyz="0 0.0 0.0" rpy="${-roll_mount} 0.0 0.0"/>
-        <parent link="dummy_l"/>
-        <child link="l_arm_mount_frame"/>
-    </joint>
-</xacro:if>
-<xacro:unless value="$(arg load_sol)">
     <joint name="roll_r" type="revolute">
         <origin xyz="0.0 0.0 0.0" rpy="0.0 0.0 0.0"/>
@@ -102,9 +109,9 @@
         <limit lower="${shoulder_roll_lb}" upper="${shoulder_roll_ub}" effort="0.0" velocity="0.0"/>
     </joint>
+    <link name="r_arm_mount_frame">
+    </link>
+    <link name="l_arm_mount_frame">
+    </link>
 </xacro:unless>
-<link name="r_arm_mount_frame">
-</link>
-<link name="l_arm_mount_frame">
-</link>
 <xacro:repair_arm base_link="r_arm_mount_frame" id="1" is_sliding_wrist="$(arg is_sliding_wrist)"
 show_softhand="$(arg show_softhand)" show_coll="$(arg show_coll)" load_sol="$(arg load_sol)"/>

File: repair_urdf/urdf/utils.urdf.xacro (robot description, xacro)
@@ -11,4 +11,7 @@
 <xacro:property name="PI_4" value="0.7853981633974483" />
 <xacro:property name="DEG2RAD" value="${PI/180.0}" />
+<xacro:property name="gazebo_cutoff_inertia" value="0.00000100000000000001" /> <!-- below this value, Gazebo parser ignores links
+To give some  perspective, a grain of sand weights  0.0000045 grams. So this corresponds to less than 1/4 of a grain of sand of
+fake inertia -> it is acceptable. -->
 <xacro:property name="x_joint_limit_margin" value="0.1" />
 <xacro:property name="z_joint_limit_margin" value="0.1" />
@@ -32,9 +35,16 @@
     <color rgba="0.6 0.6 0.6 1"/>
 </material>
+<!-- Macro for adding fake inertias to auxiliary links, so that
+Gazebo does not ignore them. gazebo_cutoff_inertia is the lowest admissible mass value
+under which Gazebo starts to neglect links. The rotational inertias can be put to 0
+without problems.-->
 <xacro:macro name="fake_inertial">
+    <!-- dummy intertia to make Gazebo urdf2sdf converter work -->
     <inertial>
-        <mass value="0.1"/>
-        <inertia ixx="0.0001" ixy="0" ixz="0" iyy="0.0001" iyz="0" izz="0.0001"/>
-        <origin xyz="0 0 0"/>
+      <mass value="${gazebo_cutoff_inertia}" />
+      <origin xyz="0 0 0" />
+      <inertia ixx="0" ixy="0"  ixz="0"
+               iyy="0" iyz="0"
+               izz="0" />
     </inertial>
 </xacro:macro>

Commit message: fixed wrong dummy inertias and added tentative torso mass

File: repair_urdf/urdf/repair_cage.urdf.xacro (robot description, xacro)
@@ -309,5 +309,12 @@
   </joint>
   <link name="working_surface_link">
-    <xacro:fake_inertial/>
+    <!-- Huge inertia (does not matter, is fixed to the world)-->
+      <inertial>
+          <mass value="1" />
+          <origin xyz="0 0 0" />
+          <inertia ixx="0" ixy="0"  ixz="0"
+                  iyy="0" iyz="0"
+                  izz="0" />
+      </inertial>
   </link>
 </robot>

File: repair_urdf/urdf/repair_full.urdf.xacro (robot description, xacro)
@@ -10,19 +10,19 @@
 <xacro:if value="$(arg load_sol)">
     <joint name="x_joint" type="prismatic">
-        <origin xyz="0.0 0.0 0.0" rpy="0.0 0.0 0.0"/>
+        <origin xyz="0.0 0.0 ${mount_h}" rpy="0.0 0.0 0.0"/>
         <parent link="working_surface_link"/>
-        <child link="dummy_link"/>
+        <child link="base_link"/>
         <axis xyz="1 0 0"/>
         <limit lower="${- cage_depth/2 + x_joint_limit_margin}" upper= "${cage_depth/2 - x_joint_limit_margin}" effort="1000.0" velocity="20.0"/>
     </joint>
-    <link name="dummy_link">
-    </link>
-    <!-- RePAIR assembly (two arms) -->
-    <joint name="z_joint" type="fixed">
-        <origin xyz="0.0 0.0 ${mount_h}" rpy="0.0 0.0 0.0"/>
-        <parent link="dummy_link"/>
-        <child link="base_link"/>
-    </joint>
     <link name="base_link">
+        <!-- torso inertias + stuff attached to the sliding guide -->
+        <inertial>
+          <mass value="1000000" />
+          <origin xyz="0 0 0" />
+          <inertia ixx="0" ixy="0"  ixz="0"
+                  iyy="0" iyz="0"
+                  izz="0" />
+        </inertial>
     </link>
     <joint name="r_arm_mount_joint" type="fixed">
@@ -51,8 +51,8 @@
     </joint>
     <link name="r_arm_mount_frame">
-        <xacro:fake_inertial/>
+        <xacro:aux_inertia cutoff_inertia="${gazebo_cutoff_inertia}"/>
     </link>
     <link name="l_arm_mount_frame">
-        <xacro:fake_inertial/>
+        <xacro:aux_inertia cutoff_inertia="${gazebo_cutoff_inertia}"/>
     </link>
 </xacro:if>

File: repair_urdf/urdf/utils.urdf.xacro (robot description, xacro)
@@ -14,4 +14,5 @@
 To give some  perspective, a grain of sand weights  0.0000045 grams. So this corresponds to less than 1/4 of a grain of sand of
 fake inertia -> it is acceptable. -->
+<xacro:property name="full_torso_mass" value="5.0" />
 <xacro:property name="x_joint_limit_margin" value="0.1" />
 <xacro:property name="z_joint_limit_margin" value="0.1" />
@@ -35,12 +36,12 @@
     <color rgba="0.6 0.6 0.6 1"/>
 </material>
-<!-- Macro for adding fake inertias to auxiliary links, so that
+<!-- Macro for adding simple fake inertias to auxiliary links, so that
 Gazebo does not ignore them. gazebo_cutoff_inertia is the lowest admissible mass value
 under which Gazebo starts to neglect links. The rotational inertias can be put to 0
 without problems.-->
-<xacro:macro name="fake_inertial">
+<xacro:macro name="aux_inertia" params="cutoff_inertia">
     <!-- dummy intertia to make Gazebo urdf2sdf converter work -->
     <inertial>
-      <mass value="${gazebo_cutoff_inertia}" />
+      <mass value="${cutoff_inertia}" />
       <origin xyz="0 0 0" />
       <inertia ixx="0" ixy="0"  ixz="0"

Commit message: small update

File: repair_urdf/urdf/repair_cage.urdf.xacro (robot description, xacro)
@@ -14,4 +14,11 @@
   <xacro:property name="PI" value="3.14159265359" />
   <xacro:property name="PI_2" value="1.57079632679" />
+  <!-- only something to avoid collisions between leg and ground plane when using Gaz. -->
+  <xacro:if value="$(arg shorten_table_legs_coll)">
+    <xacro:property name="leg_z_offset_gz" value="0.05" />
+  </xacro:if>
+  <xacro:unless value="$(arg shorten_table_legs_coll)">
+    <xacro:property name="leg_z_offset_gz" value="0.0" />
+  </xacro:unless>
   <material name="wood">
     <color rgba="0.522 0.369 0.259 0.8"/>
@@ -56,5 +63,5 @@
     </visual>
     <collision>
-      <origin xyz="0.0 0.0 ${-table_height/2}" rpy="0.0 0.0 0.0" />
+      <origin xyz="0.0 0.0 ${-table_height/2 + leg_z_offset_gz}" rpy="0.0 0.0 0.0" />
       <geometry>
         <cylinder radius="${leg_radius}" length="${table_height}" />
@@ -96,5 +103,5 @@
     </visual>
     <collision>
-      <origin xyz="0.0 0.0 ${-table_height/2}" rpy="0.0 0.0 0.0" />
+      <origin xyz="0.0 0.0 ${-table_height/2 + leg_z_offset_gz}" rpy="0.0 0.0 0.0" />
       <geometry>
         <cylinder radius="${leg_radius}" length="${table_height}" />
@@ -136,5 +143,5 @@
     </visual>
     <collision>
-      <origin xyz="0.0 0.0 ${-table_height/2}" rpy="0.0 0.0 0.0" />
+      <origin xyz="0.0 0.0 ${-table_height/2 + leg_z_offset_gz}" rpy="0.0 0.0 0.0" />
       <geometry>
         <cylinder radius="${leg_radius}" length="${table_height}" />
@@ -176,5 +183,5 @@
     </visual>
     <collision>
-      <origin xyz="0.0 0.0 ${-table_height/2}" rpy="0.0 0.0 0.0" />
+      <origin xyz="0.0 0.0 ${-table_height/2 + leg_z_offset_gz}" rpy="0.0 0.0 0.0" />
       <geometry>
         <cylinder radius="${leg_radius}" length="${table_height}" />

File: repair_urdf/urdf/repair_full.urdf.xacro (robot description, xacro)
@@ -1,11 +1,16 @@
 <?xml version="1.0"?>
 <robot name = "repair_full" xmlns:xacro="http://ros.org/wiki/xacro">
-<xacro:include filename="$(find repair_urdf)/urdf/repair_arm.urdf.xacro"/>
-<xacro:include filename="$(find repair_urdf)/urdf/repair_cage.urdf.xacro"/>
-<xacro:include filename="$(find repair_urdf)/urdf/repair_opt_mount_params.urdf.xacro"/>
 <xacro:arg name="is_sliding_wrist" default="false" />
 <xacro:arg name="show_softhand" default="false" />
 <xacro:arg name="show_coll" default="false" />
 <xacro:arg name="load_sol" default="false" />
+<xacro:arg name="xbot" default="false" />
+<xacro:arg name="shorten_table_legs_coll" default="false" />
+<xacro:include filename="$(find repair_urdf)/urdf/repair_arm.urdf.xacro"/>
+<xacro:include filename="$(find repair_urdf)/urdf/repair_cage.urdf.xacro"/>
+<xacro:include filename="$(find repair_urdf)/urdf/repair_opt_mount_params.urdf.xacro"/>
+<xacro:if value="$(arg xbot)">
+    <xacro:include filename="$(find repair_urdf)/urdf/xbot2.gazebo.xacro"/>
+</xacro:if>
 <xacro:if value="$(arg load_sol)">
     <joint name="x_joint" type="prismatic">

Commit message: fixed inertias to minimize bouncy behaviour in gz

File: repair_urdf/urdf/repair_cage.urdf.xacro (robot description, xacro)
@@ -318,5 +318,5 @@
     <!-- Huge inertia (does not matter, is fixed to the world)-->
       <inertial>
-          <mass value="1" />
+          <mass value="1000" />
           <origin xyz="0 0 0" />
           <inertia ixx="0" ixy="0"  ixz="0"

File: repair_urdf/urdf/repair_full.urdf.xacro (robot description, xacro)
@@ -6,5 +6,5 @@
 <xacro:arg name="load_sol" default="false" />
 <xacro:arg name="xbot" default="false" />
-<xacro:arg name="shorten_table_legs_coll" default="false" />
+<xacro:arg name="shorten_table_legs_coll" default="false" /> <!-- just to avoid flickering contact when loading into Gazebo -->
 <xacro:include filename="$(find repair_urdf)/urdf/repair_arm.urdf.xacro"/>
 <xacro:include filename="$(find repair_urdf)/urdf/repair_cage.urdf.xacro"/>
@@ -24,5 +24,5 @@
         <!-- torso inertias + stuff attached to the sliding guide -->
         <inertial>
-          <mass value="1000000" />
+          <mass value="${full_torso_mass}" />
           <origin xyz="0 0 0" />
           <inertia ixx="0" ixy="0"  ixz="0"

Commit message: polishing before repo sharing

File: repair_urdf/urdf/repair_cage.urdf.xacro (robot description, xacro)
@@ -16,10 +16,4 @@
   <xacro:property name="PI" value="3.14159265359" />
   <xacro:property name="PI_2" value="1.57079632679" />
-  <!-- only something to avoid collisions between leg and ground plane when using Gaz. -->
-  <!-- <xacro:if value="$(arg shorten_table_legs_coll)">
-    <xacro:property name="leg_z_offset_gz" value="0.05" />
-  </xacro:if>
-    <xacro:property name="leg_z_offset_gz" value="0.0" />
-  </xacro:unless> -->
   <xacro:property name="leg_z_offset_gz" value="0.0" />
   <material name="wood">

File: repair_urdf/urdf/repair_full.urdf.xacro (robot description, xacro)
@@ -9,5 +9,4 @@
 <!-- use_updated_wrist: visual parameter. if true, we load the latest meshes (which are adapted to the
 results of the optimization), otherwise we go with the old ones (generated for a spherical wrist) -->
-<!-- xbot: if true, we add the gazebo tags necessary to use the URDF with XBot2 framework -->
 <robot name = "repair_full" xmlns:xacro="http://ros.org/wiki/xacro">
 <xacro:arg name="is_sliding_wrist" default="false" />
@@ -15,12 +14,8 @@
 <xacro:arg name="load_sol" default="false" />
 <xacro:arg name="use_updated_wrist" default="false" />
-<xacro:arg name="xbot" default="false" />
 <xacro:include filename="$(find repair_urdf)/urdf/repair_arm.urdf.xacro"/>
 <xacro:include filename="$(find repair_urdf)/urdf/repair_cage.urdf.xacro"/>
 <xacro:include filename="$(find repair_urdf)/urdf/repair_opt_mount_params.urdf.xacro"/>
 <xacro:include filename="$(find repair_urdf)/urdf/materials.gazebo.xacro"/>
-<xacro:if value="$(arg xbot)">
-    <xacro:include filename="$(find repair_urdf)/urdf/xbot2.gazebo.xacro"/>
-</xacro:if>
 <!-- <xacro:if value="$(arg gen_coll)">
     <xacro:include filename="$(find repair_urdf)/urdf/repair_torso_coll_params.urdf.xacro"/>
