Commit message: added softhand simple visual

File: repair_urdf/urdf/repair_arm.urdf.xacro (robot description, xacro)
@@ -5,9 +5,10 @@
 <xacro:property name="mid_tau_max" value="200.0" />
 <xacro:property name="sm_tau_max" value="200.0" />
-<xacro:macro name="repair_arm" params="id base_link is_sliding_wrist" >
+<xacro:macro name="repair_arm" params="id base_link is_sliding_wrist show_softhand" >
 <!-- id: 1 for right arm, everything else is considered left arm -->
 <!-- base_link: name of base link a the single arm -->
 <!-- is_sliding_wrist: whether to add a sliding joint along the axis of wrist's second d.o.f.
     (true -> yes), everything else -> no -->
+    <!-- show_softhand: whether to use softhand or not at the TCP -->
 <joint name="arm_${id}_joint_1" type="revolute">
     <xacro:if value="${id == 1}">
@@ -242,8 +243,27 @@
     </collision>
     <visual name="arm_${id}_link_7_visual">
-        <geometry>
-            <mesh filename="package://repair_urdf/meshes/link_7.stl" scale="${mmTom} ${mmTom} ${mmTom}"/>
-        </geometry>
-        <material name="dark"/>
+        <xacro:if value="${show_softhand == True}">
+            <xacro:if value="${id == 1}">
+                <origin xyz="0 0 ${10.0 * mmTom}" rpy="0 ${-(PI_2 + PI_4)} ${-(PI_2)}"/>
+                <geometry>
+                    <mesh filename="package://repair_urdf/meshes/link_7_sh.stl" scale="${mmTom} ${mmTom} ${mmTom}"/>
+                </geometry>
+                <material name="dark"/>
+            </xacro:if>
+            <xacro:unless value="${id == 1}">
+                <origin xyz="0 0 ${10.0 * mmTom}" rpy="0 ${-(PI_2 + PI_4)} ${-(PI_2 + PI)}"/>
+                <geometry>
+                    <mesh filename="package://repair_urdf/meshes/link_7_sh.stl" scale="${mmTom} ${mmTom} ${mmTom}"/>
+                </geometry>
+                <material name="dark"/>
+            </xacro:unless>
+        </xacro:if>
+        <xacro:unless value="${show_softhand == True}">
+            <origin xyz="0 0 0" rpy="0 0 0"/>
+            <geometry>
+                <mesh filename="package://repair_urdf/meshes/link_7.stl" scale="${mmTom} ${mmTom} ${mmTom}"/>
+            </geometry>
+            <material name="dark"/>
+        </xacro:unless>
     </visual>
 </link>

File: repair_urdf/urdf/repair_full.urdf.xacro (robot description, xacro)
@@ -4,4 +4,5 @@
 <xacro:include filename="$(find repair_urdf)/urdf/repair_cage.urdf.xacro"/>
 <xacro:arg name="is_sliding_wrist" default="false" />
+<xacro:arg name="show_softhand" default="false" />
 <joint name="x_joint" type="prismatic">
     <origin xyz="0.0 0.0 0.0" rpy="0.0 0.0 0.0"/>
@@ -59,5 +60,7 @@
 <link name="l_arm_mount_frame">
 </link>
-<xacro:repair_arm base_link="r_arm_mount_frame" id="1" is_sliding_wrist="$(arg is_sliding_wrist)"/>
-<xacro:repair_arm base_link="l_arm_mount_frame" id="2" is_sliding_wrist="$(arg is_sliding_wrist)"/>
+<xacro:repair_arm base_link="r_arm_mount_frame" id="1" is_sliding_wrist="$(arg is_sliding_wrist)"
+show_softhand="$(arg show_softhand)"/>
+<xacro:repair_arm base_link="l_arm_mount_frame" id="2" is_sliding_wrist="$(arg is_sliding_wrist)"
+show_softhand="$(arg show_softhand)"/>
 </robot>

Commit message: added softhand tcp link

File: repair_urdf/urdf/repair_arm.urdf.xacro (robot description, xacro)
@@ -242,36 +242,38 @@
         <material name="dark"/>
     </collision>
-    <visual name="arm_${id}_link_7_visual">
-        <xacro:if value="${show_softhand == True}">
-            <xacro:if value="${id == 1}">
-                <origin xyz="0 0 ${10.0 * mmTom}" rpy="0 ${-(PI_2 + PI_4)} ${-(PI_2)}"/>
+    <xacro:unless value="${show_softhand == True}">
+        <visual name="arm_${id}_link_7_visual">
+                <origin xyz="0 0 0" rpy="0 0 0"/>
                 <geometry>
-                    <mesh filename="package://repair_urdf/meshes/link_7_sh.stl" scale="${mmTom} ${mmTom} ${mmTom}"/>
+                    <mesh filename="package://repair_urdf/meshes/link_7.stl" scale="${mmTom} ${mmTom} ${mmTom}"/>
                 </geometry>
                 <material name="dark"/>
-            </xacro:if>
-            <xacro:unless value="${id == 1}">
-                <origin xyz="0 0 ${10.0 * mmTom}" rpy="0 ${-(PI_2 + PI_4)} ${-(PI_2 + PI)}"/>
-                <geometry>
-                    <mesh filename="package://repair_urdf/meshes/link_7_sh.stl" scale="${mmTom} ${mmTom} ${mmTom}"/>
-                </geometry>
-                <material name="dark"/>
-            </xacro:unless>
-        </xacro:if>
-        <xacro:unless value="${show_softhand == True}">
+        </visual>
+    </xacro:unless>
+</link>
+<xacro:if value="${show_softhand == True}">
+    <joint name="arm_${id}_tcp_joint" type="fixed">
+        <origin xyz="0 0 ${10.0 * mmTom}" rpy="0 ${-(PI_2 + PI_4)} ${-(PI_2)}"/>
+        <parent link="arm_${id}_link_7"/>
+        <child link="arm_${id}_tcp"/>
+    </joint>
+    <link name="arm_${id}_tcp">
+        <visual name="arm_${id}_tcp_visual">
             <origin xyz="0 0 0" rpy="0 0 0"/>
             <geometry>
-                <mesh filename="package://repair_urdf/meshes/link_7.stl" scale="${mmTom} ${mmTom} ${mmTom}"/>
-            </geometry>
-            <material name="dark"/>
-        </xacro:unless>
-    </visual>
-</link>
-<joint name="arm_${id}_tcp_joint" type="fixed">
-    <origin xyz="0 0 0" rpy="0 0 0"/>
-    <parent link="arm_${id}_link_7"/>
-    <child link="arm_${id}_tcp"/>
-</joint>
-<link name="arm_${id}_tcp"/>
+                <mesh filename="package://repair_urdf/meshes/link_7_sh.stl" scale="${mmTom} ${mmTom} ${mmTom}"/>
+            </geometry>
+            <material name="dark"/>
+        </visual>
+    </link>
+</xacro:if>
+<xacro:unless value="${show_softhand == True}">
+    <joint name="arm_${id}_tcp_joint" type="fixed">
+        <origin xyz="0 0 0" rpy="0 0 0"/>
+        <parent link="arm_${id}_link_7"/>
+        <child link="arm_${id}_tcp"/>
+    </joint>
+    <link name="arm_${id}_tcp"/>
+</xacro:unless>
 </xacro:macro>
 </robot>

Commit message: added object size directly in description file

File: repair_urdf/urdf/repair_arm.urdf.xacro (robot description, xacro)
@@ -254,5 +254,6 @@
 <xacro:if value="${show_softhand == True}">
     <joint name="arm_${id}_tcp_joint" type="fixed">
-        <origin xyz="0 0 ${10.0 * mmTom}" rpy="0 ${-(PI_2 + PI_4)} ${-(PI_2)}"/>
+        <origin xyz="0 ${- object_size *  sin(softhand_mount_angle)} ${10.0 * mmTom + object_size *  cos(softhand_mount_angle)}"
+                rpy="0 ${-(PI_2 + softhand_mount_angle)} ${-(PI_2)}"/>
         <parent link="arm_${id}_link_7"/>
         <child link="arm_${id}_tcp"/>
@@ -260,5 +261,5 @@
     <link name="arm_${id}_tcp">
         <visual name="arm_${id}_tcp_visual">
-            <origin xyz="0 0 0" rpy="0 0 0"/>
+            <origin xyz="0 0 ${object_size}" rpy="0 0 0"/>
             <geometry>
                 <mesh filename="package://repair_urdf/meshes/link_7_sh.stl" scale="${mmTom} ${mmTom} ${mmTom}"/>

File: repair_urdf/urdf/utils.urdf.xacro (robot description, xacro)
@@ -18,4 +18,6 @@
 <xacro:property name="sliding_wrist_deltaz_lb" value="0" />
 <xacro:property name="sliding_wrist_deltaz_ub" value="0.05" />
+<xacro:property name="softhand_mount_angle" value="${PI_4}" />
+<xacro:property name="object_size" value="0.08" />
 <!-- color -->
 <material name="darkblue">

Commit message: so many changes. I should have commited before

File: repair_urdf/urdf/repair_arm.urdf.xacro (robot description, xacro)
@@ -5,5 +5,9 @@
 <xacro:property name="mid_tau_max" value="200.0" />
 <xacro:property name="sm_tau_max" value="200.0" />
-<xacro:macro name="repair_arm" params="id base_link is_sliding_wrist show_softhand" >
+<xacro:include filename="$(find repair_urdf)/urdf/repair_arm_coll_params.urdf.xacro"/>
+<xacro:macro name="repair_arm" params="id base_link is_sliding_wrist show_softhand show_coll" >
+<xacro:if value="${show_coll == True}">
+    <xacro:include filename="$(find repair_urdf)/urdf/repair_arm_coll.urdf.xacro"/>
+</xacro:if>
 <!-- id: 1 for right arm, everything else is considered left arm -->
 <!-- base_link: name of base link a the single arm -->

File: repair_urdf/urdf/repair_full.urdf.xacro (robot description, xacro)
@@ -5,4 +5,5 @@
 <xacro:arg name="is_sliding_wrist" default="false" />
 <xacro:arg name="show_softhand" default="false" />
+<xacro:arg name="show_coll" default="false" />
 <joint name="x_joint" type="prismatic">
     <origin xyz="0.0 0.0 0.0" rpy="0.0 0.0 0.0"/>
@@ -61,6 +62,6 @@
 </link>
 <xacro:repair_arm base_link="r_arm_mount_frame" id="1" is_sliding_wrist="$(arg is_sliding_wrist)"
-show_softhand="$(arg show_softhand)"/>
+show_softhand="$(arg show_softhand)" show_coll="$(arg show_coll)"/>
 <xacro:repair_arm base_link="l_arm_mount_frame" id="2" is_sliding_wrist="$(arg is_sliding_wrist)"
-show_softhand="$(arg show_softhand)"/>
+show_softhand="$(arg show_softhand)" show_coll="$(arg show_coll)"/>
 </robot>

File: repair_urdf/urdf/utils.urdf.xacro (robot description, xacro)
@@ -11,5 +11,5 @@
 <xacro:property name="x_joint_limit_margin" value="0.1" />
 <xacro:property name="z_joint_limit_margin" value="0.1" />
-<xacro:property name="z_joint_lb" value="0.5" />
+<xacro:property name="z_joint_lb" value="0.0" />
 <xacro:property name="shoulder_width_lb" value="0.25" /> <!-- wrt shoulder center -->
 <xacro:property name="shoulder_width_ub" value="0.5" />
@@ -19,8 +19,11 @@
 <xacro:property name="sliding_wrist_deltaz_ub" value="0.05" />
 <xacro:property name="softhand_mount_angle" value="${PI_4}" />
-<xacro:property name="object_size" value="0.01" />
+<xacro:property name="object_size" value="0.02" />
 <!-- color -->
 <material name="darkblue">
     <color rgba="0.0 0.3 0.9 1"/>
+</material>
+<material name="darkred">
+    <color rgba="0.55 0.0 0.0 1"/>
 </material>
 <material name="dark">

Commit message: make tcp frame symmetric from left to right

File: repair_urdf/urdf/repair_arm.urdf.xacro (robot description, xacro)
@@ -227,5 +227,6 @@
     </xacro:if>
     <xacro:unless value="${id == 1}">
-        <origin xyz="${180.000 * mmTom} 0 0" rpy="${-PI_2} 0 ${-PI_2}"/>
+        <origin xyz="${180.000 * mmTom} 0 0" rpy="${-PI_2} ${PI} ${-PI_2}"/>
+        <!-- <origin xyz="${180.000 * mmTom} 0 0" rpy="${-PI_2} 0 ${-PI_2}"/> -->
     </xacro:unless>
     <parent link="arm_${id}_link_6"/>

Commit message: added inertial parameters

File: repair_urdf/urdf/repair_arm.urdf.xacro (robot description, xacro)
@@ -29,7 +29,7 @@
 <link name="arm_${id}_link_1">
     <inertial>
-        <mass value="0.1"/>
-        <inertia ixx="0.0001" ixy="0" ixz="0" iyy="0.0001" iyz="0" izz="0.0001"/>
-        <origin xyz="0 0 0"/>
+        <mass value="2"/>
+        <inertia ixx="${1500 * kgmm2_2_kgm2}" ixy="${-100 * kgmm2_2_kgm2}" ixz="${0 * kgmm2_2_kgm2}" iyy="{2700 * kgmm2_2_kgm2}" iyz="${100 * kgmm2_2_kgm2}" izz="${2800 * kgmm2_2_kgm2}"/>
+        <origin xyz="0 0 ${-10.0 * mmTom}"/>
     </inertial>
     <xacro:if value="${id == 1}">
@@ -76,7 +76,7 @@
 <link name="arm_${id}_link_2">
     <inertial>
-        <mass value="0.1"/>
-        <inertia ixx="0.0001" ixy="0" ixz="0" iyy="0.0001" iyz="0" izz="0.0001"/>
-        <origin xyz="0 0 0"/>
+        <mass value="0.4"/>
+        <inertia ixx="${670 * kgmm2_2_kgm2}" ixy="${0 * kgmm2_2_kgm2}" ixz="${180 * kgmm2_2_kgm2}" iyy="{970 * kgmm2_2_kgm2}" iyz="${0 * kgmm2_2_kgm2}" izz="${1000 * kgmm2_2_kgm2}"/>
+        <origin xyz="${40 * mmTom} ${0 * mmTom} ${35.0 * mmTom}"/>
     </inertial>
     <collision name="arm_${id}_link_2_collision">
@@ -107,7 +107,7 @@
 <link name="arm_${id}_link_3">
     <inertial>
-        <mass value="0.1"/>
-        <inertia ixx="0.0001" ixy="0" ixz="0" iyy="0.0001" iyz="0" izz="0.0001"/>
-        <origin xyz="0 0 0"/>
+        <mass value="3.3"/>
+        <inertia ixx="${25000 * kgmm2_2_kgm2}" ixy="${0 * kgmm2_2_kgm2}" ixz="${0 * kgmm2_2_kgm2}" iyy="{26000 * kgmm2_2_kgm2}" iyz="${0 * kgmm2_2_kgm2}" izz="${22000 * kgmm2_2_kgm2}"/>
+        <origin xyz="${0 * mmTom} ${-25 * mmTom} ${230.0 * mmTom}"/>
     </inertial>
     <collision name="arm_${id}_link_3_collision">
@@ -133,7 +133,7 @@
 <link name="arm_${id}_link_4">
     <inertial>
-        <mass value="0.1"/>
-        <inertia ixx="0.0001" ixy="0" ixz="0" iyy="0.0001" iyz="0" izz="0.0001"/>
-        <origin xyz="0 0 0"/>
+        <mass value="0.4"/>
+        <inertia ixx="${670 * kgmm2_2_kgm2}" ixy="${0 * kgmm2_2_kgm2}" ixz="${180 * kgmm2_2_kgm2}" iyy="{970 * kgmm2_2_kgm2}" iyz="${0 * kgmm2_2_kgm2}" izz="${1000 * kgmm2_2_kgm2}"/>
+        <origin xyz="${40 * mmTom} ${0 * mmTom} ${35.0 * mmTom}"/>
     </inertial>
     <collision name="arm_${id}_link_4_collision">
@@ -159,7 +159,7 @@
 <link name="arm_${id}_link_5">
     <inertial>
-        <mass value="0.1"/>
-        <inertia ixx="0.0001" ixy="0" ixz="0" iyy="0.0001" iyz="0" izz="0.0001"/>
-        <origin xyz="0 0 0"/>
+        <mass value="2.8"/>
+        <inertia ixx="${32000 * kgmm2_2_kgm2}" ixy="${0 * kgmm2_2_kgm2}" ixz="${1700 * kgmm2_2_kgm2}" iyy="{34000 * kgmm2_2_kgm2}" iyz="${0 * kgmm2_2_kgm2}" izz="${29000 * kgmm2_2_kgm2}"/>
+        <origin xyz="${-5 * mmTom} ${0 * mmTom} ${200.0 * mmTom}"/>
     </inertial>
     <collision name="arm_${id}_link_5_collision">
@@ -205,7 +205,7 @@
 <link name="arm_${id}_link_6">
     <inertial>
-        <mass value="0.1"/>
-        <inertia ixx="0.0001" ixy="0" ixz="0" iyy="0.0001" iyz="0" izz="0.0001"/>
-        <origin xyz="0 0 0"/>
+        <mass value="1.8"/>
+        <inertia ixx="${1700 * kgmm2_2_kgm2}" ixy="${0 * kgmm2_2_kgm2}" ixz="${0 * kgmm2_2_kgm2}" iyy="{2500 * kgmm2_2_kgm2}" iyz="${100 * kgmm2_2_kgm2}" izz="${2700 * kgmm2_2_kgm2}"/>
+        <origin xyz="${0 * mmTom} ${0 * mmTom} ${0 * mmTom}"/>
     </inertial>
     <collision name="arm_${id}_link_6_collision">
@@ -237,7 +237,7 @@
 <link name="arm_${id}_link_7">
     <inertial>
-        <mass value="0.1"/>
-        <inertia ixx="0.0001" ixy="0" ixz="0" iyy="0.0001" iyz="0" izz="0.0001"/>
-        <origin xyz="0 0 0"/>
+        <mass value="1.5"/>
+        <inertia ixx="${25000 * kgmm2_2_kgm2}" ixy="${0 * kgmm2_2_kgm2}" ixz="${0 * kgmm2_2_kgm2}" iyy="{25000 * kgmm2_2_kgm2}" iyz="${100 * kgmm2_2_kgm2}" izz="${23000 * kgmm2_2_kgm2}"/>
+        <origin xyz="${0 * mmTom} ${0 * mmTom} ${0 * mmTom}"/>
     </inertial>
     <collision name="arm_${id}_link_7_collision">

File: repair_urdf/urdf/utils.urdf.xacro (robot description, xacro)
@@ -5,4 +5,5 @@
 <xacro:property name="mm2Tom2" value="${0.001*0.001}" />
 <xacro:property name="tonsToKg" value="1000.0" />
+<xacro:property name="kgmm2_2_kgm2" value="${1e-06}" />
 <xacro:property name="PI" value="3.14159265359" />
 <xacro:property name="PI_2" value="1.57079632679" />

Commit message: little update

File: repair_urdf/urdf/repair_arm.urdf.xacro (robot description, xacro)
@@ -30,5 +30,5 @@
     <inertial>
         <mass value="2"/>
-        <inertia ixx="${1500 * kgmm2_2_kgm2}" ixy="${-100 * kgmm2_2_kgm2}" ixz="${0 * kgmm2_2_kgm2}" iyy="{2700 * kgmm2_2_kgm2}" iyz="${100 * kgmm2_2_kgm2}" izz="${2800 * kgmm2_2_kgm2}"/>
+        <inertia ixx="${1500.0 * kgmm2_2_kgm2}" ixy="${-100.0 * kgmm2_2_kgm2}" ixz="${0.0 * kgmm2_2_kgm2}" iyy="${2700.0 * kgmm2_2_kgm2}" iyz="${100.0 * kgmm2_2_kgm2}" izz="${2800.0 * kgmm2_2_kgm2}"/>
         <origin xyz="0 0 ${-10.0 * mmTom}"/>
     </inertial>
@@ -77,5 +77,5 @@
     <inertial>
         <mass value="0.4"/>
-        <inertia ixx="${670 * kgmm2_2_kgm2}" ixy="${0 * kgmm2_2_kgm2}" ixz="${180 * kgmm2_2_kgm2}" iyy="{970 * kgmm2_2_kgm2}" iyz="${0 * kgmm2_2_kgm2}" izz="${1000 * kgmm2_2_kgm2}"/>
+        <inertia ixx="${670 * kgmm2_2_kgm2}" ixy="${0 * kgmm2_2_kgm2}" ixz="${180 * kgmm2_2_kgm2}" iyy="${970 * kgmm2_2_kgm2}" iyz="${0 * kgmm2_2_kgm2}" izz="${1000 * kgmm2_2_kgm2}"/>
         <origin xyz="${40 * mmTom} ${0 * mmTom} ${35.0 * mmTom}"/>
     </inertial>
@@ -108,5 +108,5 @@
     <inertial>
         <mass value="3.3"/>
-        <inertia ixx="${25000 * kgmm2_2_kgm2}" ixy="${0 * kgmm2_2_kgm2}" ixz="${0 * kgmm2_2_kgm2}" iyy="{26000 * kgmm2_2_kgm2}" iyz="${0 * kgmm2_2_kgm2}" izz="${22000 * kgmm2_2_kgm2}"/>
+        <inertia ixx="${25000 * kgmm2_2_kgm2}" ixy="${0 * kgmm2_2_kgm2}" ixz="${0 * kgmm2_2_kgm2}" iyy="${26000 * kgmm2_2_kgm2}" iyz="${0 * kgmm2_2_kgm2}" izz="${22000 * kgmm2_2_kgm2}"/>
         <origin xyz="${0 * mmTom} ${-25 * mmTom} ${230.0 * mmTom}"/>
     </inertial>
@@ -134,5 +134,5 @@
     <inertial>
         <mass value="0.4"/>
-        <inertia ixx="${670 * kgmm2_2_kgm2}" ixy="${0 * kgmm2_2_kgm2}" ixz="${180 * kgmm2_2_kgm2}" iyy="{970 * kgmm2_2_kgm2}" iyz="${0 * kgmm2_2_kgm2}" izz="${1000 * kgmm2_2_kgm2}"/>
+        <inertia ixx="${670 * kgmm2_2_kgm2}" ixy="${0 * kgmm2_2_kgm2}" ixz="${180 * kgmm2_2_kgm2}" iyy="${970 * kgmm2_2_kgm2}" iyz="${0 * kgmm2_2_kgm2}" izz="${1000 * kgmm2_2_kgm2}"/>
         <origin xyz="${40 * mmTom} ${0 * mmTom} ${35.0 * mmTom}"/>
     </inertial>
@@ -160,5 +160,5 @@
     <inertial>
         <mass value="2.8"/>
-        <inertia ixx="${32000 * kgmm2_2_kgm2}" ixy="${0 * kgmm2_2_kgm2}" ixz="${1700 * kgmm2_2_kgm2}" iyy="{34000 * kgmm2_2_kgm2}" iyz="${0 * kgmm2_2_kgm2}" izz="${29000 * kgmm2_2_kgm2}"/>
+        <inertia ixx="${32000 * kgmm2_2_kgm2}" ixy="${0 * kgmm2_2_kgm2}" ixz="${1700 * kgmm2_2_kgm2}" iyy="${34000 * kgmm2_2_kgm2}" iyz="${0 * kgmm2_2_kgm2}" izz="${29000 * kgmm2_2_kgm2}"/>
         <origin xyz="${-5 * mmTom} ${0 * mmTom} ${200.0 * mmTom}"/>
     </inertial>
@@ -206,5 +206,5 @@
     <inertial>
         <mass value="1.8"/>
-        <inertia ixx="${1700 * kgmm2_2_kgm2}" ixy="${0 * kgmm2_2_kgm2}" ixz="${0 * kgmm2_2_kgm2}" iyy="{2500 * kgmm2_2_kgm2}" iyz="${100 * kgmm2_2_kgm2}" izz="${2700 * kgmm2_2_kgm2}"/>
+        <inertia ixx="${1700 * kgmm2_2_kgm2}" ixy="${0 * kgmm2_2_kgm2}" ixz="${0 * kgmm2_2_kgm2}" iyy="${2500 * kgmm2_2_kgm2}" iyz="${100 * kgmm2_2_kgm2}" izz="${2700 * kgmm2_2_kgm2}"/>
         <origin xyz="${0 * mmTom} ${0 * mmTom} ${0 * mmTom}"/>
     </inertial>
@@ -238,5 +238,5 @@
     <inertial>
         <mass value="1.5"/>
-        <inertia ixx="${25000 * kgmm2_2_kgm2}" ixy="${0 * kgmm2_2_kgm2}" ixz="${0 * kgmm2_2_kgm2}" iyy="{25000 * kgmm2_2_kgm2}" iyz="${100 * kgmm2_2_kgm2}" izz="${23000 * kgmm2_2_kgm2}"/>
+        <inertia ixx="${25000 * kgmm2_2_kgm2}" ixy="${0 * kgmm2_2_kgm2}" ixz="${0 * kgmm2_2_kgm2}" iyy="${25000 * kgmm2_2_kgm2}" iyz="${100 * kgmm2_2_kgm2}" izz="${23000 * kgmm2_2_kgm2}"/>
         <origin xyz="${0 * mmTom} ${0 * mmTom} ${0 * mmTom}"/>
     </inertial>
