Commit message: added option to fix urdf to optimal paramters

File: repair_urdf/urdf/repair_arm.urdf.xacro (robot description, xacro)
@@ -6,7 +6,8 @@
 <xacro:property name="sm_tau_max" value="200.0" />
 <xacro:include filename="$(find repair_urdf)/urdf/repair_arm_coll_params.urdf.xacro"/>
-<xacro:macro name="repair_arm" params="id base_link is_sliding_wrist show_softhand show_coll" >
+<xacro:macro name="repair_arm" params="id base_link is_sliding_wrist show_softhand show_coll load_sol" >
 <xacro:if value="${show_coll == True}">
     <xacro:include filename="$(find repair_urdf)/urdf/repair_arm_coll.urdf.xacro"/>
+    <xacro:repair_coll load_sol="${load_sol}"/>
 </xacro:if>
 <!-- id: 1 for right arm, everything else is considered left arm -->
@@ -187,19 +188,28 @@
 <xacro:unless value="${is_sliding_wrist != True}">
     <joint name="arm_${id}_joint_6" type="revolute">
-        <origin xyz="0 0 ${321.000 * mmTom}" rpy="0 ${-PI_2} 0"/>
-        <parent link="arm_${id}_link_5"/>
-        <child link="dummy_sliding_wrist${id}_link"/>
-        <axis xyz="0 0 1"/>
-        <limit lower="${-150.0 * DEG2RAD}" upper="${150.0 * DEG2RAD}" effort="${big_tau_max}" velocity="10.0"/>
+            <origin xyz="0 0 ${321.000 * mmTom}" rpy="0 ${-PI_2} 0"/>
+            <parent link="arm_${id}_link_5"/>
+            <child link="dummy_sliding_wrist${id}_link"/>
+            <axis xyz="0 0 1"/>
+            <limit lower="${-150.0 * DEG2RAD}" upper="${150.0 * DEG2RAD}" effort="${big_tau_max}" velocity="10.0"/>
     </joint>
     <link name="dummy_sliding_wrist${id}_link">
     </link>
-    <joint name="dummy_sliding_wrist${id}_joint" type="prismatic">
-        <origin xyz="0.0 0.0 0.0" rpy="0 0 0"/>
-        <parent link="dummy_sliding_wrist${id}_link"/>
-        <child link="arm_${id}_link_6"/>
-        <axis xyz="0 0 -1"/>
-        <limit lower="${sliding_wrist_deltaz_lb}" upper= "${sliding_wrist_deltaz_ub}" effort="1000.0" velocity="20.0"/>
-    </joint>
+    <xacro:if value="${load_sol == True}">
+        <joint name="dummy_sliding_wrist${id}_joint" type="fixed">
+            <origin xyz="0.0 0.0 ${-wrist_off}" rpy="0 0 0"/>
+            <parent link="dummy_sliding_wrist${id}_link"/>
+            <child link="arm_${id}_link_6"/>
+        </joint>
+    </xacro:if>
+    <xacro:unless value="${load_sol == True}">
+        <joint name="dummy_sliding_wrist${id}_joint" type="prismatic">
+            <origin xyz="0.0 0.0 0.0" rpy="0 0 0"/>
+            <parent link="dummy_sliding_wrist${id}_link"/>
+            <child link="arm_${id}_link_6"/>
+            <axis xyz="0 0 -1"/>
+            <limit lower="${sliding_wrist_deltaz_lb}" upper= "${sliding_wrist_deltaz_ub}" effort="1000.0" velocity="20.0"/>
+        </joint>
+    </xacro:unless>
 </xacro:unless>
 <link name="arm_${id}_link_6">

File: repair_urdf/urdf/repair_arm_coll.urdf.xacro (robot description, xacro)
@@ -1,4 +1,5 @@
 <?xml version="1.0"?>
 <robot xmlns:xacro="http://www.ros.org/wiki/xacro">
+<xacro:macro name="repair_coll" params="load_sol" />
 <joint name="arm_${id}_link_1_coll_joint" type="fixed">
     <origin xyz="${link1_coll_offset_x} ${link1_coll_offset_y} ${link1_coll_offset_z}" rpy="0 0 0"/>
@@ -57,11 +58,20 @@
     </visual>
 </link>
-<joint name="arm_${id}_link_5_coll_joint" type="prismatic">
-    <origin xyz="${link5_coll_offset_x} ${link5_coll_offset_y} ${link5_coll_offset_z}" rpy="0 0 0"/>
-    <parent link="arm_${id}_link_5"/>
-    <child link="arm_${id}_link5_coll"/>
-    <limit lower="${0}" upper="${sliding_wrist_deltaz_ub}" effort="${big_tau_max}" velocity="10.0"/>
-    <axis xyz="1 0 0"/>
-</joint>
+<xacro:if value="${load_sol == True}">
+    <joint name="arm_${id}_link_5_coll_joint" type="fixed">
+         <origin xyz="${link5_coll_offset_x + wrist_off} ${link5_coll_offset_y} ${link5_coll_offset_z}" rpy="0 0 0"/>
+        <parent link="arm_${id}_link_5"/>
+        <child link="arm_${id}_link5_coll"/>
+    </joint>
+</xacro:if>
+<xacro:unless value="${load_sol == True}">
+    <joint name="arm_${id}_link_5_coll_joint" type="prismatic">
+        <origin xyz="${link5_coll_offset_x} ${link5_coll_offset_y} ${link5_coll_offset_z}" rpy="0 0 0"/>
+        <parent link="arm_${id}_link_5"/>
+        <child link="arm_${id}_link5_coll"/>
+        <limit lower="${0}" upper="${sliding_wrist_deltaz_ub}" effort="${big_tau_max}" velocity="10.0"/>
+        <axis xyz="1 0 0"/>
+    </joint>
+</xacro:unless>
 <link name="arm_${id}_link5_coll">
     <visual name="arm_${id}_link5_coll_visual">

File: repair_urdf/urdf/repair_cage.urdf.xacro (robot description, xacro)
@@ -28,11 +28,4 @@
   </joint>
   <link name="table_top_link">
-    <inertial>
-      <mass value="1.0" />
-      <origin xyz="${table_x} ${table_y} ${table_z+table_height-table_top_thickness/2}" />
-      <inertia ixx="1" ixy="0"  ixz="0"
-               iyy="1" iyz="0"
-               izz="1" />
-    </inertial>
     <visual>
       <origin xyz="${table_x} ${table_y} ${table_z+table_height-table_top_thickness/2}" />
@@ -55,11 +48,4 @@
   </joint>
   <link name="leg1_link">
-    <inertial>
-      <mass value="1.0" />
-      <origin xyz="0 0 ${-table_height/2}" />
-      <inertia ixx="0.1" ixy="0"  ixz="0"
-               iyy="0.1" iyz="0"
-               izz="0.01" />
-    </inertial>
     <visual>
       <origin xyz="0.0 0.0 ${-table_height/2}" rpy="0 0 0" />
@@ -82,4 +68,246 @@
   </joint>
   <link name="vbar1_link">
+    <visual>
+      <origin xyz="0.0 0.0 0" rpy="0 0 0" />
+      <geometry>
+        <cylinder radius="${leg_radius}" length="${cage_height}" />
+      </geometry>
+    <material name="silver_gray" />
+    </visual>
+    <collision>
+      <origin xyz="0.0 0.0 0" rpy="0.0 0.0 0.0" />
+      <geometry>
+        <cylinder radius="${leg_radius}" length="${cage_height}" />
+      </geometry>
+    </collision>
+  </link>
+  <joint name="leg2_joint" type="fixed" >
+    <parent link="table_top_link" />
+    <origin xyz="${table_x-cage_width/2} ${table_y+cage_depth/2} ${table_z+table_height}" rpy="0 0 0" />
+    <child link="leg2_link" />
+  </joint>
+  <link name="leg2_link">
+    <visual>
+      <origin xyz="0.0 0.0 ${-table_height/2}" rpy="0 0 0" />
+      <geometry>
+        <cylinder radius="${leg_radius}" length="${table_height}" />
+      </geometry>
+      <material name="silver_gray" />
+    </visual>
+    <collision>
+      <origin xyz="0.0 0.0 ${-table_height/2}" rpy="0.0 0.0 0.0" />
+      <geometry>
+        <cylinder radius="${leg_radius}" length="${table_height}" />
+      </geometry>
+    </collision>
+  </link>
+  <joint name="vbar2_joint" type="fixed" >
+    <parent link="leg2_link" />
+    <origin xyz="0 0 ${cage_height/2}" rpy="0 0 0" />
+    <child link="vbar2_link" />
+  </joint>
+  <link name="vbar2_link">
+    <visual>
+      <origin xyz="0.0 0.0 0" rpy="0 0 0" />
+      <geometry>
+        <cylinder radius="${leg_radius}" length="${cage_height}" />
+      </geometry>
+    <material name="silver_gray" />
+    </visual>
+    <collision>
+      <origin xyz="0.0 0.0 0" rpy="0.0 0.0 0.0" />
+      <geometry>
+        <cylinder radius="${leg_radius}" length="${cage_height}" />
+      </geometry>
+    </collision>
+  </link>
+  <joint name="leg3_joint" type="fixed" >
+    <parent link="table_top_link" />
+    <origin xyz="${table_x+cage_width/2} ${table_y-cage_depth/2} ${table_z+table_height}" rpy="0 0 0" />
+    <child link="leg3_link" />
+  </joint>
+  <link name="leg3_link">
+    <visual>
+      <origin xyz="0.0 0.0 ${-table_height/2}" rpy="0 0 0" />
+      <geometry>
+        <cylinder radius="${leg_radius}" length="${table_height}" />
+      </geometry>
+      <material name="silver_gray" />
+    </visual>
+    <collision>
+      <origin xyz="0.0 0.0 ${-table_height/2}" rpy="0.0 0.0 0.0" />
+      <geometry>
+        <cylinder radius="${leg_radius}" length="${table_height}" />
+      </geometry>
+    </collision>
+  </link>
+  <joint name="vbar3_joint" type="fixed" >
+    <parent link="leg3_link" />
+    <origin xyz="0 0 ${cage_height/2}" rpy="0 0 0" />
+    <child link="vbar3_link" />
+  </joint>
+  <link name="vbar3_link">
+    <visual>
+      <origin xyz="0.0 0.0 0" rpy="0 0 0" />
+      <geometry>
+        <cylinder radius="${leg_radius}" length="${cage_height}" />
+      </geometry>
+    <material name="silver_gray" />
+    </visual>
+    <collision>
+      <origin xyz="0.0 0.0 0" rpy="0.0 0.0 0.0" />
+      <geometry>
+        <cylinder radius="${leg_radius}" length="${cage_height}" />
+      </geometry>
+    </collision>
+  </link>
+  <joint name="leg4_joint" type="fixed" >
+    <parent link="table_top_link" />
+    <origin xyz="${table_x-cage_width/2} ${table_y-cage_depth/2} ${table_z+table_height}" rpy="0 0 0" />
+    <child link="leg4_link" />
+  </joint>
+  <link name="leg4_link">
+    <visual>
+      <origin xyz="0.0 0.0 ${-table_height/2}" rpy="0 0 0" />
+      <geometry>
+        <cylinder radius="${leg_radius}" length="${table_height}" />
+      </geometry>
+      <material name="silver_gray" />
+    </visual>
+    <collision>
+      <origin xyz="0.0 0.0 ${-table_height/2}" rpy="0.0 0.0 0.0" />
+      <geometry>
+        <cylinder radius="${leg_radius}" length="${table_height}" />
+      </geometry>
+    </collision>
+  </link>
+  <joint name="vbar4_joint" type="fixed" >
+    <parent link="leg4_link" />
+    <origin xyz="0 0 ${cage_height/2}" rpy="0 0 0" />
+    <child link="vbar4_link" />
+  </joint>
+  <link name="vbar4_link">
+    <visual>
+      <origin xyz="0.0 0.0 0" rpy="0 0 0" />
+      <geometry>
+        <cylinder radius="${leg_radius}" length="${cage_height}" />
+      </geometry>
+    <material name="silver_gray" />
+    </visual>
+    <collision>
+      <origin xyz="0.0 0.0 0" rpy="0.0 0.0 0.0" />
+      <geometry>
+        <cylinder radius="${leg_radius}" length="${cage_height}" />
+      </geometry>
+    </collision>
+  </link>
+  <joint name="obar1_joint" type="fixed" >
+    <parent link="vbar1_link" />
+    <origin xyz="-${cage_width/2} 0 ${cage_height/2}" rpy="0 -${PI_2} 0" />
+    <child link="obar1_link" />
+  </joint>
+  <link name="obar1_link">
+    <visual>
+      <origin xyz="0.0 0.0 0" rpy="0 0 0" />
+      <geometry>
+        <cylinder radius="${leg_radius}" length="${cage_width}" />
+      </geometry>
+    <material name="silver_gray" />
+    </visual>
+    <collision>
+      <origin xyz="0.0 0.0 0" rpy="0.0 0.0 0.0" />
+      <geometry>
+        <cylinder radius="${leg_radius}" length="${cage_width}" />
+      </geometry>
+    </collision>
+  </link>
+  <joint name="obar2_joint" type="fixed" >
+    <parent link="vbar3_link" />
+    <origin xyz="-${cage_width/2} 0 ${cage_height/2}" rpy="0 -${PI_2} 0" />
+    <child link="obar2_link" />
+  </joint>
+  <link name="obar2_link">
+    <visual>
+      <origin xyz="0.0 0.0 0" rpy="0 0 0" />
+      <geometry>
+        <cylinder radius="${leg_radius}" length="${cage_width}" />
+      </geometry>
+    <material name="silver_gray" />
+    </visual>
+    <collision>
+      <origin xyz="0.0 0.0 0" rpy="0.0 0.0 0.0" />
+      <geometry>
+        <cylinder radius="${leg_radius}" length="${cage_width}" />
+      </geometry>
+    </collision>
+  </link>
+  <joint name="obar3_joint" type="fixed" >
+    <parent link="vbar3_link" />
+    <origin xyz="0 ${cage_depth/2} ${cage_height/2}" rpy="-${PI_2} 0 0" />
+    <child link="obar3_link" />
+  </joint>
+  <link name="obar3_link">
+    <visual>
+      <origin xyz="0.0 0.0 0" rpy="0 0 0" />
+      <geometry>
+        <cylinder radius="${leg_radius}" length="${cage_depth}" />
+      </geometry>
+    <material name="silver_gray" />
+    </visual>
+    <collision>
+      <origin xyz="0.0 0.0 0" rpy="0.0 0.0 0.0" />
+      <geometry>
+        <cylinder radius="${leg_radius}" length="${cage_depth}" />
+      </geometry>
+    </collision>
+  </link>
+  <joint name="obar4_joint" type="fixed" >
+    <parent link="vbar4_link" />
+    <origin xyz="0 ${cage_depth/2} ${cage_height/2}" rpy="-${PI_2} 0 0" />
+    <child link="obar4_link" />
+  </joint>
+  <link name="obar4_link">
+    <!-- dummy intertia to make Gazebo urdf2sdf converter work -->
+    <visual>
+      <origin xyz="0.0 0.0 0" rpy="0 0 0" />
+      <geometry>
+        <cylinder radius="${leg_radius}" length="${cage_depth}" />
+      </geometry>
+    <material name="silver_gray" />
+    </visual>
+    <collision>
+      <origin xyz="0.0 0.0 0" rpy="0.0 0.0 0.0" />
+      <geometry>
+        <cylinder radius="${leg_radius}" length="${cage_depth}" />
+      </geometry>
+    </collision>
+  </link>
+  <joint name="sliding_guide_joint" type="fixed" >
+    <parent link="obar2_link" />
+    <origin xyz="0 ${cage_depth/2} 0" rpy="-${PI_2} 0 0" />
+    <child link="sliding_guide_link" />
+  </joint>
+  <link name="sliding_guide_link">
+    <visual>
+      <origin xyz="0.0 0.0 0" rpy="0 0 0" />
+      <geometry>
+        <box size="0.001 ${sliding_guide_width} ${cage_depth}" />
+      </geometry>
+    <material name="silver_gray" />
+    </visual>
+    <collision>
+      <origin xyz="0.0 0.0 0" rpy="0.0 0.0 0.0" />
+      <geometry>
+        <cylinder radius="${leg_radius}" length="${cage_depth}" />
+      </geometry>
+    </collision>
+  </link>
+  <joint name="working_surface_joint" type="fixed" >
+    <parent link="sliding_guide_link" />
+    <origin xyz="-${cage_height} 0 0" rpy="0.0 -${PI_2} ${PI}" />
+    <child link="working_surface_link" />
+  </joint>
+  <link name="working_surface_link">
+    <!-- dummy intertia to make Gazebo urdf2sdf converter work -->
     <inertial>
       <mass value="1.0" />
@@ -89,321 +317,4 @@
                izz="0.01" />
     </inertial>
-    <visual>
-      <origin xyz="0.0 0.0 0" rpy="0 0 0" />
-      <geometry>
-        <cylinder radius="${leg_radius}" length="${cage_height}" />
-      </geometry>
-    <material name="silver_gray" />
-    </visual>
-    <collision>
-      <origin xyz="0.0 0.0 0" rpy="0.0 0.0 0.0" />
-      <geometry>
-        <cylinder radius="${leg_radius}" length="${cage_height}" />
-      </geometry>
-    </collision>
-  </link>
-  <joint name="leg2_joint" type="fixed" >
-    <parent link="table_top_link" />
-    <origin xyz="${table_x-cage_width/2} ${table_y+cage_depth/2} ${table_z+table_height}" rpy="0 0 0" />
-    <child link="leg2_link" />
-  </joint>
-  <link name="leg2_link">
-    <inertial>
-      <mass value="1.0" />
-      <origin xyz="0 0 ${-table_height/2}" />
-      <inertia ixx="0.1" ixy="0"  ixz="0"
-               iyy="0.1" iyz="0"
-               izz="0.01" />
-    </inertial>
-    <visual>
-      <origin xyz="0.0 0.0 ${-table_height/2}" rpy="0 0 0" />
-      <geometry>
-        <cylinder radius="${leg_radius}" length="${table_height}" />
-      </geometry>
-      <material name="silver_gray" />
-    </visual>
-    <collision>
-      <origin xyz="0.0 0.0 ${-table_height/2}" rpy="0.0 0.0 0.0" />
-      <geometry>
-        <cylinder radius="${leg_radius}" length="${table_height}" />
-      </geometry>
-    </collision>
-  </link>
-  <joint name="vbar2_joint" type="fixed" >
-    <parent link="leg2_link" />
-    <origin xyz="0 0 ${cage_height/2}" rpy="0 0 0" />
-    <child link="vbar2_link" />
-  </joint>
-  <link name="vbar2_link">
-    <inertial>
-      <mass value="1.0" />
-      <origin xyz="0 0 0" />
-      <inertia ixx="0.1" ixy="0"  ixz="0"
-               iyy="0.1" iyz="0"
-               izz="0.01" />
-    </inertial>
-    <visual>
-      <origin xyz="0.0 0.0 0" rpy="0 0 0" />
-      <geometry>
-        <cylinder radius="${leg_radius}" length="${cage_height}" />
-      </geometry>
-    <material name="silver_gray" />
-    </visual>
-    <collision>
-      <origin xyz="0.0 0.0 0" rpy="0.0 0.0 0.0" />
-      <geometry>
-        <cylinder radius="${leg_radius}" length="${cage_height}" />
-      </geometry>
-    </collision>
-  </link>
-  <joint name="leg3_joint" type="fixed" >
-    <parent link="table_top_link" />
-    <origin xyz="${table_x+cage_width/2} ${table_y-cage_depth/2} ${table_z+table_height}" rpy="0 0 0" />
-    <child link="leg3_link" />
-  </joint>
-  <link name="leg3_link">
-    <inertial>
-      <mass value="1.0" />
-      <origin xyz="0 0 ${-table_height/2}" />
-      <inertia ixx="0.1" ixy="0"  ixz="0"
-               iyy="0.1" iyz="0"
-               izz="0.01" />
-    </inertial>
-    <visual>
-      <origin xyz="0.0 0.0 ${-table_height/2}" rpy="0 0 0" />
-      <geometry>
-        <cylinder radius="${leg_radius}" length="${table_height}" />
-      </geometry>
-      <material name="silver_gray" />
-    </visual>
-    <collision>
-      <origin xyz="0.0 0.0 ${-table_height/2}" rpy="0.0 0.0 0.0" />
-      <geometry>
-        <cylinder radius="${leg_radius}" length="${table_height}" />
-      </geometry>
-    </collision>
-  </link>
-  <joint name="vbar3_joint" type="fixed" >
-    <parent link="leg3_link" />
-    <origin xyz="0 0 ${cage_height/2}" rpy="0 0 0" />
-    <child link="vbar3_link" />
-  </joint>
-  <link name="vbar3_link">
-    <inertial>
-      <mass value="1.0" />
-      <origin xyz="0 0 0" />
-      <inertia ixx="0.1" ixy="0"  ixz="0"
-               iyy="0.1" iyz="0"
-               izz="0.01" />
-    </inertial>
-    <visual>
-      <origin xyz="0.0 0.0 0" rpy="0 0 0" />
-      <geometry>
-        <cylinder radius="${leg_radius}" length="${cage_height}" />
-      </geometry>
-    <material name="silver_gray" />
-    </visual>
-    <collision>
-      <origin xyz="0.0 0.0 0" rpy="0.0 0.0 0.0" />
-      <geometry>
-        <cylinder radius="${leg_radius}" length="${cage_height}" />
-      </geometry>
-    </collision>
-  </link>
-  <joint name="leg4_joint" type="fixed" >
-    <parent link="table_top_link" />
-    <origin xyz="${table_x-cage_width/2} ${table_y-cage_depth/2} ${table_z+table_height}" rpy="0 0 0" />
-    <child link="leg4_link" />
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