Commit message: added option to fix urdf to optimal paramters

File: repair_urdf/urdf/repair_full.urdf.xacro (robot description, xacro)
@@ -3,7 +3,9 @@
 <xacro:include filename="$(find repair_urdf)/urdf/repair_arm.urdf.xacro"/>
 <xacro:include filename="$(find repair_urdf)/urdf/repair_cage.urdf.xacro"/>
+<xacro:include filename="$(find repair_urdf)/urdf/repair_opt_mount_params.urdf.xacro"/>
 <xacro:arg name="is_sliding_wrist" default="false" />
 <xacro:arg name="show_softhand" default="false" />
 <xacro:arg name="show_coll" default="false" />
+<xacro:arg name="load_sol" default="false" />
 <joint name="x_joint" type="prismatic">
     <origin xyz="0.0 0.0 0.0" rpy="0.0 0.0 0.0"/>
@@ -14,47 +16,91 @@
 </joint>
 <link name="dummy_link">
+    <inertial>
+      <mass value="1.0" />
+      <origin xyz="0 0 0" />
+      <inertia ixx="0.1" ixy="0"  ixz="0"
+               iyy="0.1" iyz="0"
+               izz="0.01" />
+    </inertial>
 </link>
-<joint name="z_joint" type="prismatic">
-    <origin xyz="0.0 0.0 0.0" rpy="0.0 0.0 0.0"/>
-    <parent link="dummy_link"/>
-    <child link="base_link"/>
-    <axis xyz="0 0 1"/>
-    <limit lower="${z_joint_lb}" upper= "2" effort="1000.0" velocity="20.0"/>
-</joint>
+<xacro:if value="$(arg load_sol)">
+    <joint name="z_joint" type="fixed">
+        <origin xyz="0.0 0.0 ${mount_h}" rpy="0.0 0.0 0.0"/>
+        <parent link="dummy_link"/>
+        <child link="base_link"/>
+    </joint>
+</xacro:if>
+<xacro:unless value="$(arg load_sol)">
+    <joint name="z_joint" type="prismatic">
+        <origin xyz="0.0 0.0 0.0" rpy="0.0 0.0 0.0"/>
+        <parent link="dummy_link"/>
+        <child link="base_link"/>
+        <axis xyz="0 0 1"/>
+        <limit lower="${z_joint_lb}" upper= "2" effort="1000.0" velocity="20.0"/>
+    </joint>
+</xacro:unless>
 <!-- RePAIR assembly (two arms) -->
 <link name="base_link">
 </link>
-<joint name="r_arm_mount_joint" type="prismatic">
-    <origin xyz="0.0 0.0 0.0" rpy="0 0 0"/>
-    <parent link="base_link"/>
-    <child link="dummy_r"/>
-    <axis xyz="0 -1 0"/>
-    <limit lower="${shoulder_width_lb}" upper= "${shoulder_width_ub}" effort="1000.0" velocity="20.0"/>
-</joint>
-<joint name="l_arm_mount_joint" type="prismatic">
-    <origin xyz="0.0 0.0 0.0" rpy="0 0 0"/>
-    <parent link="base_link"/>
-    <child link="dummy_l"/>
-    <axis xyz="0 1 0"/>
-    <limit lower="${shoulder_width_lb}" upper= "${shoulder_width_ub}" effort="1000.0" velocity="20.0"/>
-</joint>
+<xacro:if value="$(arg load_sol)">
+    <joint name="r_arm_mount_joint" type="fixed">
+        <origin xyz="0.0 ${-should_w} 0.0" rpy="0 0 0"/>
+        <parent link="base_link"/>
+        <child link="dummy_r"/>
+    </joint>
+    <joint name="l_arm_mount_joint" type="fixed">
+        <origin xyz="0.0 ${should_w} 0.0" rpy="0 0 0"/>
+        <parent link="base_link"/>
+        <child link="dummy_l"/>
+    </joint>
+</xacro:if>
+<xacro:unless value="$(arg load_sol)">
+    <joint name="r_arm_mount_joint" type="prismatic">
+        <origin xyz="0.0 0.0 0.0" rpy="0 0 0"/>
+        <parent link="base_link"/>
+        <child link="dummy_r"/>
+        <axis xyz="0 -1 0"/>
+        <limit lower="${shoulder_width_lb}" upper= "${shoulder_width_ub}" effort="1000.0" velocity="20.0"/>
+    </joint>
+    <joint name="l_arm_mount_joint" type="prismatic">
+        <origin xyz="0.0 0.0 0.0" rpy="0 0 0"/>
+        <parent link="base_link"/>
+        <child link="dummy_l"/>
+        <axis xyz="0 1 0"/>
+        <limit lower="${shoulder_width_lb}" upper= "${shoulder_width_ub}" effort="1000.0" velocity="20.0"/>
+    </joint>
+</xacro:unless>
 <link name="dummy_r">
 </link>
 <link name="dummy_l">
 </link>
-<joint name="roll_r" type="revolute">
-    <origin xyz="0.0 0.0 0.0" rpy="0.0 0.0 0.0"/>
-    <parent link="dummy_r"/>
-    <child link="r_arm_mount_frame"/>
-    <axis xyz="1 0 0"/>
-    <limit lower="${shoulder_roll_lb}" upper="${shoulder_roll_ub}" effort="0.0" velocity="0.0"/>
-</joint>
-<joint name="roll_l" type="revolute">
-    <origin xyz="0.0 0.0 0.0" rpy="0.0 0.0 0.0"/>
-    <parent link="dummy_l"/>
-    <child link="l_arm_mount_frame"/>
-    <axis xyz="-1 0 0"/>
-    <limit lower="${shoulder_roll_lb}" upper="${shoulder_roll_ub}" effort="0.0" velocity="0.0"/>
-</joint>
+<xacro:if value="$(arg load_sol)">
+    <joint name="roll_r" type="fixed">
+        <origin xyz="0 0.0 0.0" rpy="${roll_mount} 0.0 0.0"/>
+        <parent link="dummy_r"/>
+        <child link="r_arm_mount_frame"/>
+    </joint>
+    <joint name="roll_l" type="fixed">
+        <origin xyz="0 0.0 0.0" rpy="${-roll_mount} 0.0 0.0"/>
+        <parent link="dummy_l"/>
+        <child link="l_arm_mount_frame"/>
+    </joint>
+</xacro:if>
+<xacro:unless value="$(arg load_sol)">
+    <joint name="roll_r" type="revolute">
+        <origin xyz="0.0 0.0 0.0" rpy="0.0 0.0 0.0"/>
+        <parent link="dummy_r"/>
+        <child link="r_arm_mount_frame"/>
+        <axis xyz="1 0 0"/>
+        <limit lower="${shoulder_roll_lb}" upper="${shoulder_roll_ub}" effort="0.0" velocity="0.0"/>
+    </joint>
+    <joint name="roll_l" type="revolute">
+        <origin xyz="0.0 0.0 0.0" rpy="0.0 0.0 0.0"/>
+        <parent link="dummy_l"/>
+        <child link="l_arm_mount_frame"/>
+        <axis xyz="-1 0 0"/>
+        <limit lower="${shoulder_roll_lb}" upper="${shoulder_roll_ub}" effort="0.0" velocity="0.0"/>
+    </joint>
+</xacro:unless>
 <link name="r_arm_mount_frame">
 </link>
@@ -62,6 +108,6 @@
 </link>
 <xacro:repair_arm base_link="r_arm_mount_frame" id="1" is_sliding_wrist="$(arg is_sliding_wrist)"
-show_softhand="$(arg show_softhand)" show_coll="$(arg show_coll)"/>
+show_softhand="$(arg show_softhand)" show_coll="$(arg show_coll)" load_sol="$(arg load_sol)"/>
 <xacro:repair_arm base_link="l_arm_mount_frame" id="2" is_sliding_wrist="$(arg is_sliding_wrist)"
-show_softhand="$(arg show_softhand)" show_coll="$(arg show_coll)"/>
+show_softhand="$(arg show_softhand)" show_coll="$(arg show_coll)" load_sol="$(arg load_sol)"/>
 </robot>

Commit message: huge improvs (plots, hand mesh, data storage )

File: repair_urdf/urdf/repair_arm.urdf.xacro (robot description, xacro)
@@ -277,7 +277,14 @@
         <visual name="arm_${id}_tcp_visual">
             <origin xyz="0 0 ${object_size}" rpy="0 0 0"/>
-            <geometry>
-                <mesh filename="package://repair_urdf/meshes/link_7_sh.stl" scale="${mmTom} ${mmTom} ${mmTom}"/>
-            </geometry>
+            <xacro:if value="${id == 1}">
+                <geometry>
+                    <mesh filename="package://repair_urdf/meshes/link_7_sh.stl" scale="${mmTom} ${mmTom} ${mmTom}"/>
+                </geometry>
+            </xacro:if>
+            <xacro:unless value="${id == 1}">
+                <geometry>
+                    <mesh filename="package://repair_urdf/meshes/link_7_rh.stl" scale="${mmTom} ${mmTom} ${mmTom}"/>
+                </geometry>>
+            </xacro:unless>
             <material name="dark"/>
         </visual>
