Commit message: updated urdf with new meshes

File: repair_urdf/urdf/repair_arm.urdf.xacro (robot description, xacro)
@@ -9,5 +9,5 @@
 <xacro:if value="${show_coll == True}">
     <xacro:include filename="$(find repair_urdf)/urdf/repair_arm_coll.urdf.xacro"/>
-    <xacro:repair_coll load_sol="${load_sol}"/>
+    <xacro:repair_arm_coll load_sol="${load_sol}"/>
 </xacro:if>
 <!-- id: 1 for right arm, everything else is considered left arm -->
@@ -37,5 +37,10 @@
         <collision name="arm_${id}_link_1_collision">
             <geometry>
-                <mesh filename="package://repair_urdf/meshes/link_1.stl" scale="${mmTom} ${mmTom} ${mmTom}"/>
+                <xacro:if value="$(arg load_sol)">
+                    <mesh filename="package://repair_urdf/meshes/optimized/link_1.stl" scale="${mmTom} ${mmTom} ${mmTom}"/>
+                </xacro:if>
+                <xacro:unless value="$(arg load_sol)">
+                    <mesh filename="package://repair_urdf/meshes/base_meshes/link_1.stl" scale="${mmTom} ${mmTom} ${mmTom}"/>
+                </xacro:unless>
             </geometry>
             <material name="dark"/>
@@ -43,5 +48,10 @@
         <visual name="arm_${id}_link_1_visual">
             <geometry>
-                <mesh filename="package://repair_urdf/meshes/link_1.stl" scale="${mmTom} ${mmTom} ${mmTom}"/>
+                <xacro:if value="$(arg load_sol)">
+                    <mesh filename="package://repair_urdf/meshes/optimized/link_1.stl" scale="${mmTom} ${mmTom} ${mmTom}"/>
+                </xacro:if>
+                <xacro:unless value="$(arg load_sol)">
+                    <mesh filename="package://repair_urdf/meshes/base_meshes/link_1.stl" scale="${mmTom} ${mmTom} ${mmTom}"/>
+                </xacro:unless>
             </geometry>
             <material name="dark"/>
@@ -51,5 +61,10 @@
         <collision name="arm_${id}_link_1_collision">
             <geometry>
-                <mesh filename="package://repair_urdf/meshes/link_1_mirror.stl" scale="${mmTom} ${mmTom} ${mmTom}"/>
+                <xacro:if value="$(arg load_sol)">
+                    <mesh filename="package://repair_urdf/meshes/optimized/link_1_mirror.stl" scale="${mmTom} ${mmTom} ${mmTom}"/>
+                </xacro:if>
+                <xacro:unless value="$(arg load_sol)">
+                    <mesh filename="package://repair_urdf/meshes/base_meshes/link_1_mirror.stl" scale="${mmTom} ${mmTom} ${mmTom}"/>
+                </xacro:unless>
             </geometry>
             <material name="dark"/>
@@ -57,5 +72,10 @@
         <visual name="arm_${id}_link_1_visual">
             <geometry>
-                <mesh filename="package://repair_urdf/meshes/link_1_mirror.stl" scale="${mmTom} ${mmTom} ${mmTom}"/>
+                <xacro:if value="$(arg load_sol)">
+                    <mesh filename="package://repair_urdf/meshes/optimized/link_1_mirror.stl" scale="${mmTom} ${mmTom} ${mmTom}"/>
+                </xacro:if>
+                <xacro:unless value="$(arg load_sol)">
+                    <mesh filename="package://repair_urdf/meshes/base_meshes/link_1_mirror.stl" scale="${mmTom} ${mmTom} ${mmTom}"/>
+                </xacro:unless>
             </geometry>
             <material name="dark"/>
@@ -83,5 +103,10 @@
     <collision name="arm_${id}_link_2_collision">
         <geometry>
-            <mesh filename="package://repair_urdf/meshes/link_2.stl" scale="${mmTom} ${mmTom} ${mmTom}"/>
+            <xacro:if value="$(arg load_sol)">
+                <mesh filename="package://repair_urdf/meshes/optimized/link_2.stl" scale="${mmTom} ${mmTom} ${mmTom}"/>
+            </xacro:if>
+            <xacro:unless value="$(arg load_sol)">
+                <mesh filename="package://repair_urdf/meshes/base_meshes/link_2.stl" scale="${mmTom} ${mmTom} ${mmTom}"/>
+            </xacro:unless>
         </geometry>
         <material name="dark"/>
@@ -89,5 +114,10 @@
     <visual name="arm_${id}_link_2_visual">
         <geometry>
-            <mesh filename="package://repair_urdf/meshes/link_2.stl" scale="${mmTom} ${mmTom} ${mmTom}"/>
+            <xacro:if value="$(arg load_sol)">
+                <mesh filename="package://repair_urdf/meshes/optimized/link_2.stl" scale="${mmTom} ${mmTom} ${mmTom}"/>
+            </xacro:if>
+            <xacro:unless value="$(arg load_sol)">
+                <mesh filename="package://repair_urdf/meshes/base_meshes/link_2.stl" scale="${mmTom} ${mmTom} ${mmTom}"/>
+            </xacro:unless>
         </geometry>
         <material name="dark"/>
@@ -114,5 +144,10 @@
     <collision name="arm_${id}_link_3_collision">
         <geometry>
-            <mesh filename="package://repair_urdf/meshes/link_3.stl" scale="${mmTom} ${mmTom} ${mmTom}"/>
+            <xacro:if value="$(arg load_sol)">
+                <mesh filename="package://repair_urdf/meshes/optimized/link_3.stl" scale="${mmTom} ${mmTom} ${mmTom}"/>
+            </xacro:if>
+            <xacro:unless value="$(arg load_sol)">
+                <mesh filename="package://repair_urdf/meshes/base_meshes/link_3.stl" scale="${mmTom} ${mmTom} ${mmTom}"/>
+            </xacro:unless>
         </geometry>
         <material name="dark"/>
@@ -120,5 +155,10 @@
     <visual name="arm_${id}_link_3_visual">
         <geometry>
-            <mesh filename="package://repair_urdf/meshes/link_3.stl" scale="${mmTom} ${mmTom} ${mmTom}"/>
+            <xacro:if value="$(arg load_sol)">
+                <mesh filename="package://repair_urdf/meshes/optimized/link_3.stl" scale="${mmTom} ${mmTom} ${mmTom}"/>
+            </xacro:if>
+            <xacro:unless value="$(arg load_sol)">
+                <mesh filename="package://repair_urdf/meshes/base_meshes/link_3.stl" scale="${mmTom} ${mmTom} ${mmTom}"/>
+            </xacro:unless>
         </geometry>
         <material name="dark"/>
@@ -140,5 +180,10 @@
     <collision name="arm_${id}_link_4_collision">
         <geometry>
-            <mesh filename="package://repair_urdf/meshes/link_4.stl" scale="${mmTom} ${mmTom} ${mmTom}"/>
+            <xacro:if value="$(arg load_sol)">
+                <mesh filename="package://repair_urdf/meshes/optimized/link_4.stl" scale="${mmTom} ${mmTom} ${mmTom}"/>
+            </xacro:if>
+            <xacro:unless value="$(arg load_sol)">
+                <mesh filename="package://repair_urdf/meshes/base_meshes/link_4.stl" scale="${mmTom} ${mmTom} ${mmTom}"/>
+            </xacro:unless>
         </geometry>
         <material name="dark"/>
@@ -146,5 +191,10 @@
     <visual name="arm_${id}_link_4_visual">
         <geometry>
-            <mesh filename="package://repair_urdf/meshes/link_4.stl" scale="${mmTom} ${mmTom} ${mmTom}"/>
+            <xacro:if value="$(arg load_sol)">
+                <mesh filename="package://repair_urdf/meshes/optimized/link_4.stl" scale="${mmTom} ${mmTom} ${mmTom}"/>
+            </xacro:if>
+            <xacro:unless value="$(arg load_sol)">
+                <mesh filename="package://repair_urdf/meshes/base_meshes/link_4.stl" scale="${mmTom} ${mmTom} ${mmTom}"/>
+            </xacro:unless>
         </geometry>
         <material name="dark"/>
@@ -166,5 +216,10 @@
     <collision name="arm_${id}_link_5_collision">
         <geometry>
-            <mesh filename="package://repair_urdf/meshes/link_5.stl" scale="${mmTom} ${mmTom} ${mmTom}"/>
+            <xacro:if value="$(arg load_sol)">
+                <mesh filename="package://repair_urdf/meshes/optimized/link_5.stl" scale="${mmTom} ${mmTom} ${mmTom}"/>
+            </xacro:if>
+            <xacro:unless value="$(arg load_sol)">
+                <mesh filename="package://repair_urdf/meshes/base_meshes/link_5.stl" scale="${mmTom} ${mmTom} ${mmTom}"/>
+            </xacro:unless>
         </geometry>
         <material name="dark"/>
@@ -172,5 +227,10 @@
     <visual name="arm_${id}_link_5_visual">
         <geometry>
-            <mesh filename="package://repair_urdf/meshes/link_5.stl" scale="${mmTom} ${mmTom} ${mmTom}"/>
+            <xacro:if value="$(arg load_sol)">
+                <mesh filename="package://repair_urdf/meshes/optimized/link_5.stl" scale="${mmTom} ${mmTom} ${mmTom}"/>
+            </xacro:if>
+            <xacro:unless value="$(arg load_sol)">
+                <mesh filename="package://repair_urdf/meshes/base_meshes/link_5.stl" scale="${mmTom} ${mmTom} ${mmTom}"/>
+            </xacro:unless>
         </geometry>
         <material name="dark"/>
@@ -221,5 +281,10 @@
     <collision name="arm_${id}_link_6_collision">
         <geometry>
-            <mesh filename="package://repair_urdf/meshes/link_6.stl" scale="${mmTom} ${mmTom} ${mmTom}"/>
+            <xacro:if value="$(arg load_sol)">
+                <mesh filename="package://repair_urdf/meshes/optimized/link_6.stl" scale="${mmTom} ${mmTom} ${mmTom}"/>
+            </xacro:if>
+            <xacro:unless value="$(arg load_sol)">
+                <mesh filename="package://repair_urdf/meshes/base_meshes/link_6.stl" scale="${mmTom} ${mmTom} ${mmTom}"/>
+            </xacro:unless>
         </geometry>
         <material name="dark"/>
@@ -227,5 +292,10 @@
     <visual name="arm_${id}_link_6_visual">
         <geometry>
-            <mesh filename="package://repair_urdf/meshes/link_6.stl" scale="${mmTom} ${mmTom} ${mmTom}"/>
+            <xacro:if value="$(arg load_sol)">
+                <mesh filename="package://repair_urdf/meshes/optimized/link_6.stl" scale="${mmTom} ${mmTom} ${mmTom}"/>
+            </xacro:if>
+            <xacro:unless value="$(arg load_sol)">
+                <mesh filename="package://repair_urdf/meshes/base_meshes/link_6.stl" scale="${mmTom} ${mmTom} ${mmTom}"/>
+            </xacro:unless>
         </geometry>
         <material name="dark"/>
@@ -253,5 +323,10 @@
     <collision name="arm_${id}_link_7_collision">
         <geometry>
-            <mesh filename="package://repair_urdf/meshes/link_7.stl" scale="${mmTom} ${mmTom} ${mmTom}"/>
+            <xacro:if value="$(arg load_sol)">
+                <mesh filename="package://repair_urdf/meshes/optimized/link_7_sh.stl" scale="${mmTom} ${mmTom} ${mmTom}"/>
+            </xacro:if>
+            <xacro:unless value="$(arg load_sol)">
+                <mesh filename="package://repair_urdf/meshes/base_meshes/link_7.stl" scale="${mmTom} ${mmTom} ${mmTom}"/>
+            </xacro:unless>
         </geometry>
         <material name="dark"/>
@@ -261,5 +336,10 @@
                 <origin xyz="0 0 0" rpy="0 0 0"/>
                 <geometry>
-                    <mesh filename="package://repair_urdf/meshes/link_7.stl" scale="${mmTom} ${mmTom} ${mmTom}"/>
+                    <xacro:if value="$(arg load_sol)">
+                        <mesh filename="package://repair_urdf/meshes/optimized/link_7_rh.stl" scale="${mmTom} ${mmTom} ${mmTom}"/>
+                    </xacro:if>
+                    <xacro:unless value="$(arg load_sol)">
+                        <mesh filename="package://repair_urdf/meshes/base_meshes/link_7.stl" scale="${mmTom} ${mmTom} ${mmTom}"/>
+                    </xacro:unless>
                 </geometry>
                 <material name="dark"/>
@@ -275,18 +355,20 @@
     </joint>
     <link name="arm_${id}_tcp">
-        <visual name="arm_${id}_tcp_visual">
-            <origin xyz="0 0 ${object_size}" rpy="0 0 0"/>
-            <xacro:if value="${id == 1}">
-                <geometry>
-                    <mesh filename="package://repair_urdf/meshes/link_7_sh.stl" scale="${mmTom} ${mmTom} ${mmTom}"/>
-                </geometry>
-            </xacro:if>
-            <xacro:unless value="${id == 1}">
-                <geometry>
-                    <mesh filename="package://repair_urdf/meshes/link_7_rh.stl" scale="${mmTom} ${mmTom} ${mmTom}"/>
-                </geometry>>
-            </xacro:unless>
-            <material name="dark"/>
-        </visual>
+        <xacro:unless value="$(arg load_sol)">
+            <visual name="arm_${id}_tcp_visual">
+                <origin xyz="0 0 ${object_size}" rpy="0 0 0"/>
+                <xacro:if value="${id == 1}">
+                    <geometry>
+                        <mesh filename="package://repair_urdf/meshes/base_meshes/link_7_sh.stl" scale="${mmTom} ${mmTom} ${mmTom}"/>
+                    </geometry>
+                </xacro:if>
+                <xacro:unless value="${id == 1}">
+                        <geometry>
+                            <mesh filename="package://repair_urdf/meshes/base_meshes/link_7_rh.stl" scale="${mmTom} ${mmTom} ${mmTom}"/>
+                        </geometry>
+                </xacro:unless>
+                <material name="dark"/>
+            </visual>
+        </xacro:unless>
     </link>
 </xacro:if>

File: repair_urdf/urdf/repair_arm_coll.urdf.xacro (robot description, xacro)
@@ -1,5 +1,5 @@
 <?xml version="1.0"?>
 <robot xmlns:xacro="http://www.ros.org/wiki/xacro">
-<xacro:macro name="repair_coll" params="load_sol" />
+<xacro:macro name="repair_arm_coll" params="load_sol" />
 <joint name="arm_${id}_link_1_coll_joint" type="fixed">
     <origin xyz="${link1_coll_offset_x} ${link1_coll_offset_y} ${link1_coll_offset_z}" rpy="0 0 0"/>

File: repair_urdf/urdf/repair_full.urdf (robot description, URDF)
Before this commit: robot repair_full, 39 links, 38 joints
Links:
- link arm_1_link_1: geometry collision mesh filename=package://repair_urdf/meshes/optimized/link_1.stl scale=0.001 0.001 0.001; visual mesh filename=package://repair_urdf/meshes/optimized/link_1.stl scale=0.001 0.001 0.001
- link arm_1_link_2: geometry collision mesh filename=package://repair_urdf/meshes/optimized/link_2.stl scale=0.001 0.001 0.001; visual mesh filename=package://repair_urdf/meshes/optimized/link_2.stl scale=0.001 0.001 0.001
- link arm_1_link_3: geometry collision mesh filename=package://repair_urdf/meshes/optimized/link_3.stl scale=0.001 0.001 0.001; visual mesh filename=package://repair_urdf/meshes/optimized/link_3.stl scale=0.001 0.001 0.001
- link arm_1_link_4: geometry collision mesh filename=package://repair_urdf/meshes/optimized/link_4.stl scale=0.001 0.001 0.001; visual mesh filename=package://repair_urdf/meshes/optimized/link_4.stl scale=0.001 0.001 0.001
- link arm_1_link_5: geometry collision mesh filename=package://repair_urdf/meshes/optimized/link_5.stl scale=0.001 0.001 0.001; visual mesh filename=package://repair_urdf/meshes/optimized/link_5.stl scale=0.001 0.001 0.001
- link arm_1_link_6: geometry collision mesh filename=package://repair_urdf/meshes/optimized/link_6.stl scale=0.001 0.001 0.001; visual mesh filename=package://repair_urdf/meshes/optimized/link_6.stl scale=0.001 0.001 0.001
- link arm_1_link_7: geometry collision mesh filename=package://repair_urdf/meshes/optimized/link_7_sh.stl scale=0.001 0.001 0.001
- link arm_2_link_1: geometry collision mesh filename=package://repair_urdf/meshes/optimized/link_1_mirror.stl scale=0.001 0.001 0.001; visual mesh filename=package://repair_urdf/meshes/optimized/link_1_mirror.stl scale=0.001 0.001 0.001
- link arm_2_link_2: geometry collision mesh filename=package://repair_urdf/meshes/optimized/link_2.stl scale=0.001 0.001 0.001; visual mesh filename=package://repair_urdf/meshes/optimized/link_2.stl scale=0.001 0.001 0.001
- link arm_2_link_3: geometry collision mesh filename=package://repair_urdf/meshes/optimized/link_3.stl scale=0.001 0.001 0.001; visual mesh filename=package://repair_urdf/meshes/optimized/link_3.stl scale=0.001 0.001 0.001
- link arm_2_link_4: geometry collision mesh filename=package://repair_urdf/meshes/optimized/link_4.stl scale=0.001 0.001 0.001; visual mesh filename=package://repair_urdf/meshes/optimized/link_4.stl scale=0.001 0.001 0.001
- link arm_2_link_5: geometry collision mesh filename=package://repair_urdf/meshes/optimized/link_5.stl scale=0.001 0.001 0.001; visual mesh filename=package://repair_urdf/meshes/optimized/link_5.stl scale=0.001 0.001 0.001
- link arm_2_link_6: geometry collision mesh filename=package://repair_urdf/meshes/optimized/link_6.stl scale=0.001 0.001 0.001; visual mesh filename=package://repair_urdf/meshes/optimized/link_6.stl scale=0.001 0.001 0.001
- link arm_2_link_7: geometry collision mesh filename=package://repair_urdf/meshes/optimized/link_7_sh.stl scale=0.001 0.001 0.001
Joints:
- joint arm_1_tcp_joint: origin xyz=0 0 0 rpy=0 0 0 -> xyz=0 -0.014142135623730949 0.02414213562373095 rpy=0 -2.3561944901874483 -1.57079632679
- joint arm_2_tcp_joint: origin xyz=0 0 0 rpy=0 0 0 -> xyz=0 -0.014142135623730949 0.02414213562373095 rpy=0 -2.3561944901874483 -1.57079632679

File: repair_urdf/urdf/repair_full.urdf.xacro (robot description, xacro)
@@ -14,4 +14,9 @@
 <xacro:if value="$(arg xbot)">
     <xacro:include filename="$(find repair_urdf)/urdf/xbot2.gazebo.xacro"/>
+</xacro:if>
+<xacro:if value="$(arg show_coll)">
+    <xacro:include filename="$(find repair_urdf)/urdf/repair_torso_coll_params.urdf.xacro"/>
+    <xacro:include filename="$(find repair_urdf)/urdf/repair_torso_coll.urdf.xacro"/>
+    <xacro:repair_torso_coll />
 </xacro:if>
 <xacro:if value="$(arg load_sol)">
@@ -32,4 +37,33 @@
                   izz="0" />
         </inertial>
+        <xacro:if value="$(arg show_coll)">
+            <visual name="link0_coll_visual1">
+                <origin xyz="0 0 0" rpy="0 0 0"/>
+                <geometry>
+                    <sphere radius="${coll_radius_link1}"/>
+                </geometry>
+                <material name="darkred"/>
+            </visual>
+            <visual name="link0_coll_visual2">
+                <origin xyz="0 ${link2_coll_offset_y} 0" rpy="0 0 0"/>
+                <geometry>
+                    <sphere radius="${coll_radius_link1}"/>
+                </geometry>
+                <material name="darkred"/>
+            </visual>
+            <visual name="link0_coll_visual3">
+                <origin xyz="0 ${- link2_coll_offset_y} 0" rpy="0 0 0"/>
+                <geometry>
+                    <sphere radius="${coll_radius_link1}"/>
+                </geometry>
+                <material name="darkred"/>
+            </visual>
+        </xacro:if>
+        <visual name="base_link_visual">
+            <geometry>
+                <mesh filename="package://repair_urdf/meshes/optimized/link_0.stl" scale="${mmTom} ${mmTom} ${mmTom}"/>
+            </geometry>
+            <material name="dark"/>
+        </visual>
     </link>
     <joint name="r_arm_mount_joint" type="fixed">

Commit message: monday work

File: repair_urdf/urdf/repair_arm.urdf.xacro (robot description, xacro)
@@ -202,5 +202,5 @@
 </link>
 <joint name="arm_${id}_joint_5" type="revolute">
-    <origin xyz="${5 * mmTom} 0 0" rpy="${-PI_2} 0 ${-PI_2}"/>
+    <origin xyz="${5 * mmTom} 0 0" rpy="0 0 ${-PI_2}"/>
     <parent link="arm_${id}_link_4"/>
     <child link="arm_${id}_link_5"/>
@@ -248,5 +248,5 @@
 <xacro:unless value="${is_sliding_wrist != True}">
     <joint name="arm_${id}_joint_6" type="revolute">
-            <origin xyz="0 0 ${321.000 * mmTom}" rpy="0 ${-PI_2} 0"/>
+            <origin xyz="0 ${321.000 * mmTom} 0" rpy="${PI + PI_2} ${PI + PI_2} ${0}"/>
             <parent link="arm_${id}_link_5"/>
             <child link="dummy_sliding_wrist${id}_link"/>
@@ -322,4 +322,5 @@
     </inertial>
     <collision name="arm_${id}_link_7_collision">
+        <origin xyz="0 0 0" rpy="0 0 0"/>
         <geometry>
             <xacro:if value="$(arg load_sol)">
@@ -332,5 +333,5 @@
         <material name="dark"/>
     </collision>
-    <xacro:unless value="${show_softhand == True}">
+    <xacro:if value="${show_softhand == True}">
         <visual name="arm_${id}_link_7_visual">
                 <origin xyz="0 0 0" rpy="0 0 0"/>
@@ -345,5 +346,5 @@
                 <material name="dark"/>
         </visual>
-    </xacro:unless>
+    </xacro:if>
 </link>
 <xacro:if value="${show_softhand == True}">

Commit message: update

File: repair_urdf/urdf/repair_arm.urdf.xacro (robot description, xacro)
@@ -239,5 +239,5 @@
 <xacro:if value="${is_sliding_wrist != True}">
     <joint name="arm_${id}_joint_6" type="revolute">
-        <origin xyz="0 0 ${321.000 * mmTom}" rpy="0 ${-PI_2} 0"/>
+        <origin xyz="${96.000 * mmTom} ${321.000 * mmTom} 0" rpy="0 ${-PI_2} 0"/>
         <parent link="arm_${id}_link_5"/>
         <child link="arm_${id}_link_6"/>
@@ -248,5 +248,5 @@
 <xacro:unless value="${is_sliding_wrist != True}">
     <joint name="arm_${id}_joint_6" type="revolute">
-            <origin xyz="0 ${321.000 * mmTom} 0" rpy="${PI + PI_2} ${PI + PI_2} ${0}"/>
+            <origin xyz="${96.000 * mmTom} ${321.000 * mmTom} 0" rpy="${PI} ${0} ${PI_2}"/>
             <parent link="arm_${id}_link_5"/>
             <child link="dummy_sliding_wrist${id}_link"/>
