Commit message: too many things, no time to commit properly

File: repair_urdf/urdf/repair_arm.urdf.xacro (robot description, xacro)
@@ -6,6 +6,6 @@
 <xacro:property name="sm_tau_max" value="200.0" />
 <xacro:include filename="$(find repair_urdf)/urdf/repair_arm_coll_params.urdf.xacro"/>
-<xacro:macro name="repair_arm" params="id base_link is_sliding_wrist show_softhand show_coll load_sol" >
-<xacro:if value="${show_coll == True}">
+<xacro:macro name="repair_arm" params="id base_link is_sliding_wrist gen_coll load_sol use_updated_wrist" >
+<xacro:if value="${gen_coll == True}">
     <xacro:include filename="$(find repair_urdf)/urdf/repair_arm_coll.urdf.xacro"/>
     <xacro:repair_arm_coll load_sol="${load_sol}"/>
@@ -15,5 +15,4 @@
 <!-- is_sliding_wrist: whether to add a sliding joint along the axis of wrist's second d.o.f.
     (true -> yes), everything else -> no -->
-    <!-- show_softhand: whether to use softhand or not at the TCP -->
 <joint name="arm_${id}_joint_1" type="revolute">
     <xacro:if value="${id == 1}">
@@ -37,8 +36,8 @@
         <collision name="arm_${id}_link_1_collision">
             <geometry>
-                <xacro:if value="$(arg load_sol)">
+                <xacro:if value="$(arg use_updated_wrist)">
                     <mesh filename="package://repair_urdf/meshes/optimized/link_1.stl" scale="${mmTom} ${mmTom} ${mmTom}"/>
                 </xacro:if>
-                <xacro:unless value="$(arg load_sol)">
+                <xacro:unless value="$(arg use_updated_wrist)">
                     <mesh filename="package://repair_urdf/meshes/base_meshes/link_1.stl" scale="${mmTom} ${mmTom} ${mmTom}"/>
                 </xacro:unless>
@@ -48,8 +47,8 @@
         <visual name="arm_${id}_link_1_visual">
             <geometry>
-                <xacro:if value="$(arg load_sol)">
+                <xacro:if value="$(arg use_updated_wrist)">
                     <mesh filename="package://repair_urdf/meshes/optimized/link_1.stl" scale="${mmTom} ${mmTom} ${mmTom}"/>
                 </xacro:if>
-                <xacro:unless value="$(arg load_sol)">
+                <xacro:unless value="$(arg use_updated_wrist)">
                     <mesh filename="package://repair_urdf/meshes/base_meshes/link_1.stl" scale="${mmTom} ${mmTom} ${mmTom}"/>
                 </xacro:unless>
@@ -61,8 +60,8 @@
         <collision name="arm_${id}_link_1_collision">
             <geometry>
-                <xacro:if value="$(arg load_sol)">
+                <xacro:if value="$(arg use_updated_wrist)">
                     <mesh filename="package://repair_urdf/meshes/optimized/link_1_mirror.stl" scale="${mmTom} ${mmTom} ${mmTom}"/>
                 </xacro:if>
-                <xacro:unless value="$(arg load_sol)">
+                <xacro:unless value="$(arg use_updated_wrist)">
                     <mesh filename="package://repair_urdf/meshes/base_meshes/link_1_mirror.stl" scale="${mmTom} ${mmTom} ${mmTom}"/>
                 </xacro:unless>
@@ -72,8 +71,8 @@
         <visual name="arm_${id}_link_1_visual">
             <geometry>
-                <xacro:if value="$(arg load_sol)">
+                <xacro:if value="$(arg use_updated_wrist)">
                     <mesh filename="package://repair_urdf/meshes/optimized/link_1_mirror.stl" scale="${mmTom} ${mmTom} ${mmTom}"/>
                 </xacro:if>
-                <xacro:unless value="$(arg load_sol)">
+                <xacro:unless value="$(arg use_updated_wrist)">
                     <mesh filename="package://repair_urdf/meshes/base_meshes/link_1_mirror.stl" scale="${mmTom} ${mmTom} ${mmTom}"/>
                 </xacro:unless>
@@ -103,8 +102,8 @@
     <collision name="arm_${id}_link_2_collision">
         <geometry>
-            <xacro:if value="$(arg load_sol)">
+            <xacro:if value="$(arg use_updated_wrist)">
                 <mesh filename="package://repair_urdf/meshes/optimized/link_2.stl" scale="${mmTom} ${mmTom} ${mmTom}"/>
             </xacro:if>
-            <xacro:unless value="$(arg load_sol)">
+            <xacro:unless value="$(arg use_updated_wrist)">
                 <mesh filename="package://repair_urdf/meshes/base_meshes/link_2.stl" scale="${mmTom} ${mmTom} ${mmTom}"/>
             </xacro:unless>
@@ -114,8 +113,8 @@
     <visual name="arm_${id}_link_2_visual">
         <geometry>
-            <xacro:if value="$(arg load_sol)">
+            <xacro:if value="$(arg use_updated_wrist)">
                 <mesh filename="package://repair_urdf/meshes/optimized/link_2.stl" scale="${mmTom} ${mmTom} ${mmTom}"/>
             </xacro:if>
-            <xacro:unless value="$(arg load_sol)">
+            <xacro:unless value="$(arg use_updated_wrist)">
                 <mesh filename="package://repair_urdf/meshes/base_meshes/link_2.stl" scale="${mmTom} ${mmTom} ${mmTom}"/>
             </xacro:unless>
@@ -144,8 +143,8 @@
     <collision name="arm_${id}_link_3_collision">
         <geometry>
-            <xacro:if value="$(arg load_sol)">
+            <xacro:if value="$(arg use_updated_wrist)">
                 <mesh filename="package://repair_urdf/meshes/optimized/link_3.stl" scale="${mmTom} ${mmTom} ${mmTom}"/>
             </xacro:if>
-            <xacro:unless value="$(arg load_sol)">
+            <xacro:unless value="$(arg use_updated_wrist)">
                 <mesh filename="package://repair_urdf/meshes/base_meshes/link_3.stl" scale="${mmTom} ${mmTom} ${mmTom}"/>
             </xacro:unless>
@@ -155,8 +154,8 @@
     <visual name="arm_${id}_link_3_visual">
         <geometry>
-            <xacro:if value="$(arg load_sol)">
+            <xacro:if value="$(arg use_updated_wrist)">
                 <mesh filename="package://repair_urdf/meshes/optimized/link_3.stl" scale="${mmTom} ${mmTom} ${mmTom}"/>
             </xacro:if>
-            <xacro:unless value="$(arg load_sol)">
+            <xacro:unless value="$(arg use_updated_wrist)">
                 <mesh filename="package://repair_urdf/meshes/base_meshes/link_3.stl" scale="${mmTom} ${mmTom} ${mmTom}"/>
             </xacro:unless>
@@ -180,8 +179,8 @@
     <collision name="arm_${id}_link_4_collision">
         <geometry>
-            <xacro:if value="$(arg load_sol)">
+            <xacro:if value="$(arg use_updated_wrist)">
                 <mesh filename="package://repair_urdf/meshes/optimized/link_4.stl" scale="${mmTom} ${mmTom} ${mmTom}"/>
             </xacro:if>
-            <xacro:unless value="$(arg load_sol)">
+            <xacro:unless value="$(arg use_updated_wrist)">
                 <mesh filename="package://repair_urdf/meshes/base_meshes/link_4.stl" scale="${mmTom} ${mmTom} ${mmTom}"/>
             </xacro:unless>
@@ -191,8 +190,8 @@
     <visual name="arm_${id}_link_4_visual">
         <geometry>
-            <xacro:if value="$(arg load_sol)">
+            <xacro:if value="$(arg use_updated_wrist)">
                 <mesh filename="package://repair_urdf/meshes/optimized/link_4.stl" scale="${mmTom} ${mmTom} ${mmTom}"/>
             </xacro:if>
-            <xacro:unless value="$(arg load_sol)">
+            <xacro:unless value="$(arg use_updated_wrist)">
                 <mesh filename="package://repair_urdf/meshes/base_meshes/link_4.stl" scale="${mmTom} ${mmTom} ${mmTom}"/>
             </xacro:unless>
@@ -202,5 +201,5 @@
 </link>
 <joint name="arm_${id}_joint_5" type="revolute">
-    <origin xyz="${5 * mmTom} 0 0" rpy="0 0 ${-PI_2}"/>
+    <origin xyz="${5 * mmTom} 0 0" rpy="${-PI_2} ${0} ${-PI_2}"/>
     <parent link="arm_${id}_link_4"/>
     <child link="arm_${id}_link_5"/>
@@ -215,41 +214,40 @@
     </inertial>
     <collision name="arm_${id}_link_5_collision">
-        <geometry>
-            <xacro:if value="$(arg load_sol)">
+        <xacro:if value="$(arg use_updated_wrist)">
+            <origin xyz="0 0 0" rpy="${PI_2} ${0} ${0}"/>
+            <geometry>
                 <mesh filename="package://repair_urdf/meshes/optimized/link_5.stl" scale="${mmTom} ${mmTom} ${mmTom}"/>
-            </xacro:if>
-            <xacro:unless value="$(arg load_sol)">
+            </geometry>
+        </xacro:if>
+        <xacro:unless value="$(arg use_updated_wrist)">
+            <origin xyz="0 0 0" rpy="${0} ${0} ${0}"/>
+            <geometry>
                 <mesh filename="package://repair_urdf/meshes/base_meshes/link_5.stl" scale="${mmTom} ${mmTom} ${mmTom}"/>
-            </xacro:unless>
-        </geometry>
+            </geometry>
+        </xacro:unless>
         <material name="dark"/>
     </collision>
     <visual name="arm_${id}_link_5_visual">
-        <geometry>
-            <xacro:if value="$(arg load_sol)">
+        <xacro:if value="$(arg use_updated_wrist)">
+            <origin xyz="0 0 0" rpy="${PI_2} ${0} ${0}"/>
+            <geometry>
                 <mesh filename="package://repair_urdf/meshes/optimized/link_5.stl" scale="${mmTom} ${mmTom} ${mmTom}"/>
-            </xacro:if>
-            <xacro:unless value="$(arg load_sol)">
+            </geometry>
+        </xacro:if>
+        <xacro:unless value="$(arg use_updated_wrist)">
+            <origin xyz="0 0 0" rpy="${0} ${0} ${0}"/>
+            <geometry>
                 <mesh filename="package://repair_urdf/meshes/base_meshes/link_5.stl" scale="${mmTom} ${mmTom} ${mmTom}"/>
-            </xacro:unless>
-        </geometry>
-        <material name="dark"/>
-    </visual>
-</link>
-<xacro:if value="${is_sliding_wrist != True}">
+            </geometry>
+        </xacro:unless>
+        <material name="dark"/>
+    </visual>
+</link>
+<xacro:if value="${is_sliding_wrist == True}">
     <joint name="arm_${id}_joint_6" type="revolute">
-        <origin xyz="${96.000 * mmTom} ${321.000 * mmTom} 0" rpy="0 ${-PI_2} 0"/>
-        <parent link="arm_${id}_link_5"/>
-        <child link="arm_${id}_link_6"/>
-        <axis xyz="0 0 1"/>
-        <limit lower="${-150.0 * DEG2RAD}" upper="${150.0 * DEG2RAD}" effort="${big_tau_max}" velocity="10.0"/>
-    </joint>
-</xacro:if>
-<xacro:unless value="${is_sliding_wrist != True}">
-    <joint name="arm_${id}_joint_6" type="revolute">
-            <origin xyz="${96.000 * mmTom} ${321.000 * mmTom} 0" rpy="${PI} ${0} ${PI_2}"/>
+            <origin xyz="0 ${0.000 * mmTom} ${321.000 * mmTom} " rpy="${0} ${-PI_2} ${0}"/>
+            <axis xyz="0 0 1"/>
             <parent link="arm_${id}_link_5"/>
             <child link="dummy_sliding_wrist${id}_link"/>
-            <axis xyz="0 0 1"/>
             <limit lower="${-150.0 * DEG2RAD}" upper="${150.0 * DEG2RAD}" effort="${big_tau_max}" velocity="10.0"/>
     </joint>
@@ -272,4 +270,13 @@
         </joint>
     </xacro:unless>
+</xacro:if>
+<xacro:unless value="${is_sliding_wrist == True}">
+    <joint name="arm_${id}_joint_6" type="revolute">
+        <origin xyz="${96.000 * mmTom} ${321.000 * mmTom} 0" rpy="0 ${-PI_2} 0"/>
+        <parent link="arm_${id}_link_5"/>
+        <child link="arm_${id}_link_6"/>
+        <axis xyz="0 0 1"/>
+        <limit lower="${-150.0 * DEG2RAD}" upper="${150.0 * DEG2RAD}" effort="${big_tau_max}" velocity="10.0"/>
+    </joint>
 </xacro:unless>
 <link name="arm_${id}_link_6">
@@ -280,23 +287,31 @@
     </inertial>
     <collision name="arm_${id}_link_6_collision">
-        <geometry>
-            <xacro:if value="$(arg load_sol)">
+        <xacro:if value="$(arg use_updated_wrist)">
+            <origin xyz="0 0 0" rpy="${PI_2} ${0} ${0}"/>
+            <geometry>
                 <mesh filename="package://repair_urdf/meshes/optimized/link_6.stl" scale="${mmTom} ${mmTom} ${mmTom}"/>
-            </xacro:if>
-            <xacro:unless value="$(arg load_sol)">
+            </geometry>
+        </xacro:if>
+        <xacro:unless value="$(arg use_updated_wrist)">
+            <origin xyz="0 0 0" rpy="${0} ${0} ${0}"/>
+            <geometry>
                 <mesh filename="package://repair_urdf/meshes/base_meshes/link_6.stl" scale="${mmTom} ${mmTom} ${mmTom}"/>
-            </xacro:unless>
-        </geometry>
+            </geometry>
+        </xacro:unless>
         <material name="dark"/>
     </collision>
     <visual name="arm_${id}_link_6_visual">
-        <geometry>
-            <xacro:if value="$(arg load_sol)">
+        <xacro:if value="$(arg use_updated_wrist)">
+            <origin xyz="0 0 0" rpy="${PI_2} ${0} ${0}"/>
+            <geometry>
                 <mesh filename="package://repair_urdf/meshes/optimized/link_6.stl" scale="${mmTom} ${mmTom} ${mmTom}"/>
-            </xacro:if>
-            <xacro:unless value="$(arg load_sol)">
+            </geometry>
+        </xacro:if>
+        <xacro:unless value="$(arg use_updated_wrist)">
+            <origin xyz="0 0 0" rpy="${0} ${0} ${0}"/>
+            <geometry>
                 <mesh filename="package://repair_urdf/meshes/base_meshes/link_6.stl" scale="${mmTom} ${mmTom} ${mmTom}"/>
-            </xacro:unless>
-        </geometry>
+            </geometry>
+        </xacro:unless>
         <material name="dark"/>
     </visual>
@@ -321,65 +336,27 @@
         <origin xyz="${0 * mmTom} ${0 * mmTom} ${0 * mmTom}"/>
     </inertial>
-    <collision name="arm_${id}_link_7_collision">
-        <origin xyz="0 0 0" rpy="0 0 0"/>
-        <geometry>
-            <xacro:if value="$(arg load_sol)">
-                <mesh filename="package://repair_urdf/meshes/optimized/link_7_sh.stl" scale="${mmTom} ${mmTom} ${mmTom}"/>
-            </xacro:if>
-            <xacro:unless value="$(arg load_sol)">
-                <mesh filename="package://repair_urdf/meshes/base_meshes/link_7.stl" scale="${mmTom} ${mmTom} ${mmTom}"/>
-            </xacro:unless>
-        </geometry>
-        <material name="dark"/>
-    </collision>
-    <xacro:if value="${show_softhand == True}">
-        <visual name="arm_${id}_link_7_visual">
-                <origin xyz="0 0 0" rpy="0 0 0"/>
+</link>
+<joint name="arm_${id}_tcp_joint" type="fixed">
+    <origin xyz="0 ${- object_size *  sin(softhand_mount_angle)} ${10.0 * mmTom + object_size *  cos(softhand_mount_angle)}"
+            rpy="0 ${-(PI_2 + softhand_mount_angle)} ${-(PI_2)}"/>
+    <parent link="arm_${id}_link_7"/>
+    <child link="arm_${id}_tcp"/>
+</joint>
+<link name="arm_${id}_tcp">
+    <visual name="arm_${id}_tcp_visual">
+        <origin xyz="0 0 ${object_size}" rpy="0 0 0"/>
+        <xacro:if value="${id == 1}">
+            <geometry>
+                <mesh filename="package://repair_urdf/meshes/link_7_sh.stl" scale="${mmTom} ${mmTom} ${mmTom}"/>
+            </geometry>
+        </xacro:if>
+        <xacro:unless value="${id == 1}">
                 <geometry>
-                    <xacro:if value="$(arg load_sol)">
-                        <mesh filename="package://repair_urdf/meshes/optimized/link_7_rh.stl" scale="${mmTom} ${mmTom} ${mmTom}"/>
-                    </xacro:if>
-                    <xacro:unless value="$(arg load_sol)">
-                        <mesh filename="package://repair_urdf/meshes/base_meshes/link_7.stl" scale="${mmTom} ${mmTom} ${mmTom}"/>
-                    </xacro:unless>
+                    <mesh filename="package://repair_urdf/meshes/link_7_rh.stl" scale="${mmTom} ${mmTom} ${mmTom}"/>
                 </geometry>
-                <material name="dark"/>
-        </visual>
-    </xacro:if>
-</link>
-<xacro:if value="${show_softhand == True}">
-    <joint name="arm_${id}_tcp_joint" type="fixed">
-        <origin xyz="0 ${- object_size *  sin(softhand_mount_angle)} ${10.0 * mmTom + object_size *  cos(softhand_mount_angle)}"
-                rpy="0 ${-(PI_2 + softhand_mount_angle)} ${-(PI_2)}"/>
-        <parent link="arm_${id}_link_7"/>
-        <child link="arm_${id}_tcp"/>
-    </joint>
-    <link name="arm_${id}_tcp">
-        <xacro:unless value="$(arg load_sol)">
-            <visual name="arm_${id}_tcp_visual">
-                <origin xyz="0 0 ${object_size}" rpy="0 0 0"/>
-                <xacro:if value="${id == 1}">
-                    <geometry>
-                        <mesh filename="package://repair_urdf/meshes/base_meshes/link_7_sh.stl" scale="${mmTom} ${mmTom} ${mmTom}"/>
-                    </geometry>
-                </xacro:if>
-                <xacro:unless value="${id == 1}">
-                        <geometry>
-                            <mesh filename="package://repair_urdf/meshes/base_meshes/link_7_rh.stl" scale="${mmTom} ${mmTom} ${mmTom}"/>
-                        </geometry>
-                </xacro:unless>
-                <material name="dark"/>
-            </visual>
-        </xacro:unless>
-    </link>
-</xacro:if>
-<xacro:unless value="${show_softhand == True}">
-    <joint name="arm_${id}_tcp_joint" type="fixed">
-        <origin xyz="0 0 0" rpy="0 0 0"/>
-        <parent link="arm_${id}_link_7"/>
-        <child link="arm_${id}_tcp"/>
-    </joint>
-    <link name="arm_${id}_tcp"/>
-</xacro:unless>
+        </xacro:unless>
+        <material name="dark"/>
+    </visual>
+</link>
 </xacro:macro>
 </robot>

File: repair_urdf/urdf/repair_arm_coll.urdf.xacro (robot description, xacro)
@@ -60,5 +60,5 @@
 <xacro:if value="${load_sol == True}">
     <joint name="arm_${id}_link_5_coll_joint" type="fixed">
-         <origin xyz="${link5_coll_offset_x + wrist_off} ${link5_coll_offset_y} ${link5_coll_offset_z}" rpy="0 0 0"/>
+        <origin xyz="${link5_coll_offset_x + wrist_off} ${link5_coll_offset_y} ${link5_coll_offset_z}" rpy="0 0 0"/>
         <parent link="arm_${id}_link_5"/>
         <child link="arm_${id}_link5_coll"/>
@@ -67,5 +67,5 @@
 <xacro:unless value="${load_sol == True}">
     <joint name="arm_${id}_link_5_coll_joint" type="prismatic">
-        <origin xyz="${link5_coll_offset_x} ${link5_coll_offset_y} ${link5_coll_offset_z}" rpy="0 0 0"/>
+        <origin xyz="${link5_coll_offset_x } ${link5_coll_offset_y} ${link5_coll_offset_z}" rpy="0 0 0"/>
         <parent link="arm_${id}_link_5"/>
         <child link="arm_${id}_link5_coll"/>
