Commit message: too many things, no time to commit properly

File: repair_urdf/urdf/repair_full.urdf (robot description, URDF)
Before this commit: robot repair_full, 39 links, 38 joints
Links:
- removed link dummy_sliding_wrist1_link
- removed link dummy_sliding_wrist2_link
- added link arm_1_link1_coll; visual sphere radius=0.07
- added link arm_1_link2_coll; visual sphere radius=0.053
- added link arm_1_link3_coll; visual sphere radius=0.08
- added link arm_1_link4_coll; visual sphere radius=0.08
- added link arm_1_link5_coll; visual sphere radius=0.05
- added link arm_1_link6_coll; visual sphere radius=0.07
- added link arm_1_link7_coll; visual sphere radius=0.05
- added link arm_2_link1_coll; visual sphere radius=0.07
- added link arm_2_link2_coll; visual sphere radius=0.053
- added link arm_2_link3_coll; visual sphere radius=0.08
- added link arm_2_link4_coll; visual sphere radius=0.08
- added link arm_2_link5_coll; visual sphere radius=0.05
- added link arm_2_link6_coll; visual sphere radius=0.07
- added link arm_2_link7_coll; visual sphere radius=0.05
- link arm_1_link_1: geometry collision mesh filename=package://repair_urdf/meshes/base_meshes/link_1.stl scale=0.001 0.001 0.001; visual mesh filename=package://repair_urdf/meshes/base_meshes/link_1.stl scale=0.001 0.001 0.001
- link arm_1_link_2: geometry collision mesh filename=package://repair_urdf/meshes/base_meshes/link_2.stl scale=0.001 0.001 0.001; visual mesh filename=package://repair_urdf/meshes/base_meshes/link_2.stl scale=0.001 0.001 0.001
- link arm_1_link_3: geometry collision mesh filename=package://repair_urdf/meshes/base_meshes/link_3.stl scale=0.001 0.001 0.001; visual mesh filename=package://repair_urdf/meshes/base_meshes/link_3.stl scale=0.001 0.001 0.001
- link arm_1_link_4: geometry collision mesh filename=package://repair_urdf/meshes/base_meshes/link_4.stl scale=0.001 0.001 0.001; visual mesh filename=package://repair_urdf/meshes/base_meshes/link_4.stl scale=0.001 0.001 0.001
- link arm_1_link_5: geometry collision mesh filename=package://repair_urdf/meshes/base_meshes/link_5.stl scale=0.001 0.001 0.001; visual mesh filename=package://repair_urdf/meshes/base_meshes/link_5.stl scale=0.001 0.001 0.001
- link arm_1_link_6: geometry collision mesh filename=package://repair_urdf/meshes/base_meshes/link_6.stl scale=0.001 0.001 0.001; visual mesh filename=package://repair_urdf/meshes/base_meshes/link_6.stl scale=0.001 0.001 0.001
- link arm_1_link_7: geometry 
- link arm_1_tcp: geometry visual mesh filename=package://repair_urdf/meshes/link_7_sh.stl scale=0.001 0.001 0.001
- link arm_2_link_1: geometry collision mesh filename=package://repair_urdf/meshes/base_meshes/link_1_mirror.stl scale=0.001 0.001 0.001; visual mesh filename=package://repair_urdf/meshes/base_meshes/link_1_mirror.stl scale=0.001 0.001 0.001
- link arm_2_link_2: geometry collision mesh filename=package://repair_urdf/meshes/base_meshes/link_2.stl scale=0.001 0.001 0.001; visual mesh filename=package://repair_urdf/meshes/base_meshes/link_2.stl scale=0.001 0.001 0.001
- link arm_2_link_3: geometry collision mesh filename=package://repair_urdf/meshes/base_meshes/link_3.stl scale=0.001 0.001 0.001; visual mesh filename=package://repair_urdf/meshes/base_meshes/link_3.stl scale=0.001 0.001 0.001
- link arm_2_link_4: geometry collision mesh filename=package://repair_urdf/meshes/base_meshes/link_4.stl scale=0.001 0.001 0.001; visual mesh filename=package://repair_urdf/meshes/base_meshes/link_4.stl scale=0.001 0.001 0.001
- link arm_2_link_5: geometry collision mesh filename=package://repair_urdf/meshes/base_meshes/link_5.stl scale=0.001 0.001 0.001; visual mesh filename=package://repair_urdf/meshes/base_meshes/link_5.stl scale=0.001 0.001 0.001
- link arm_2_link_6: geometry collision mesh filename=package://repair_urdf/meshes/base_meshes/link_6.stl scale=0.001 0.001 0.001; visual mesh filename=package://repair_urdf/meshes/base_meshes/link_6.stl scale=0.001 0.001 0.001
- link arm_2_link_7: geometry 
- link arm_2_tcp: geometry visual mesh filename=package://repair_urdf/meshes/link_7_rh.stl scale=0.001 0.001 0.001
- link base_link: geometry visual sphere radius=0.07; visual sphere radius=0.07
Joints:
- removed joint dummy_sliding_wrist1_joint
- removed joint dummy_sliding_wrist2_joint
- added joint arm_1_link7_coll_joint: type fixed, parent arm_1_link_7, child arm_1_link7_coll, origin xyz=0.0 0.0 -0.06 rpy=0 0 0
- added joint arm_1_link_1_coll_joint: type fixed, parent arm_1_link_1, child arm_1_link1_coll, origin xyz=0.0 0.0 0.0 rpy=0 0 0
- added joint arm_1_link_2_coll_joint: type fixed, parent arm_1_link_2, child arm_1_link2_coll, origin xyz=0.0 0 0.03 rpy=0 0 0
- added joint arm_1_link_3_coll_joint: type fixed, parent arm_1_link_3, child arm_1_link3_coll, origin xyz=0.0 0.0 0.22 rpy=0 0 0
- added joint arm_1_link_4_coll_joint: type fixed, parent arm_1_link_4, child arm_1_link4_coll, origin xyz=0.1 0.0 0.0 rpy=0 0 0
- added joint arm_1_link_5_coll_joint: type fixed, parent arm_1_link_5, child arm_1_link5_coll, origin xyz=-0.004109236058802465 0.0 0.321 rpy=0 0 0
- added joint arm_1_link_6_coll_joint: type fixed, parent arm_1_link_6, child arm_1_link6_coll, origin xyz=0.0 0.0 0.0 rpy=0 0 0
- added joint arm_2_link7_coll_joint: type fixed, parent arm_2_link_7, child arm_2_link7_coll, origin xyz=0.0 0.0 -0.06 rpy=0 0 0
- added joint arm_2_link_1_coll_joint: type fixed, parent arm_2_link_1, child arm_2_link1_coll, origin xyz=0.0 0.0 0.0 rpy=0 0 0
- added joint arm_2_link_2_coll_joint: type fixed, parent arm_2_link_2, child arm_2_link2_coll, origin xyz=0.0 0 0.03 rpy=0 0 0
- added joint arm_2_link_3_coll_joint: type fixed, parent arm_2_link_3, child arm_2_link3_coll, origin xyz=0.0 0.0 0.22 rpy=0 0 0
- added joint arm_2_link_4_coll_joint: type fixed, parent arm_2_link_4, child arm_2_link4_coll, origin xyz=0.1 0.0 0.0 rpy=0 0 0
- added joint arm_2_link_5_coll_joint: type fixed, parent arm_2_link_5, child arm_2_link5_coll, origin xyz=-0.004109236058802465 0.0 0.321 rpy=0 0 0
- added joint arm_2_link_6_coll_joint: type fixed, parent arm_2_link_6, child arm_2_link6_coll, origin xyz=0.0 0.0 0.0 rpy=0 0 0
- joint arm_1_joint_6: child dummy_sliding_wrist1_link -> arm_1_link_6; origin xyz=0 0 0.321 rpy=0 -1.57079632679 0 -> xyz=0.096 0.321 0 rpy=0 -1.57079632679 0
- joint arm_2_joint_6: child dummy_sliding_wrist2_link -> arm_2_link_6; origin xyz=0 0 0.321 rpy=0 -1.57079632679 0 -> xyz=0.096 0.321 0 rpy=0 -1.57079632679 0

File: repair_urdf/urdf/repair_full.urdf.xacro (robot description, xacro)
@@ -2,7 +2,7 @@
 <robot name = "repair_full" xmlns:xacro="http://ros.org/wiki/xacro">
 <xacro:arg name="is_sliding_wrist" default="false" />
-<xacro:arg name="show_softhand" default="false" />
-<xacro:arg name="show_coll" default="false" />
+<xacro:arg name="gen_coll" default="false" />
 <xacro:arg name="load_sol" default="false" />
+<xacro:arg name="use_updated_wrist" default="false" />
 <xacro:arg name="xbot" default="false" />
 <xacro:arg name="shorten_table_legs_coll" default="false" /> <!-- just to avoid flickering contact when loading into Gazebo -->
@@ -15,5 +15,5 @@
     <xacro:include filename="$(find repair_urdf)/urdf/xbot2.gazebo.xacro"/>
 </xacro:if>
-<!-- <xacro:if value="$(arg show_coll)">
+<!-- <xacro:if value="$(arg gen_coll)">
     <xacro:include filename="$(find repair_urdf)/urdf/repair_torso_coll_params.urdf.xacro"/>
     <xacro:include filename="$(find repair_urdf)/urdf/repair_torso_coll.urdf.xacro"/>
@@ -37,5 +37,5 @@
                   izz="0" />
         </inertial>
-        <xacro:if value="$(arg show_coll)">
+        <xacro:if value="$(arg gen_coll)">
             <visual name="link0_coll_visual1">
                 <origin xyz="0 0 0" rpy="0 0 0"/>
@@ -60,10 +60,12 @@
             </visual>
         </xacro:if>
-        <visual name="base_link_visual">
-            <geometry>
-                <mesh filename="package://repair_urdf/meshes/optimized/link_0.stl" scale="${mmTom} ${mmTom} ${mmTom}"/>
-            </geometry>
-            <material name="dark"/>
-        </visual>
+        <xacro:if value="$(arg use_updated_wrist)">
+            <visual name="base_link_visual">
+                <geometry>
+                    <mesh filename="package://repair_urdf/meshes/optimized/link_0.stl" scale="${mmTom} ${mmTom} ${mmTom}"/>
+                </geometry>
+                <material name="dark"/>
+            </visual>
+        </xacro:if>
     </link>
     <joint name="r_arm_mount_joint" type="fixed">
@@ -117,4 +119,43 @@
     <!-- RePAIR assembly (two arms) -->
     <link name="base_link">
+        <!-- torso inertias + stuff attached to the sliding guide -->
+        <inertial>
+            <mass value="${full_torso_mass}" />
+            <origin xyz="0 0 0" />
+            <inertia ixx="0" ixy="0"  ixz="0"
+                    iyy="0" iyz="0"
+                    izz="0" />
+          </inertial>
+          <xacro:if value="$(arg gen_coll)">
+            <visual name="link0_coll_visual1">
+                <origin xyz="0 0 0" rpy="0 0 0"/>
+                <geometry>
+                    <sphere radius="${coll_radius_link1}"/>
+                </geometry>
+                <material name="darkred"/>
+            </visual>
+            <visual name="link0_coll_visual2">
+                <origin xyz="0 ${link2_coll_offset_y} 0" rpy="0 0 0"/>
+                <geometry>
+                    <sphere radius="${coll_radius_link1}"/>
+                </geometry>
+                <material name="darkred"/>
+            </visual>
+            <visual name="link0_coll_visual3">
+                <origin xyz="0 ${- link2_coll_offset_y} 0" rpy="0 0 0"/>
+                <geometry>
+                    <sphere radius="${coll_radius_link1}"/>
+                </geometry>
+                <material name="darkred"/>
+            </visual>
+        </xacro:if>
+        <xacro:if value="$(arg use_updated_wrist)">
+            <visual name="base_link_visual">
+                <geometry>
+                    <mesh filename="package://repair_urdf/meshes/optimized/link_0.stl" scale="${mmTom} ${mmTom} ${mmTom}"/>
+                </geometry>
+                <material name="dark"/>
+            </visual>
+        </xacro:if>
     </link>
     <link name="dummy_r">
@@ -156,7 +197,7 @@
 </xacro:unless>
 <xacro:repair_arm base_link="r_arm_mount_frame" id="1" is_sliding_wrist="$(arg is_sliding_wrist)"
-show_softhand="$(arg show_softhand)" show_coll="$(arg show_coll)" load_sol="$(arg load_sol)"/>
+gen_coll="$(arg gen_coll)" load_sol="$(arg load_sol)" use_updated_wrist = "$(arg use_updated_wrist)"/>
 <xacro:repair_arm base_link="l_arm_mount_frame" id="2" is_sliding_wrist="$(arg is_sliding_wrist)"
-show_softhand="$(arg show_softhand)" show_coll="$(arg show_coll)" load_sol="$(arg load_sol)"/>
+gen_coll="$(arg gen_coll)" load_sol="$(arg load_sol)" use_updated_wrist = "$(arg use_updated_wrist)"/>
 <xacro:repair_arm_materials id="1" />
 <xacro:repair_arm_materials id="2" />

Commit message: fixed wrong joint limit

File: repair_urdf/urdf/repair_arm.urdf.xacro (robot description, xacro)
@@ -169,5 +169,5 @@
     <child link="arm_${id}_link_4"/>
     <axis xyz="0 0 1"/>
-    <limit lower="${-150.0 * DEG2RAD}" upper="${120.0 * DEG2RAD}" effort="${big_tau_max}" velocity="10.0"/>
+    <limit lower="${-150.0 * DEG2RAD}" upper="${60.0 * DEG2RAD}" effort="${big_tau_max}" velocity="10.0"/>
 </joint>
 <link name="arm_${id}_link_4">

Commit message: final polishing

File: repair_urdf/urdf/repair_arm.urdf.xacro (robot description, xacro)
@@ -14,5 +14,5 @@
 <xacro:property name="sm_tau_max" value="200.0" />
 <xacro:include filename="$(find repair_urdf)/urdf/repair_arm_coll_params.urdf.xacro"/>
-<xacro:macro name="repair_arm" params="id base_link is_sliding_wrist gen_coll load_sol use_updated_wrist" >
+<xacro:macro name="repair_arm" params="id base_link is_sliding_wrist gen_coll load_sol use_updated_wrist gz_self_collide" >
 <xacro:if value="${gen_coll == True}">
     <xacro:include filename="$(find repair_urdf)/urdf/repair_arm_coll.urdf.xacro"/>
@@ -367,4 +367,24 @@
     </visual>
 </link>
+<xacro:if value="${gz_self_collide == 1}">
+    <gazebo reference="arm_${id}_link_1">
+        <selfCollide> 1 </selfCollide>
+    </gazebo>
+    <gazebo reference="arm_${id}_link_2">
+        <selfCollide> 1 </selfCollide>
+    </gazebo>
+    <gazebo reference="arm_${id}_link_3">
+        <selfCollide> 1 </selfCollide>
+    </gazebo>
+    <gazebo reference="arm_${id}_link_4">
+        <selfCollide> 1 </selfCollide>
+    </gazebo>
+    <gazebo reference="arm_${id}_link_5">
+        <selfCollide> 1 </selfCollide>
+    </gazebo>
+    <gazebo reference="arm_${id}_link_6">
+        <selfCollide> 1 </selfCollide>
+    </gazebo>
+</xacro:if>
 </xacro:macro>
 </robot>

File: repair_urdf/urdf/repair_full.urdf.xacro (robot description, xacro)
@@ -10,17 +10,13 @@
 results of the optimization), otherwise we go with the old ones (generated for a spherical wrist) -->
 <robot name = "repair_full" xmlns:xacro="http://ros.org/wiki/xacro">
-<xacro:arg name="is_sliding_wrist" default="false" />
+<xacro:arg name="is_sliding_wrist" default="true" />
 <xacro:arg name="gen_coll" default="false" />
-<xacro:arg name="load_sol" default="false" />
+<xacro:arg name="load_sol" default="true" />
 <xacro:arg name="use_updated_wrist" default="false" />
+<xacro:arg name="gz_self_collide" default="true" />
 <xacro:include filename="$(find repair_urdf)/urdf/repair_arm.urdf.xacro"/>
 <xacro:include filename="$(find repair_urdf)/urdf/repair_cage.urdf.xacro"/>
 <xacro:include filename="$(find repair_urdf)/urdf/repair_opt_mount_params.urdf.xacro"/>
 <xacro:include filename="$(find repair_urdf)/urdf/materials.gazebo.xacro"/>
-<!-- <xacro:if value="$(arg gen_coll)">
-    <xacro:include filename="$(find repair_urdf)/urdf/repair_torso_coll_params.urdf.xacro"/>
-    <xacro:include filename="$(find repair_urdf)/urdf/repair_torso_coll.urdf.xacro"/>
-    <xacro:repair_torso_coll />
-</xacro:if> -->
 <xacro:if value="$(arg load_sol)">
     <joint name="x_joint" type="prismatic">
@@ -154,9 +150,16 @@
 </xacro:unless>
 <xacro:repair_arm base_link="r_arm_mount_frame" id="1" is_sliding_wrist="$(arg is_sliding_wrist)"
-gen_coll="$(arg gen_coll)" load_sol="$(arg load_sol)" use_updated_wrist = "$(arg use_updated_wrist)"/>
+gen_coll="$(arg gen_coll)" load_sol="$(arg load_sol)" use_updated_wrist = "$(arg use_updated_wrist)"
+gz_self_collide = "$(arg gz_self_collide)" />
 <xacro:repair_arm base_link="l_arm_mount_frame" id="2" is_sliding_wrist="$(arg is_sliding_wrist)"
-gen_coll="$(arg gen_coll)" load_sol="$(arg load_sol)" use_updated_wrist = "$(arg use_updated_wrist)"/>
+gen_coll="$(arg gen_coll)" load_sol="$(arg load_sol)" use_updated_wrist = "$(arg use_updated_wrist)"
+gz_self_collide = "$(arg gz_self_collide)" />
 <xacro:repair_arm_materials id="1" />
 <xacro:repair_arm_materials id="2" />
 <xacro:repair_torso_materials />
+<xacro:if value="$(arg gz_self_collide)">
+    <gazebo reference="table_top_link">
+        <selfCollide> 1 </selfCollide>
+    </gazebo>
+</xacro:if>
 </robot>

Commit message: added softhands v1 simple to URDF

File: repair_urdf/urdf/repair_arm.urdf.xacro (robot description, xacro)
@@ -10,4 +10,6 @@
 <robot name = "repair_arm" xmlns:xacro="http://ros.org/wiki/xacro">
 <xacro:include filename="$(find repair_urdf)/urdf/utils.urdf.xacro" />
+<xacro:include filename="$(find softhands_description)/urdf/softhands.xacro" />
+<!-- <xacro:include filename="$(find softhands_description)/urdf/utils.urdf.xacro" /> -->
 <xacro:property name="big_tau_max" value="200.0" />
 <xacro:property name="mid_tau_max" value="200.0" />
@@ -327,8 +329,8 @@
 <joint name="arm_${id}_joint_7" type="revolute">
     <xacro:if value="${id == 1}">
-        <origin xyz="${180.000 * mmTom} 0 0" rpy="${PI_2} 0 ${PI_2}"/>
+        <origin xyz="0.08 0 0" rpy="${PI_2} 0 ${PI_2}"/>
     </xacro:if>
     <xacro:unless value="${id == 1}">
-        <origin xyz="${180.000 * mmTom} 0 0" rpy="${-PI_2} ${PI} ${-PI_2}"/>
+        <origin xyz="0.08 0 0" rpy="${-PI_2} ${PI} ${-PI_2}"/>
         <!-- <origin xyz="${180.000 * mmTom} 0 0" rpy="${-PI_2} 0 ${-PI_2}"/> -->
     </xacro:unless>
@@ -345,26 +347,24 @@
     </inertial>
 </link>
-<joint name="arm_${id}_tcp_joint" type="fixed">
-    <origin xyz="0 ${- object_size *  sin(softhand_mount_angle)} ${10.0 * mmTom + object_size *  cos(softhand_mount_angle)}"
-            rpy="0 ${-(PI_2 + softhand_mount_angle)} ${-(PI_2)}"/>
-    <parent link="arm_${id}_link_7"/>
-    <child link="arm_${id}_tcp"/>
-</joint>
-<link name="arm_${id}_tcp">
-    <visual name="arm_${id}_tcp_visual">
-        <origin xyz="0 0 ${object_size}" rpy="0 0 0"/>
-        <xacro:if value="${id == 1}">
-            <geometry>
-                <mesh filename="package://repair_urdf/meshes/link_7_sh.stl" scale="${mmTom} ${mmTom} ${mmTom}"/>
-            </geometry>
-        </xacro:if>
-        <xacro:unless value="${id == 1}">
-                <geometry>
-                    <mesh filename="package://repair_urdf/meshes/link_7_rh.stl" scale="${mmTom} ${mmTom} ${mmTom}"/>
-                </geometry>
-        </xacro:unless>
-        <material name="dark"/>
-    </visual>
-</link>
+<xacro:if value="${id == 1}">
+    <xacro:softhands type="right"
+        version="v1.0_simple"
+        parent="arm_${id}_link_7"
+        position="0 -0.015 0"
+        orientation="0 0 0"
+        operation_mode="0"
+        translation="0">
+    </xacro:softhands>
+</xacro:if>
+<xacro:unless value="${id == 1}">
+    <xacro:softhands type="left"
+        version="v1.0_simple"
+        parent="arm_${id}_link_7"
+        position="0 -0.015 0"
+        orientation="0 0 0"
+        operation_mode="0"
+        translation="0">
+    </xacro:softhands>
+</xacro:unless>
 <xacro:if value="${gz_self_collide == 1}">
     <gazebo reference="arm_${id}_link_1">

Commit message: fixed mounting orientation and position of SoftHands

File: repair_urdf/urdf/repair_arm.urdf.xacro (robot description, xacro)
@@ -351,8 +351,8 @@
         version="v1.0_simple"
         parent="arm_${id}_link_7"
-        position="0 -0.015 0"
+        position="0 0 -0.015"
         orientation="0 0 0"
+        translation="0"
         operation_mode="0"
-        translation="0"
         fixed_hands="${fixed_hands}">
     </xacro:softhands>
@@ -362,8 +362,8 @@
         version="v1.0_simple"
         parent="arm_${id}_link_7"
-        position="0 -0.015 0"
-        orientation="0 0 0"
+        position="0 0.013900 -0.015"
+        orientation="0 0.0 ${PI}"
+        translation="0"
         operation_mode="0"
-        translation="0"
         fixed_hands="${fixed_hands}">
     </xacro:softhands>

File: repair_urdf/urdf/repair_full.urdf (robot description, URDF)
Before this commit: robot repair_full, 79 links, 78 joints
Joints:
- joint left_hand_base_joint: origin xyz=0 -0.015 0 rpy=0 0 0 -> xyz=0 0.013900 -0.015 rpy=0 0.0 3.14159265359
- joint right_hand_base_joint: origin xyz=0 -0.015 0 rpy=0 0 0 -> xyz=0 0 -0.015 rpy=0 0 0
