Commit message: fully working simulation pipeline

File: repair_urdf/urdf/materials.gazebo.xacro (robot description, xacro)
@@ -6,5 +6,5 @@
 </gazebo>
 <gazebo reference="arm_${id}_link_2">
-	<material>Gazebo/DarkMagentaTransparent   </material>
+	<material>Gazebo/GreenTransparent    </material>
 </gazebo>
 <gazebo reference="arm_${id}_link_3">
@@ -12,5 +12,5 @@
 </gazebo>
 <gazebo reference="arm_${id}_link_4">
-	<material>Gazebo/DarkMagentaTransparent   </material>
+	<material>Gazebo/GreenTransparent    </material>
 </gazebo>
 <gazebo reference="arm_${id}_link_5">
@@ -18,5 +18,5 @@
 </gazebo>
 <gazebo reference="arm_${id}_link_6">
-	<material>Gazebo/DarkMagentaTransparent   </material>
+	<material>Gazebo/GreenTransparent    </material>
 </gazebo>
 <gazebo reference="arm_${id}_link_7">
@@ -24,5 +24,5 @@
 </gazebo>
 <gazebo reference="arm_${id}_tcp">
-	<material>Gazebo/BlackTransparent   </material>
+	<material>Gazebo/GreyTransparent    </material>
 </gazebo>
 </xacro:macro>

File: repair_urdf/urdf/repair_full.urdf.xacro (robot description, xacro)
@@ -7,4 +7,5 @@
 <xacro:arg name="xbot" default="false" />
 <xacro:arg name="shorten_table_legs_coll" default="false" /> <!-- just to avoid flickering contact when loading into Gazebo -->
+<xacro:arg name="self_collide_gz" default="true" />
 <xacro:include filename="$(find repair_urdf)/urdf/repair_arm.urdf.xacro"/>
 <xacro:include filename="$(find repair_urdf)/urdf/repair_cage.urdf.xacro"/>

File: repair_urdf/urdf/utils.urdf.xacro (robot description, xacro)
@@ -50,3 +50,9 @@
     </inertial>
 </xacro:macro>
+<!-- just used to write more compactly the self collision gazebo ref tag -->
+<xacro:macro name="gz_self_collide" params="collide">
+    <xacro:if value="${collide == True}">
+        <self_collide>1</self_collide>
+    </xacro:if>
+</xacro:macro>
 </robot>

Commit message: some gain tuning

File: repair_urdf/urdf/materials.gazebo.xacro (robot description, xacro)
@@ -25,4 +25,9 @@
 <gazebo reference="arm_${id}_tcp">
 	<material>Gazebo/GreyTransparent    </material>
+</gazebo>
+</xacro:macro>
+<xacro:macro name="repair_torso_materials" >
+<gazebo reference="base_link">
+	<material>Gazebo/GreenTransparent   </material>
 </gazebo>
 </xacro:macro>

File: repair_urdf/urdf/repair_full.urdf (robot description, URDF)
Before this commit: robot repair_full, 39 links, 38 joints
Links:
- link base_link: geometry visual mesh filename=package://repair_urdf/meshes/optimized/link_0.stl scale=0.001 0.001 0.001

File: repair_urdf/urdf/repair_full.urdf.xacro (robot description, xacro)
@@ -161,3 +161,4 @@
 <xacro:repair_arm_materials id="1" />
 <xacro:repair_arm_materials id="2" />
+<xacro:repair_torso_materials />
 </robot>

Commit message: cleaned repo and added comments to improve usability

File: repair_urdf/urdf/materials.gazebo.xacro (robot description, xacro)
@@ -1,3 +1,4 @@
 <?xml version="1.0"?>
+<!-- Just definitions of materials for visualization purposes -->
 <robot xmlns:xacro="http://ros.org/wiki/xacro">
 <xacro:macro name="repair_arm_materials" params="id">

File: repair_urdf/urdf/repair_arm.urdf.xacro (robot description, xacro)
@@ -1,3 +1,11 @@
 <?xml version="1.0"?>
+<!-- macro for generating the urdf associated with a single arm of the RePair platform -->
+<!-- id: specifies the id of the arm (e.g. 0 for left arm and 1 for right) -->
+<!-- base_link: name of base link a the single arm -->
+<!-- is_sliding_wrist: whether to add a sliding joint along the wrist second d.o.f.
+    (true -> yes), everything else -> no. This is used to generate the URDF for the optimization.  -->
+<!-- gen_coll: whether to add the approximate collision  model of the platform -->
+<!-- use_updated_wrist: visual parameter. if true, we load the latest meshes (which are adapted to the
+results of the optimization), otherwise we go with the old ones (generated for a spherical wrist) -->
 <robot name = "repair_arm" xmlns:xacro="http://ros.org/wiki/xacro">
 <xacro:include filename="$(find repair_urdf)/urdf/utils.urdf.xacro" />

File: repair_urdf/urdf/repair_arm_coll.urdf.xacro (robot description, xacro)
@@ -1,4 +1,7 @@
 <?xml version="1.0"?>
 <robot xmlns:xacro="http://www.ros.org/wiki/xacro">
+<!-- File defining a macro for generating the collision links for the RePair platform -->
+<!-- load_sol = true is used when the wrist auxiliary d.o.f. (used inside the optimization) has to be
+removed -->
 <xacro:macro name="repair_arm_coll" params="load_sol" />
 <joint name="arm_${id}_link_1_coll_joint" type="fixed">

File: repair_urdf/urdf/repair_arm_coll_params.urdf.xacro (robot description, xacro)
@@ -1,7 +1,10 @@
 <?xml version="1.0"?>
 <robot xmlns:xacro="http://www.ros.org/wiki/xacro">
-<!-- Reading some parameters from a YAML config file -->
+<!-- Reading some parameters from a YAML config file for the approximate collision model for RePair.
+Links are approximated as spheres with hand-tuned radii and positions -->
+<!-- loading yaml and its tags -->
 <xacro:property name="yaml_file" value="$(find repair_urdf)/config/arm_coll.yaml" />
 <xacro:property name="coll_props" value="${xacro.load_yaml(yaml_file)}"/>
+<!-- reading relevant properties -->
 <xacro:property name="coll_radius_link1" value="${coll_props['link1_coll']['coll_radius']}" />
 <xacro:property name="coll_radius_link2" value="${coll_props['link2_coll']['coll_radius']}" />
@@ -11,4 +14,5 @@
 <xacro:property name="coll_radius_link6" value="${coll_props['link6_coll']['coll_radius']}" />
 <xacro:property name="coll_radius_link7" value="${coll_props['link7_coll']['coll_radius']}" />
+<!-- collision links positions (hand-tuned) -->
 <xacro:property name="link1_coll_offset_x" value="0.0" />
 <xacro:property name="link1_coll_offset_y" value="0.0" />

File: repair_urdf/urdf/repair_cage.urdf.xacro (robot description, xacro)
@@ -1,3 +1,4 @@
 <?xml version="1.0"?>
+<!-- xacro for the cage defining the workspace of the RePair platform -->
 <robot name = "repair_cage" xmlns:xacro="http://ros.org/wiki/xacro">
   <xacro:include filename="$(find repair_urdf)/urdf/materials.gazebo.xacro"/>
@@ -16,10 +17,10 @@
   <xacro:property name="PI_2" value="1.57079632679" />
   <!-- only something to avoid collisions between leg and ground plane when using Gaz. -->
-  <xacro:if value="$(arg shorten_table_legs_coll)">
+  <!-- <xacro:if value="$(arg shorten_table_legs_coll)">
     <xacro:property name="leg_z_offset_gz" value="0.05" />
   </xacro:if>
-  <xacro:unless value="$(arg shorten_table_legs_coll)">
     <xacro:property name="leg_z_offset_gz" value="0.0" />
-  </xacro:unless>
+  </xacro:unless> -->
+  <xacro:property name="leg_z_offset_gz" value="0.0" />
   <material name="wood">
     <color rgba="0.522 0.369 0.259 0.8"/>

File: repair_urdf/urdf/repair_full.urdf.xacro (robot description, xacro)
@@ -1,3 +1,13 @@
 <?xml version="1.0"?>
+<!-- xacro for generating the full urdf of the RePair platform (cage + bimanual robot) -->
+<!-- is_sliding_wrist: whether to add a sliding joint along the wrist second d.o.f.
+    (true -> yes), everything else -> no. This is used to generate the URDF for the optimization.  -->
+<!-- gen_coll: whether to add the approximate collision  model of the platform -->
+<!-- load_sol: whether to generate the URDF without the additional d.o.f. used by the co-design optimization.
+Setting it to "true", allow to fix the additional d.o.f. to desired values
+(specified in the repair_urdf/config/arm_opt_mount_vals.yaml file) -->
+<!-- use_updated_wrist: visual parameter. if true, we load the latest meshes (which are adapted to the
+results of the optimization), otherwise we go with the old ones (generated for a spherical wrist) -->
+<!-- xbot: if true, we add the gazebo tags necessary to use the URDF with XBot2 framework -->
 <robot name = "repair_full" xmlns:xacro="http://ros.org/wiki/xacro">
 <xacro:arg name="is_sliding_wrist" default="false" />
@@ -6,6 +16,4 @@
 <xacro:arg name="use_updated_wrist" default="false" />
 <xacro:arg name="xbot" default="false" />
-<xacro:arg name="shorten_table_legs_coll" default="false" /> <!-- just to avoid flickering contact when loading into Gazebo -->
-<xacro:arg name="self_collide_gz" default="true" />
 <xacro:include filename="$(find repair_urdf)/urdf/repair_arm.urdf.xacro"/>
 <xacro:include filename="$(find repair_urdf)/urdf/repair_cage.urdf.xacro"/>

File: repair_urdf/urdf/repair_opt_mount_params.urdf.xacro (robot description, xacro)
@@ -1,5 +1,5 @@
 <?xml version="1.0"?>
 <robot xmlns:xacro="http://www.ros.org/wiki/xacro">
-<!-- Reading some parameters from a YAML config file -->
+<!-- Reading mounting paramters from YAML file -->
 <xacro:property name="yaml_file2" value="$(find repair_urdf)/config/arm_opt_mount_vals.yaml" />
 <xacro:property name="opt_mount_vals" value="${xacro.load_yaml(yaml_file2)}"/>

File: repair_urdf/urdf/repair_torso_coll.urdf.xacro (robot description, xacro)
@@ -1,4 +1,5 @@
 <?xml version="1.0"?>
 <robot xmlns:xacro="http://www.ros.org/wiki/xacro">
+<!-- RePair torso collision model  -->
 <xacro:macro name="repair_torso_coll" />
 <joint name="link0_coll_joint1" type="fixed">

File: repair_urdf/urdf/repair_torso_coll_params.urdf.xacro (robot description, xacro)
@@ -1,5 +1,5 @@
 <?xml version="1.0"?>
 <robot xmlns:xacro="http://www.ros.org/wiki/xacro">
-<!-- Reading some parameters from a YAML config file -->
+<!-- RePair torso collision parameters -->
 <xacro:property name="yaml_file" value="$(find repair_urdf)/config/arm_coll.yaml" />
 <xacro:property name="coll_props" value="${xacro.load_yaml(yaml_file)}"/>

File: repair_urdf/urdf/utils.urdf.xacro (robot description, xacro)
@@ -1,3 +1,4 @@
 <?xml version="1.0"?>
+<!-- Just definitions of useful paramters -->
 <robot xmlns:xacro="http://ros.org/wiki/xacro">
 <!-- scale -->

File: repair_urdf/urdf/xbot2.gazebo.xacro (robot description, xacro)
@@ -1,3 +1,4 @@
 <?xml version="1.0"?>
+<!-- XBot2-specific gazebo tags -->
 <robot xmlns:xacro="http://ros.org/wiki/xacro">
 <!-- xbot2 joint device driver-->
@@ -10,6 +11,6 @@
             <gain name="big_mot"    p="8000" d="50"/>
             <gain name="hugr_mot"    p="12000" d="70"/>
-            <gain name="wheel_mot"  p="0" d="10"/>
-            <pid name="x_joint" profile="big_mot"/>
+            <gain name="guide_motor"  p="8000" d="50"/>
+            <pid name="x_joint" profile="guide_motor"/>
             <pid name="arm_1_joint_1" profile="big_mot"/>
             <pid name="arm_1_joint_2" profile="big_mot"/>

Commit message: awesome color update

File: repair_urdf/urdf/materials.gazebo.xacro (robot description, xacro)
@@ -4,26 +4,26 @@
 <xacro:macro name="repair_arm_materials" params="id">
 <gazebo reference="arm_${id}_link_1">
-	<material>Gazebo/BlackTransparent   </material>
+	<material>Gazebo/Grey     </material>
 </gazebo>
 <gazebo reference="arm_${id}_link_2">
-	<material>Gazebo/GreenTransparent    </material>
+	<material>Gazebo/BlueLaser      </material>
 </gazebo>
 <gazebo reference="arm_${id}_link_3">
-	<material>Gazebo/BlackTransparent   </material>
+	<material>Gazebo/Grey      </material>
 </gazebo>
 <gazebo reference="arm_${id}_link_4">
-	<material>Gazebo/GreenTransparent    </material>
+	<material>Gazebo/BlueLaser      </material>
 </gazebo>
 <gazebo reference="arm_${id}_link_5">
-	<material>Gazebo/BlackTransparent  </material>
+	<material>Gazebo/Grey     </material>
 </gazebo>
 <gazebo reference="arm_${id}_link_6">
-	<material>Gazebo/GreenTransparent    </material>
+	<material>Gazebo/BlueLaser      </material>
 </gazebo>
 <gazebo reference="arm_${id}_link_7">
-	<material>Gazebo/BlackTransparent  </material>
+	<material>Gazebo/Grey     </material>
 </gazebo>
 <gazebo reference="arm_${id}_tcp">
-	<material>Gazebo/GreyTransparent    </material>
+	<material>Gazebo/BlueLaser      </material>
 </gazebo>
 </xacro:macro>
