Commit message: added simplified meshes

File: repair_urdf/urdf/repair_arm_macro.urdf.xacro (robot description, xacro)
@@ -25,5 +25,5 @@
             <collision>
                 <geometry>
-                    <mesh filename="package://repair_urdf/meshes/mesh_sh-pitch.stl" scale="0.001 ${rot*0.001} 0.001"/>
+                    <mesh filename="package://repair_urdf/meshes/simplified/mesh_sh-pitch.stl" scale="0.001 ${rot*0.001} 0.001"/>
                 </geometry>
             </collision>
@@ -44,5 +44,5 @@
             <collision>
                 <geometry>
-                    <mesh filename="package://repair_urdf/meshes/mesh_sh-roll.stl" scale="0.001 ${rot*0.001} 0.001"/>
+                    <mesh filename="package://repair_urdf/meshes/simplified/mesh_sh-roll.stl" scale="0.001 ${rot*0.001} 0.001"/>
                 </geometry>
             </collision>
@@ -63,5 +63,5 @@
             <collision>
                 <geometry>
-                    <mesh filename="package://repair_urdf/meshes/mesh_sh-yaw.stl" scale="0.001 ${rot*0.001} 0.001"/>
+                    <mesh filename="package://repair_urdf/meshes/simplified/mesh_sh-yaw.stl" scale="0.001 ${rot*0.001} 0.001"/>
                 </geometry>
             </collision>
@@ -82,5 +82,5 @@
             <collision>
                 <geometry>
-                    <mesh filename="package://repair_urdf/meshes/mesh_elbow.stl" scale="0.001 ${rot*0.001} 0.001"/>
+                    <mesh filename="package://repair_urdf/meshes/simplified/mesh_elbow.stl" scale="0.001 ${rot*0.001} 0.001"/>
                 </geometry>
             </collision>
@@ -101,5 +101,5 @@
             <collision>
                 <geometry>
-                    <mesh filename="package://repair_urdf/meshes/mesh_forearm-yaw.stl" scale="0.001 ${rot*0.001} 0.001"/>
+                    <mesh filename="package://repair_urdf/meshes/simplified/mesh_forearm-yaw.stl" scale="0.001 ${rot*0.001} 0.001"/>
                 </geometry>
             </collision>
@@ -120,5 +120,5 @@
             <collision>
                 <geometry>
-                    <mesh filename="package://repair_urdf/meshes/mesh_wrist-pitch.stl" scale="0.001 ${rot*0.001} 0.001"/>
+                    <mesh filename="package://repair_urdf/meshes/simplified/mesh_wrist-pitch.stl" scale="0.001 ${rot*0.001} 0.001"/>
                 </geometry>
             </collision>
@@ -139,5 +139,5 @@
             <collision>
                 <geometry>
-                    <mesh filename="package://repair_urdf/meshes/mesh_wrist-roll.stl" scale="0.001 ${rot*0.001} 0.001"/>
+                    <mesh filename="package://repair_urdf/meshes/simplified/mesh_wrist-roll.stl" scale="0.001 ${rot*0.001} 0.001"/>
                 </geometry>
             </collision>
