Commit message: stress test and signs working on real robot. First Cartesio tests on a single arm in dummy mode.

File: repair_urdf/urdf/repair_arm.urdf (robot description, URDF)
Before this commit: robot repair_arm, 10 links, 9 joints
Links:
- link base_link: mass None -> 2.7764953; geometry collision mesh filename=package://repair_urdf/meshes/simplified/mesh_base.stl scale=0.001 0.001 0.001; visual mesh filename=package://repair_urdf/meshes/mesh_base.stl scale=0.001 0.001 0.001
Joints:
- joint j_arm_1_1: origin xyz=0.0 -0.13515 -0.24215 rpy=1.570796326795 0.0 0.0 -> xyz=0.0 0.0 0.14 rpy=0.0 0.0 0.0
- joint j_arm_1_2: axis 0 0 1 -> 0 0 -1
- joint j_arm_1_3: axis 0 0 1 -> 0 0 -1
- joint j_arm_1_4: axis 0 0 1 -> 0 0 -1
- joint j_arm_1_5: axis 0 0 1 -> 0 0 -1

File: repair_urdf/urdf/repair_arm_final.urdf.xacro (robot description, xacro)
@@ -1,4 +1,4 @@
 <?xml version="1.0"?>
-<robot xmlns:xacro="http://ros.org/wiki/xacro" name="inail2arm">
+<robot xmlns:xacro="http://ros.org/wiki/xacro" name="repair_arm">
     <xacro:include filename="$(find repair_urdf)/urdf/conversions.urdf.xacro" />
     <xacro:include filename="$(find repair_urdf)/urdf/materials.urdf.xacro" />

File: repair_urdf/urdf/repair_arm_macro.urdf.xacro (robot description, xacro)
@@ -161,5 +161,5 @@
             <origin xyz="${Shoulder_2_Ox} ${rot*Shoulder_2_Oy} ${Shoulder_2_Oz}"
             rpy="${rot*Shoulder_2_roll} ${Shoulder_2_pitch} ${Shoulder_2_yaw}" />
-            <axis xyz="0 0 1" />
+            <axis xyz="0 0 -1" />
             <limit lower="${j_arm_2_lower[0]}" upper="${j_arm_2_upper[0]}"
             effort="${j_arm_2_torque[0]}" velocity="${j_arm_2_velocity[0]}" />
@@ -172,5 +172,5 @@
             <origin xyz="${Shoulder_3_Ox} ${rot*Shoulder_3_Oy} ${Shoulder_3_Oz}"
             rpy="${rot*Shoulder_3_roll} ${Shoulder_3_pitch} ${Shoulder_3_yaw}" />
-            <axis xyz="0 0 1" />
+            <axis xyz="0 0 -1" />
             <limit lower="${j_arm_3_lower[0]}" upper="${j_arm_3_upper[0]}"
             effort="${j_arm_3_torque[0]}" velocity="${j_arm_3_velocity[0]}" />
@@ -183,5 +183,5 @@
             <origin xyz="${Elbow_1_Ox} ${rot*Elbow_1_Oy} ${Elbow_1_Oz}"
             rpy="${rot*Elbow_1_roll} ${Elbow_1_pitch} ${Elbow_1_yaw}" />
-            <axis xyz="0 0 1" />
+            <axis xyz="0 0 -1" />
             <limit lower="${j_arm_4_lower[0]}" upper="${j_arm_4_upper[0]}"
             effort="${j_arm_4_torque[0]}" velocity="${j_arm_4_velocity[0]}" />
@@ -194,5 +194,5 @@
             <origin xyz="${Forearm_1_Ox} ${rot*Forearm_1_Oy} ${Forearm_1_Oz}"
             rpy="${rot*Forearm_1_roll} ${Forearm_1_pitch} ${Forearm_1_yaw}" />
-            <axis xyz="0 0 1" />
+            <axis xyz="0 0 -1" />
             <limit lower="${j_arm_5_lower[0]}" upper="${j_arm_5_upper[0]}"
             effort="${j_arm_5_torque[0]}" velocity="${j_arm_5_velocity[0]}" />

Commit message: added cartesio test

File: repair_urdf/urdf/repair_arm.urdf (robot description, URDF)
Before this commit: robot repair_arm, 10 links, 9 joints
Links:
- link arm_1_tcp: mass None -> 0.5
Joints:
- joint j_arm_1_7: origin xyz=0.0216503 0.062877 0.05 rpy=-1.570796326795 0.3316123 0.0 -> xyz=0.0 0.062877 0.05 rpy=-1.570796326795 0.3316123 0.0
