Commit message: first working test on a single arm

File: repair_urdf/urdf/limits.urdf.xacro (robot description, xacro)
@@ -2,18 +2,18 @@
 <robot  xmlns:xacro="http://ros.org/wiki/xacro">
     <!-- Origin -->
-    <xacro:property name="j_arm_1_lower" value="${[-2.85]}"/>
-    <xacro:property name="j_arm_2_lower" value="${[-2.0]}"/>
-    <xacro:property name="j_arm_3_lower" value="${[-2.2]}"/>
-    <xacro:property name="j_arm_4_lower" value="${[-2.7]}"/>
-    <xacro:property name="j_arm_5_lower" value="${[-2.2]}"/>
-    <xacro:property name="j_arm_6_lower" value="${[-2.85]}"/>
-    <xacro:property name="j_arm_7_lower" value="${[-2.85]}"/>
-    <xacro:property name="j_arm_1_upper" value="${[2.85]}"/>
-    <xacro:property name="j_arm_2_upper" value="${[2.0]}"/>
-    <xacro:property name="j_arm_3_upper" value="${[2.2]}"/>
-    <xacro:property name="j_arm_4_upper" value="${[2.7]}"/>
-    <xacro:property name="j_arm_5_upper" value="${[2.2]}"/>
-    <xacro:property name="j_arm_6_upper" value="${[2.85]}"/>
-    <xacro:property name="j_arm_7_upper" value="${[2.85]}"/>
+    <xacro:property name="j_arm_1_lower" value="${[-2.6]}"/>
+    <xacro:property name="j_arm_2_lower" value="${[-2.5]}"/>
+    <xacro:property name="j_arm_3_lower" value="${[-2.6]}"/>
+    <xacro:property name="j_arm_4_lower" value="${[-2.4]}"/>
+    <xacro:property name="j_arm_5_lower" value="${[-2.8]}"/>
+    <xacro:property name="j_arm_6_lower" value="${[-2.8]}"/>
+    <xacro:property name="j_arm_7_lower" value="${[-2.8]}"/>
+    <xacro:property name="j_arm_1_upper" value="${[2.6]}"/>
+    <xacro:property name="j_arm_2_upper" value="${[0.1]}"/>
+    <xacro:property name="j_arm_3_upper" value="${[2.6]}"/>
+    <xacro:property name="j_arm_4_upper" value="${[0.8]}"/>
+    <xacro:property name="j_arm_5_upper" value="${[2.8]}"/>
+    <xacro:property name="j_arm_6_upper" value="${[2.1]}"/>
+    <xacro:property name="j_arm_7_upper" value="${[2.8]}"/>
     <xacro:property name="j_arm_1_velocity" value="${[3.86]}"/>
     <xacro:property name="j_arm_2_velocity" value="${[3.86]}"/>

Commit message: fixed repair_full

File: repair_urdf/urdf/limits.urdf.xacro (robot description, xacro)
@@ -38,9 +38,3 @@
     <xacro:property name="j_arm_6_torque" value="${[55.00]}"/>
     <xacro:property name="j_arm_7_torque" value="${[55.00]}"/>
-    <!-- <xacro:property name="motor_A_velocity" value="8.8"/>
-    <xacro:property name="motor_B_velocity" value="8.1"/>
-    <xacro:property name="motor_C_velocity" value="20.0"/>
-    <xacro:property name="motor_A_effort" value="304"/>
-    <xacro:property name="motor_B_effort" value="147"/>
-    <xacro:property name="motor_C_effort" value="35"/> -->
     </robot>
