Commit message: added base meshes

File: repair_urdf/urdf/kinematics_properties.urdf.xacro (robot description, xacro)
@@ -2,10 +2,10 @@
 <robot  xmlns:xacro="http://ros.org/wiki/xacro">
     <!-- Origin -->
-    <xacro:property name="Shoulder_1_Ox" value=" 0.0 "/>
-    <xacro:property name="Shoulder_1_Oy" value=" -0.13515 "/>
-    <xacro:property name="Shoulder_1_Oz" value=" -0.24215 "/>
-    <xacro:property name="Shoulder_1_roll" value=" ${PI/2} "/>
-    <xacro:property name="Shoulder_1_pitch" value=" 0.0 "/>
-    <xacro:property name="Shoulder_1_yaw" value=" 0.0 "/>
+    <xacro:property name="Shoulder_1_Ox" value=" 0.0 "/>  <!-- 0.0  -->
+    <xacro:property name="Shoulder_1_Oy" value=" 0.0"/> <!-- 0.13515  -->
+    <xacro:property name="Shoulder_1_Oz" value=" 0.14 "/> <!-- -0.24215  -->
+    <xacro:property name="Shoulder_1_roll" value=" 0.0 "/> <!-- ${PI/2}  -->
+    <xacro:property name="Shoulder_1_pitch" value=" 0.0 "/> <!-- 0.0  -->
+    <xacro:property name="Shoulder_1_yaw" value=" 0.0 "/> <!-- 0.0  -->
     <!-- Origin -->
     <xacro:property name="Shoulder_2_Ox" value=" -0.06"/>

File: repair_urdf/urdf/repair_base.urdf.xacro (robot description, xacro)
@@ -4,25 +4,25 @@
         <!-- base -->
         <link name="base_link">
-            <!-- <inertial>
+            <inertial>
                 <origin xyz="${Base_x} ${rot*Base_y} ${Base_z}" />
                 <mass value="${Base_mass}" />
                 <inertia ixx="${Base_xx}" ixy="${rot*Base_xy}" ixz="${Base_xz}" iyy="${Base_yy}"
                     iyz="${rot*Base_yz}" izz="${Base_zz}" />
-            </inertial> -->
-            <!-- <visual> -->
-                <!-- <origin xyz="0.0 0.0 0.0" rpy="0.0 0.0 0.0" /> -->
-                <!-- <geometry> -->
-                    <!-- <mesh filename="package://inail2arm_urdf/meshes/mesh_base.stl" -->
-                        <!-- scale="0.001 ${rot*0.001} 0.001" /> -->
-                <!-- </geometry> -->
-                <!-- <material name="dark_grey" /> -->
-            <!-- </visual> -->
-            <!-- <collision> -->
-                <!-- <origin xyz="0.0 0.0 0.0" rpy="0.0 0.0 0.0" /> -->
-                <!-- <geometry> -->
-                    <!-- <mesh filename="package://inail2arm_urdf/meshes/simple/mesh_base.stl" -->
-                        <!-- scale="0.001 ${rot*0.001} 0.001" /> -->
-                <!-- </geometry> -->
-            <!-- </collision> -->
+            </inertial>
+            <visual>
+                <origin xyz="0.0 0.0 0.0" rpy="0.0 0.0 0.0" />
+                <geometry>
+                    <mesh filename="package://repair_urdf/meshes/mesh_base.stl"
+                        scale="0.001 ${rot*0.001} 0.001" />
+                </geometry>
+                <material name="dark_grey" />
+            </visual>
+            <collision>
+                <origin xyz="0.0 0.0 0.0" rpy="0.0 0.0 0.0" />
+                <geometry>
+                    <mesh filename="package://repair_urdf/meshes/simplified/mesh_base.stl"
+                        scale="0.001 ${rot*0.001} 0.001" />
+                </geometry>
+            </collision>
         </link>
         <!-- base -->

Commit message: added torso in joint_map

File: repair_urdf/urdf/kinematics_properties.urdf.xacro (robot description, xacro)
@@ -6,5 +6,5 @@
     <xacro:property name="Cage_leg_radius" value="0.02" />
     <xacro:property name="Cage_sliding_guide_width" value="0.2" />
-    <xacro:property name="Table_x" value="0.98" />
+    <xacro:property name="Table_x" value="0.0" />
     <xacro:property name="Table_y" value="0.0" />
     <xacro:property name="Table_z" value="0.0" />

Commit message: fixed cage
Signed-off-by: FrancescoRuscelli <francescoruscelli24@gmail.com>

File: repair_urdf/urdf/kinematics_properties.urdf.xacro (robot description, xacro)
@@ -1,21 +1,23 @@
 <!--<?xml version="1.0"?>-->
 <robot  xmlns:xacro="http://ros.org/wiki/xacro">
-    <xacro:property name="Cage_x" value="1.5" />
-    <xacro:property name="Cage_y" value="2.5" />
-    <xacro:property name="Cage_z" value="1.0"/>
-    <xacro:property name="Cage_leg_radius" value="0.02" />
-    <xacro:property name="Cage_sliding_guide_width" value="0.2" />
     <xacro:property name="Table_x" value="0.0" />
     <xacro:property name="Table_y" value="0.0" />
-    <xacro:property name="Table_z" value="0.0" />
+    <xacro:property name="Table_z" value="0.0" /> <!-- w.r.t world  -->
     <xacro:property name="table_top_thickness" value="0.05"/>
-    <xacro:property name="table_height" value="0.5"/>
-    <xacro:property name="sliding_guide_width" value="0.2"/>
+    <xacro:property name="table_height" value="1.0"/>
+    <xacro:property name="Cage_x" value="1.0" />
+    <xacro:property name="Cage_y" value="2.5" />
+    <xacro:property name="Cage_z" value="1.0"/> <!-- w.r.t table  -->
+    <xacro:property name="Cage_leg_radius" value="0.02" />
+    <xacro:property name="Cage_sliding_guide_x" value="0.0"/> <!-- w.r.t world  -->
+    <xacro:property name="Cage_sliding_guide_y" value="0.0"/> <!-- w.r.t world  -->
+    <xacro:property name="Cage_sliding_guide_z" value="0.0"/> <!-- w.r.t world  -->
+    <xacro:property name="Cage_sliding_guide_width" value="0.4"/>
     <xacro:property name="Torso_Ox" value=" 0.0 "/>
     <xacro:property name="Torso_Oy" value=" 0.0 "/>
     <xacro:property name="Torso_Oz" value=" 0.0 "/>
-    <xacro:property name="Torso_roll" value=" 0.0 "/>
-    <xacro:property name="Torso_pitch" value=" ${PI/2} "/>
-    <xacro:property name="Torso_yaw" value=" 0.0 "/>
+    <xacro:property name="Torso_roll" value=" ${PI/2} "/>
+    <xacro:property name="Torso_pitch" value=" 0.0 "/>
+    <xacro:property name="Torso_yaw" value=" ${PI/2}"/>
     <!-- Origin -->
     <xacro:property name="Shoulder_1_Ox" value=" 0.0 "/>  <!-- 0.0  -->

File: repair_urdf/urdf/repair_cage_macro.urdf.xacro (robot description, xacro)
@@ -264,5 +264,5 @@
   <joint name="sliding_guide_joint" type="fixed" >
     <parent link="obar2_link" />
-    <origin xyz="0 ${Cage_y/2} 0" rpy="-${PI_2} 0 0" />
+    <origin xyz="${Cage_sliding_guide_z} ${Cage_y/2 + Cage_sliding_guide_y} ${Cage_x/2 - Cage_sliding_guide_width/2 + Cage_sliding_guide_x}" rpy="-${PI_2} 0 0" />
     <child link="sliding_guide_link" />
   </joint>
@@ -271,5 +271,5 @@
       <origin xyz="0.0 0.0 0" rpy="0 0 0" />
       <geometry>
-        <box size="0.001 ${sliding_guide_width} ${Cage_y}" />
+        <box size="0.001 ${Cage_sliding_guide_width} ${Cage_y}" />
       </geometry>
     <material name="silver_gray" />

Commit message: updated joint configs and kinematics

File: repair_urdf/urdf/kinematics_properties.urdf.xacro (robot description, xacro)
@@ -8,5 +8,5 @@
     <xacro:property name="Cage_x" value="1.0" />
     <xacro:property name="Cage_y" value="2.5" />
-    <xacro:property name="Cage_z" value="1.0"/> <!-- w.r.t table  -->
+    <xacro:property name="Cage_z" value="0.97"/> <!-- w.r.t table  -->
     <xacro:property name="Cage_leg_radius" value="0.02" />
     <xacro:property name="Cage_sliding_guide_x" value="0.0"/> <!-- w.r.t world  -->

Commit message: higher mounting on top of the table and removing hands.

File: repair_urdf/urdf/kinematics_properties.urdf.xacro (robot description, xacro)
@@ -8,5 +8,5 @@
     <xacro:property name="Cage_x" value="1.0" />
     <xacro:property name="Cage_y" value="2.5" />
-    <xacro:property name="Cage_z" value="1.05"/> <!-- w.r.t table  -->
+    <xacro:property name="Cage_z" value="2.05"/> <!-- w.r.t table  -->
     <xacro:property name="Cage_leg_radius" value="0.02" />
     <xacro:property name="Cage_sliding_guide_x" value="0.0"/> <!-- w.r.t world  -->

File: repair_urdf/urdf/repair_full.urdf.xacro (robot description, xacro)
@@ -26,22 +26,4 @@
                 rpy="${-Shoulder_1_roll} ${Shoulder_1_pitch} ${Shoulder_1_yaw}" />
       </xacro:repair_arm>
-    <xacro:softhands type="left"
-        version="v1.0_simple"
-        parent="arm_1_7"
-        position="0.0 0.0 0.0"
-        orientation="0 0.0 ${PI/2}"
-        translation="0"
-        operation_mode="0"
-        fixed_hands="true">
-    </xacro:softhands>
-    <xacro:softhands type="right"
-        version="v1.0_simple"
-        parent="arm_2_7"
-        position="0.0 0.0 0.0"
-        orientation="0.0 0.0 ${-PI/2}"
-        translation="0"
-        operation_mode="0"
-        fixed_hands="true">
-    </xacro:softhands>
     <!-- <gazebo reference="table_top_link">
         <selfCollide> 1 </selfCollide>

Commit message: new Jan24 branch

File: repair_urdf/urdf/kinematics_properties.urdf.xacro (robot description, xacro)
@@ -4,9 +4,9 @@
     <xacro:property name="Table_y" value="0.0" />
     <xacro:property name="Table_z" value="0.0" /> <!-- w.r.t world  -->
-    <xacro:property name="table_top_thickness" value="0.03"/> <!-- w.r.t. top origin of table to down  -->
-    <xacro:property name="table_height" value="0.983"/> <!-- w.r.t. working surface of the table  -->
+    <xacro:property name="table_top_thickness" value="0.05"/>
+    <xacro:property name="table_height" value="1.0"/>
     <xacro:property name="Cage_x" value="1.0" />
     <xacro:property name="Cage_y" value="2.5" />
-    <xacro:property name="Cage_z" value="1.05"/> <!-- w.r.t table  -->
+    <xacro:property name="Cage_z" value="0.97"/> <!-- w.r.t table  -->
     <xacro:property name="Cage_leg_radius" value="0.02" />
     <xacro:property name="Cage_sliding_guide_x" value="0.0"/> <!-- w.r.t world  -->
@@ -14,5 +14,5 @@
     <xacro:property name="Cage_sliding_guide_z" value="0.0"/> <!-- w.r.t world  -->
     <xacro:property name="Cage_sliding_guide_width" value="0.4"/>
-    <xacro:property name="Torso_Ox" value=" -0.13 "/>
+    <xacro:property name="Torso_Ox" value=" 0.0 "/>
     <xacro:property name="Torso_Oy" value=" 0.0 "/>
     <xacro:property name="Torso_Oz" value=" 0.0 "/>

File: repair_urdf/urdf/repair_arm_macro.urdf.xacro (robot description, xacro)
@@ -154,4 +154,11 @@
             </inertial>
         </link>
+        <link name="arm_${id}_tcp_joi">
+            <inertial>
+		<origin xyz="0.0 0.05 0.1" />
+                <mass value="0.5" />
+                <inertia ixx="0.001" ixy="0.0" ixz="0.0" iyy="0.001" iyz="0.0" izz="0.001" />
+            </inertial>
+        </link>
         <!-- JOINTS -->
         <!-- shoulder pitch -->
@@ -239,4 +246,12 @@
         </joint>
         <!-- virtual tip-->
+	<!-- virtual tip-->
+        <joint name="j_tcp_${id}_joi" type="fixed">
+            <parent link="arm_${id}_tcp" />
+            <child link="arm_${id}_tcp_joi" />
+            <origin xyz="${No_end_ft_Ox} ${rot*No_end_ft_Oy} ${No_end_ft_Oz}"
+            rpy="3.14 0 0" />
+        </joint>
+        <!-- virtual tip-->
     </xacro:macro>
 </robot>

File: repair_urdf/urdf/repair_cage_macro.urdf.xacro (robot description, xacro)
@@ -10,10 +10,10 @@
       <material name="wood" />
     </visual>
-    <!-- <collision>
+    <collision>
       <origin xyz="${Table_x} ${Table_y} ${Table_z+table_height-table_top_thickness/2}" />
       <geometry>
         <box size="${Cage_x} ${Cage_y} ${table_top_thickness}" />
       </geometry>
-    </collision> -->
+    </collision>
   </link>
   <joint name="table_top_link_joint" type="fixed" >
