Commit message: added dummy sliding guide

File: repair_urdf/urdf/repair_torso_macro.urdf.xacro (robot description, xacro)
@@ -2,5 +2,13 @@
 <robot xmlns:xacro="http://ros.org/wiki/xacro">
     <xacro:macro name="repair_torso" params="parent *origin">
-        <!-- <link name="dummy_prismatic_link"/> -->
+        <joint name="j_sliding_guide" type="prismatic">
+            <parent link="${parent}" />
+            <origin xyz="0 0 0" rpy="0 0 0"/>
+            <child link="dummy_prismatic_link"/>
+            <axis xyz="0 0 -1"/>
+            <limit lower="${j_prismatic_lower[0]/2}" upper= "${j_prismatic_upper[0]/2}" effort="${j_prismatic_torque[0]}" velocity="${j_prismatic_velocity[0]}"/>
+        </joint>
+        <link name="dummy_prismatic_link">
+        </link>
         <link name="torso_1">
             <inertial>
@@ -22,14 +30,7 @@
             </collision>
         </link>
-        <!-- <joint name="j_torso_base" type="fixed">
-            <xacro:insert_block name="origin" />
-            <parent link="${parent}" />
-            <child link="dummy_prismatic_link"/>
-            <axis xyz="0 0 1"/>
-            <limit lower="${j_prismatic_lower[0]/2}" upper= "${j_prismatic_upper[0]/2}" effort="${j_prismatic_torque[0]}" velocity="${j_prismatic_velocity[0]}"/>
-        </joint> -->
         <!-- torso -->
         <joint name="j_torso_1" type="revolute">
-            <parent link="${parent}" />
+            <parent link="dummy_prismatic_link" />
             <child link="torso_1" />
             <axis xyz="0 0 1" />
