Commit message: small ws limit update

File: repair_urdf/urdf/repair_full.urdf (robot description, URDF)
Before this commit: robot repair_full, 51 links, 50 joints
Links:
- link arm_1_link5_coll: geometry visual sphere radius=0.06
- link arm_2_link5_coll: geometry visual sphere radius=0.06
- link base_link: geometry 

File: repair_urdf/urdf/repair_full.urdf.xacro (robot description, xacro)
@@ -37,27 +37,4 @@
                   izz="0" />
         </inertial>
-        <xacro:if value="$(arg gen_coll)">
-            <visual name="link0_coll_visual1">
-                <origin xyz="0 0 0" rpy="0 0 0"/>
-                <geometry>
-                    <sphere radius="${coll_radius_link1}"/>
-                </geometry>
-                <material name="darkred"/>
-            </visual>
-            <visual name="link0_coll_visual2">
-                <origin xyz="0 ${link2_coll_offset_y} 0" rpy="0 0 0"/>
-                <geometry>
-                    <sphere radius="${coll_radius_link1}"/>
-                </geometry>
-                <material name="darkred"/>
-            </visual>
-            <visual name="link0_coll_visual3">
-                <origin xyz="0 ${- link2_coll_offset_y} 0" rpy="0 0 0"/>
-                <geometry>
-                    <sphere radius="${coll_radius_link1}"/>
-                </geometry>
-                <material name="darkred"/>
-            </visual>
-        </xacro:if>
         <xacro:if value="$(arg use_updated_wrist)">
             <visual name="base_link_visual">
@@ -127,27 +104,4 @@
                     izz="0" />
           </inertial>
-          <xacro:if value="$(arg gen_coll)">
-            <visual name="link0_coll_visual1">
-                <origin xyz="0 0 0" rpy="0 0 0"/>
-                <geometry>
-                    <sphere radius="${coll_radius_link1}"/>
-                </geometry>
-                <material name="darkred"/>
-            </visual>
-            <visual name="link0_coll_visual2">
-                <origin xyz="0 ${link2_coll_offset_y} 0" rpy="0 0 0"/>
-                <geometry>
-                    <sphere radius="${coll_radius_link1}"/>
-                </geometry>
-                <material name="darkred"/>
-            </visual>
-            <visual name="link0_coll_visual3">
-                <origin xyz="0 ${- link2_coll_offset_y} 0" rpy="0 0 0"/>
-                <geometry>
-                    <sphere radius="${coll_radius_link1}"/>
-                </geometry>
-                <material name="darkred"/>
-            </visual>
-        </xacro:if>
         <xacro:if value="$(arg use_updated_wrist)">
             <visual name="base_link_visual">

Commit message: task improvs and static torque cost addition

File: repair_urdf/urdf/repair_full.urdf (robot description, URDF)
Before this commit: robot repair_full, 51 links, 50 joints
Links:
- added link dummy_link
- added link dummy_sliding_wrist1_link
- added link dummy_sliding_wrist2_link
- link l_arm_mount_frame: mass 1.00000000000001e-06 -> None
- link r_arm_mount_frame: mass 1.00000000000001e-06 -> None
Joints:
- added joint dummy_sliding_wrist1_joint: type prismatic, parent dummy_sliding_wrist1_link, child arm_1_link_6, origin xyz=0.0 0.0 0.0 rpy=0 0 0, axis 0 0 -1, limit lower=0 upper=0.1 effort=1000.0 velocity=20.0
- added joint dummy_sliding_wrist2_joint: type prismatic, parent dummy_sliding_wrist2_link, child arm_2_link_6, origin xyz=0.0 0.0 0.0 rpy=0 0 0, axis 0 0 -1, limit lower=0 upper=0.1 effort=1000.0 velocity=20.0
- added joint z_joint: type prismatic, parent dummy_link, child base_link, origin xyz=0.0 0.0 0.0 rpy=0.0 0.0 0.0, axis 0 0 1, limit lower=0.3 upper=2 effort=1000.0 velocity=20.0
- joint arm_1_joint_6: child arm_1_link_6 -> dummy_sliding_wrist1_link; origin xyz=0.096 0.321 0 rpy=0 -1.57079632679 0 -> xyz=0 0.0 0.321  rpy=0 -1.57079632679 0
- joint arm_1_link_5_coll_joint: axis (none) -> 1 0 0; limit (none) -> lower=0 upper=0.1 effort=200.0 velocity=10.0; origin xyz=-0.004109236058802465 0.0 0.321 rpy=0 0 0 -> xyz=-0.1 0.0 0.321 rpy=0 0 0; type fixed -> prismatic
- joint arm_2_joint_6: child arm_2_link_6 -> dummy_sliding_wrist2_link; origin xyz=0.096 0.321 0 rpy=0 -1.57079632679 0 -> xyz=0 0.0 0.321  rpy=0 -1.57079632679 0
- joint arm_2_link_5_coll_joint: axis (none) -> 1 0 0; limit (none) -> lower=0 upper=0.1 effort=200.0 velocity=10.0; origin xyz=-0.004109236058802465 0.0 0.321 rpy=0 0 0 -> xyz=-0.1 0.0 0.321 rpy=0 0 0; type fixed -> prismatic
- joint l_arm_mount_joint: axis (none) -> 0 1 0; limit (none) -> lower=0.21 upper=0.5 effort=1000.0 velocity=20.0; origin xyz=0.0 0.2942172496425824 0.0 rpy=0 0 0 -> xyz=0.0 0.0 0.0 rpy=0 0 0; type fixed -> prismatic
- joint r_arm_mount_joint: axis (none) -> 0 -1 0; limit (none) -> lower=0.21 upper=0.5 effort=1000.0 velocity=20.0; origin xyz=0.0 -0.2942172496425824 0.0 rpy=0 0 0 -> xyz=0.0 0.0 0.0 rpy=0 0 0; type fixed -> prismatic
- joint roll_l: axis (none) -> -1 0 0; limit (none) -> lower=-1.047197551196598 upper=1.57079632679 effort=0.0 velocity=0.0; origin xyz=0 0.0 0.0 rpy=-0.09051373592070662 0.0 0.0 -> xyz=0.0 0.0 0.0 rpy=0.0 0.0 0.0; type fixed -> revolute
- joint roll_r: axis (none) -> 1 0 0; limit (none) -> lower=-1.047197551196598 upper=1.57079632679 effort=0.0 velocity=0.0; origin xyz=0 0.0 0.0 rpy=0.09051373592070662 0.0 0.0 -> xyz=0.0 0.0 0.0 rpy=0.0 0.0 0.0; type fixed -> revolute
- joint x_joint: child base_link -> dummy_link; origin xyz=0.0 0.0 0.3034329527232317 rpy=0.0 0.0 0.0 -> xyz=0.0 0.0 0.0 rpy=0.0 0.0 0.0

Commit message: added pre-generated urdf with sliding guide

File: repair_urdf/urdf/repair_full.urdf (robot description, URDF)
Before this commit: robot repair_full, 76 links, 75 joints
Links:
- added link arm_1_tcp_joi, mass 0.5
- added link arm_2_tcp_joi, mass 0.5
- link leg1_link: geometry collision cylinder length=1.0 radius=0.02; visual cylinder length=1.0 radius=0.02
- link leg2_link: geometry collision cylinder length=1.0 radius=0.02; visual cylinder length=1.0 radius=0.02
- link leg3_link: geometry collision cylinder length=1.0 radius=0.02; visual cylinder length=1.0 radius=0.02
- link leg4_link: geometry collision cylinder length=1.0 radius=0.02; visual cylinder length=1.0 radius=0.02
- link table_top_link: geometry collision box size=1.0 2.5 0.05; visual box size=1.0 2.5 0.05
- link vbar1_link: geometry collision cylinder length=0.97 radius=0.02; visual cylinder length=0.97 radius=0.02
- link vbar2_link: geometry collision cylinder length=0.97 radius=0.02; visual cylinder length=0.97 radius=0.02
- link vbar3_link: geometry collision cylinder length=0.97 radius=0.02; visual cylinder length=0.97 radius=0.02
- link vbar4_link: geometry collision cylinder length=0.97 radius=0.02; visual cylinder length=0.97 radius=0.02
Joints:
- added joint j_tcp_1_joi: type fixed, parent arm_1_tcp, child arm_1_tcp_joi, origin xyz=0.0 -0.0 0.0 rpy=3.14 0 0
- added joint j_tcp_2_joi: type fixed, parent arm_2_tcp, child arm_2_tcp_joi, origin xyz=0.0 0.0 0.0 rpy=3.14 0 0
- joint j_torso_1: origin xyz=-0.13 0.0 0.0 rpy=1.570796326795 0.0 1.570796326795 -> xyz=0.0 0.0 0.0 rpy=1.570796326795 0.0 1.570796326795
- joint leg1_joint: origin xyz=0.5 1.25 0.983 rpy=0 0 0 -> xyz=0.5 1.25 1.0 rpy=0 0 0
- joint leg2_joint: origin xyz=-0.5 1.25 0.983 rpy=0 0 0 -> xyz=-0.5 1.25 1.0 rpy=0 0 0
- joint leg3_joint: origin xyz=0.5 -1.25 0.983 rpy=0 0 0 -> xyz=0.5 -1.25 1.0 rpy=0 0 0
- joint leg4_joint: origin xyz=-0.5 -1.25 0.983 rpy=0 0 0 -> xyz=-0.5 -1.25 1.0 rpy=0 0 0
- joint obar1_joint: origin xyz=-0.5 0 0.525 rpy=0 -1.57079632679 0 -> xyz=-0.5 0 0.485 rpy=0 -1.57079632679 0
- joint obar2_joint: origin xyz=-0.5 0 0.525 rpy=0 -1.57079632679 0 -> xyz=-0.5 0 0.485 rpy=0 -1.57079632679 0
- joint obar3_joint: origin xyz=0 1.25 0.525 rpy=-1.57079632679 0 0 -> xyz=0 1.25 0.485 rpy=-1.57079632679 0 0
- joint obar4_joint: origin xyz=0 1.25 0.525 rpy=-1.57079632679 0 0 -> xyz=0 1.25 0.485 rpy=-1.57079632679 0 0
- joint vbar1_joint: origin xyz=0 0 0.525 rpy=0 0 0 -> xyz=0 0 0.485 rpy=0 0 0
- joint vbar2_joint: origin xyz=0 0 0.525 rpy=0 0 0 -> xyz=0 0 0.485 rpy=0 0 0
- joint vbar3_joint: origin xyz=0 0 0.525 rpy=0 0 0 -> xyz=0 0 0.485 rpy=0 0 0
- joint vbar4_joint: origin xyz=0 0 0.525 rpy=0 0 0 -> xyz=0 0 0.485 rpy=0 0 0
- joint working_surface_joint: origin xyz=-1.05 0 0 rpy=0.0 -1.57079632679 3.14159265359 -> xyz=-0.97 0 0 rpy=0.0 -1.57079632679 3.14159265359

Commit message: temporarily removed sliding guide joint

File: repair_urdf/urdf/repair_full.urdf (robot description, URDF)
Before this commit: robot repair_full, 78 links, 77 joints
Links:
- removed link dummy_prismatic_link
Joints:
- removed joint j_sliding_guide
- joint j_torso_1: parent dummy_prismatic_link -> sliding_guide_link
