Commit message: configs for second arm

File: repair_srdf/srdf/repair.srdf.xacro (robot description, xacro)
@@ -9,10 +9,18 @@
     </group>
     <group_state group="chains" name="home">
-        <joint name="arm_1_joint_2" value="-0.40"/>
-        <joint name="arm_1_joint_4" value="-1.40"/>
-        <joint name="arm_1_joint_6" value="-1.40"/>
-        <joint name="arm_2_joint_2" value="-0.40"/>
-        <joint name="arm_2_joint_4" value="-1.40"/>
-        <joint name="arm_2_joint_6" value="-1.40"/>
+        <joint name="j_arm_1_1" value="0.0"/>
+        <joint name="j_arm_1_2" value="-1.0"/>
+        <joint name="j_arm_1_3" value="1.5"/>
+        <joint name="j_arm_1_4" value="-1.0"/>
+        <joint name="j_arm_1_5" value="0.0"/>
+        <joint name="j_arm_1_6" value="0.5"/>
+        <joint name="j_arm_1_7" value="0.5"/>
+        <joint name="j_arm_2_1" value="0.0"/>
+        <joint name="j_arm_2_2" value="-1.0"/>
+        <joint name="j_arm_2_3" value="1.5"/>
+        <joint name="j_arm_2_4" value="-1.0"/>
+        <joint name="j_arm_2_5" value="0.0"/>
+        <joint name="j_arm_2_6" value="0.5"/>
+        <joint name="j_arm_2_7" value="0.5"/>
     </group_state>
 </robot>

File: repair_urdf/urdf/gazebo/xbot.gazebo.xacro (robot description, xacro)
@@ -7,5 +7,5 @@
             <gain name="small_mot"  p="1000"  d="10"/>
             <gain name="medium_mot" p="2000" d="20"/>
-            <pid name="j_arm_1_1" profile="medium_mot"/>
+            <!-- <pid name="j_arm_1_1" profile="medium_mot"/>
             <pid name="j_arm_1_2" profile="medium_mot"/>
             <pid name="j_arm_1_3" profile="medium_mot"/>
@@ -13,6 +13,6 @@
             <pid name="j_arm_1_5" profile="small_mot"/>
             <pid name="j_arm_1_6" profile="small_mot"/>
-            <pid name="j_arm_1_7" profile="small_mot"/>
-            <!-- <pid name="j_arm_2_1" profile="medium_mot"/>
+            <pid name="j_arm_1_7" profile="small_mot"/> -->
+            <pid name="j_arm_2_1" profile="medium_mot"/>
             <pid name="j_arm_2_2" profile="medium_mot"/>
             <pid name="j_arm_2_3" profile="medium_mot"/>
@@ -20,5 +20,5 @@
             <pid name="j_arm_2_5" profile="small_mot"/>
             <pid name="j_arm_2_6" profile="small_mot"/>
-            <pid name="j_arm_2_7" profile="small_mot"/> -->
+            <pid name="j_arm_2_7" profile="small_mot"/>
         </pid>
     </plugin>

File: repair_urdf/urdf/limits.urdf.xacro (robot description, xacro)
@@ -4,20 +4,20 @@
     <xacro:property name="j_prismatic_lower" value="${[2]}"/>
     <xacro:property name="j_torso_lower" value="${[-2.6]}"/>
-    <xacro:property name="j_arm_1_lower" value="${[-2.6]}"/>
-    <xacro:property name="j_arm_2_lower" value="${[-2.5]}"/>
-    <xacro:property name="j_arm_3_lower" value="${[-2.6]}"/>
-    <xacro:property name="j_arm_4_lower" value="${[-2.4]}"/>
-    <xacro:property name="j_arm_5_lower" value="${[-2.8]}"/>
-    <xacro:property name="j_arm_6_lower" value="${[-2.8]}"/>
-    <xacro:property name="j_arm_7_lower" value="${[-2.8]}"/>
+    <xacro:property name="j_arm_1_lower" value="${[-2.6, -2.6]}"/>
+    <xacro:property name="j_arm_2_lower" value="${[-0.1, -2.5]}"/>
+    <xacro:property name="j_arm_3_lower" value="${[-2.6, 2.6]}"/>
+    <xacro:property name="j_arm_4_lower" value="${[-0.8, -2.4]}"/>
+    <xacro:property name="j_arm_5_lower" value="${[-2.8, -2.8]}"/>
+    <xacro:property name="j_arm_6_lower" value="${[-2.8, -2.1]}"/>
+    <xacro:property name="j_arm_7_lower" value="${[-2.8, -2.8]}"/>
     <xacro:property name="j_prismatic_upper" value="${[-2]}"/>
     <xacro:property name="j_torso_upper" value="${[2.6]}"/>
-    <xacro:property name="j_arm_1_upper" value="${[2.6]}"/>
-    <xacro:property name="j_arm_2_upper" value="${[0.1]}"/>
-    <xacro:property name="j_arm_3_upper" value="${[2.6]}"/>
-    <xacro:property name="j_arm_4_upper" value="${[0.8]}"/>
-    <xacro:property name="j_arm_5_upper" value="${[2.8]}"/>
-    <xacro:property name="j_arm_6_upper" value="${[2.1]}"/>
-    <xacro:property name="j_arm_7_upper" value="${[2.8]}"/>
+    <xacro:property name="j_arm_1_upper" value="${[2.6, 2.6]}"/>
+    <xacro:property name="j_arm_2_upper" value="${[2.5, 0.1]}"/>
+    <xacro:property name="j_arm_3_upper" value="${[2.6, 2.6]}"/>
+    <xacro:property name="j_arm_4_upper" value="${[2.4, 0.8]}"/>
+    <xacro:property name="j_arm_5_upper" value="${[2.8, 2.8]}"/>
+    <xacro:property name="j_arm_6_upper" value="${[2.1, 2.8]}"/>
+    <xacro:property name="j_arm_7_upper" value="${[2.8, 2.8]}"/>
     <xacro:property name="j_prismatic_velocity" value="${[-5]}"/>
     <xacro:property name="j_torso_velocity" value="${[3.86]}"/>

File: repair_urdf/urdf/repair_arm_final.urdf.xacro (robot description, xacro)
@@ -10,8 +10,8 @@
     <xacro:include filename="$(find repair_urdf)/urdf/gazebo/xbot.gazebo.xacro" />
     <link name="world"/>
-    <xacro:repair_base rot="1" parent="world">
+    <xacro:repair_base parent="world">
       <origin xyz="0 0 0" rpy="0 0 0"/>
     </xacro:repair_base>
-    <xacro:repair_arm id="1"  rot="1"  parent="base_link">
+    <xacro:repair_arm id="2"  rot="1"  parent="base_link">
       <origin xyz="0.0 0.0 0.14"
               rpy="0.0 0.0 0.0" />

File: repair_urdf/urdf/repair_arm_macro.urdf.xacro (robot description, xacro)
@@ -10,4 +10,8 @@
 results of the optimization), otherwise we go with the old ones (generated for a spherical wrist) -->
     <xacro:macro name="repair_arm" params="id rot parent *origin">
+        <xacro:property name="limit_index" value="0" />
+        <xacro:if value="${rot == -1}">
+            <xacro:property name="limit_index" value="1" />
+        </xacro:if>
         <link name="arm_${id}_1">
             <inertial>
@@ -157,6 +161,6 @@
             <axis xyz="0 0 1" />
             <xacro:insert_block name="origin" />
-            <limit lower="${j_arm_1_lower[0]}" upper="${j_arm_1_upper[0]}"
-            effort="${j_arm_1_torque[0]}" velocity="${j_arm_1_velocity[0]}" />
+            <limit lower="${j_arm_1_lower[limit_index]}" upper="${j_arm_1_upper[limit_index]}"
+            effort="${j_arm_1_torque[limit_index]}" velocity="${j_arm_1_velocity[limit_index]}" />
         </joint>
         <!-- shoulder pitch -->
@@ -167,6 +171,6 @@
             <origin xyz="${Shoulder_2_Ox} ${rot*Shoulder_2_Oy} ${Shoulder_2_Oz}"
             rpy="${rot*Shoulder_2_roll} ${Shoulder_2_pitch} ${Shoulder_2_yaw}" />
-            <axis xyz="0 0 -1" />
-            <limit lower="${j_arm_2_lower[0]}" upper="${j_arm_2_upper[0]}"
+            <axis xyz="0 0 1" /> <!-- -1 -->
+            <limit lower="${j_arm_2_lower[limit_index]}" upper="${rot*j_arm_2_upper[limit_index]}"
             effort="${j_arm_2_torque[0]}" velocity="${j_arm_2_velocity[0]}" />
         </joint>
@@ -178,6 +182,6 @@
             <origin xyz="${Shoulder_3_Ox} ${rot*Shoulder_3_Oy} ${Shoulder_3_Oz}"
             rpy="${rot*Shoulder_3_roll} ${Shoulder_3_pitch} ${Shoulder_3_yaw}" />
-            <axis xyz="0 0 -1" />
-            <limit lower="${j_arm_3_lower[0]}" upper="${j_arm_3_upper[0]}"
+            <axis xyz="0 0 -1" /> <!-- -1 -->
+            <limit lower="${j_arm_3_lower[limit_index]}" upper="${j_arm_3_upper[limit_index]}"
             effort="${j_arm_3_torque[0]}" velocity="${j_arm_3_velocity[0]}" />
         </joint>
@@ -189,6 +193,6 @@
             <origin xyz="${Elbow_1_Ox} ${rot*Elbow_1_Oy} ${Elbow_1_Oz}"
             rpy="${rot*Elbow_1_roll} ${Elbow_1_pitch} ${Elbow_1_yaw}" />
-            <axis xyz="0 0 -1" />
-            <limit lower="${j_arm_4_lower[0]}" upper="${j_arm_4_upper[0]}"
+            <axis xyz="0 0 1" /> <!-- -1 -->
+            <limit lower="${j_arm_4_lower[limit_index]}" upper="${j_arm_4_upper[limit_index]}"
             effort="${j_arm_4_torque[0]}" velocity="${j_arm_4_velocity[0]}" />
         </joint>
@@ -200,6 +204,6 @@
             <origin xyz="${Forearm_1_Ox} ${rot*Forearm_1_Oy} ${Forearm_1_Oz}"
             rpy="${rot*Forearm_1_roll} ${Forearm_1_pitch} ${Forearm_1_yaw}" />
-            <axis xyz="0 0 -1" />
-            <limit lower="${j_arm_5_lower[0]}" upper="${j_arm_5_upper[0]}"
+            <axis xyz="0 0 -1" /> <!-- -1 -->
+            <limit lower="${j_arm_5_lower[limit_index]}" upper="${j_arm_5_upper[limit_index]}"
             effort="${j_arm_5_torque[0]}" velocity="${j_arm_5_velocity[0]}" />
         </joint>
@@ -212,5 +216,5 @@
             rpy="${rot*Wrist_1_roll} ${Wrist_1_pitch} ${Wrist_1_yaw}" />
             <axis xyz="0 0 1" />
-            <limit lower="${j_arm_6_lower[0]}" upper="${j_arm_6_upper[0]}"
+            <limit lower="${j_arm_6_lower[limit_index]}" upper="${j_arm_6_upper[limit_index]}"
             effort="${j_arm_6_torque[0]}" velocity="${j_arm_6_velocity[0]}" />
         </joint>
@@ -223,5 +227,5 @@
             rpy="${rot*Wrist_2_roll} ${Wrist_2_pitch} ${Wrist_2_yaw}" />
             <axis xyz="0 0 1" />
-            <limit lower="${j_arm_7_lower[0]}" upper="${j_arm_7_upper[0]}"
+            <limit lower="${j_arm_7_lower[limit_index]}" upper="${j_arm_7_upper[limit_index]}"
             effort="${j_arm_7_torque[0]}" velocity="${j_arm_7_velocity[0]}" />
         </joint>

File: repair_urdf/urdf/repair_base.urdf.xacro (robot description, xacro)
@@ -1,12 +1,12 @@
 <?xml version="1.0"?>
 <robot xmlns:xacro="http://ros.org/wiki/xacro">
-    <xacro:macro name="repair_base" params="rot parent *origin">
+    <xacro:macro name="repair_base" params="parent *origin">
         <!-- base -->
         <link name="base_link">
             <inertial>
-                <origin xyz="${Base_x} ${rot*Base_y} ${Base_z}" />
+                <origin xyz="${Base_x} ${Base_y} ${Base_z}" />
                 <mass value="${Base_mass}" />
-                <inertia ixx="${Base_xx}" ixy="${rot*Base_xy}" ixz="${Base_xz}" iyy="${Base_yy}"
-                    iyz="${rot*Base_yz}" izz="${Base_zz}" />
+                <inertia ixx="${Base_xx}" ixy="${Base_xy}" ixz="${Base_xz}" iyy="${Base_yy}"
+                    iyz="${Base_yz}" izz="${Base_zz}" />
             </inertial>
             <visual>
@@ -14,5 +14,5 @@
                 <geometry>
                     <mesh filename="package://repair_urdf/meshes/mesh_base.stl"
-                        scale="0.001 ${rot*0.001} 0.001" />
+                        scale="0.001 0.001 0.001" />
                 </geometry>
                 <material name="dark_grey" />
@@ -22,5 +22,5 @@
                 <geometry>
                     <mesh filename="package://repair_urdf/meshes/simplified/mesh_base.stl"
-                        scale="0.001 ${rot*0.001} 0.001" />
+                        scale="0.001 0.001 0.001" />
                 </geometry>
             </collision>

Commit message: repair full added

File: repair_srdf/srdf/repair.srdf.xacro (robot description, xacro)
@@ -2,6 +2,6 @@
 <robot name="repair">
     <group name="arm">
-        <chain base_link="base_link" tip_link="arm_1_tcp"/>
-        <chain base_link="base_link" tip_link="arm_2_tcp"/>
+        <chain base_link="torso_1" tip_link="arm_1_tcp"/>
+        <chain base_link="torso_1" tip_link="arm_2_tcp"/>
     </group>
     <group name="chains">
@@ -9,16 +9,16 @@
     </group>
     <group_state group="chains" name="home">
-        <joint name="j_arm_1_1" value="0.0"/>
-        <joint name="j_arm_1_2" value="-1.0"/>
-        <joint name="j_arm_1_3" value="1.5"/>
-        <joint name="j_arm_1_4" value="-1.0"/>
-        <joint name="j_arm_1_5" value="0.0"/>
+        <joint name="j_arm_1_1" value="-0.5"/>
+        <joint name="j_arm_1_2" value="-0.5"/>
+        <joint name="j_arm_1_3" value="-1.5"/>
+        <joint name="j_arm_1_4" value="1.0"/>
+        <joint name="j_arm_1_5" value="1.5"/>
         <joint name="j_arm_1_6" value="0.5"/>
         <joint name="j_arm_1_7" value="0.5"/>
-        <joint name="j_arm_2_1" value="0.0"/>
-        <joint name="j_arm_2_2" value="-1.0"/>
+        <joint name="j_arm_2_1" value="0.5"/>
+        <joint name="j_arm_2_2" value="-0.5"/>
         <joint name="j_arm_2_3" value="1.5"/>
         <joint name="j_arm_2_4" value="-1.0"/>
-        <joint name="j_arm_2_5" value="0.0"/>
+        <joint name="j_arm_2_5" value="-1.5"/>
         <joint name="j_arm_2_6" value="0.5"/>
         <joint name="j_arm_2_7" value="0.5"/>

File: repair_urdf/urdf/limits.urdf.xacro (robot description, xacro)
@@ -2,14 +2,14 @@
 <robot  xmlns:xacro="http://ros.org/wiki/xacro">
     <!-- Origin -->
-    <xacro:property name="j_prismatic_lower" value="${[2]}"/>
+    <xacro:property name="j_prismatic_lower" value="${[-2]}"/>
     <xacro:property name="j_torso_lower" value="${[-2.6]}"/>
     <xacro:property name="j_arm_1_lower" value="${[-2.6, -2.6]}"/>
     <xacro:property name="j_arm_2_lower" value="${[-0.1, -2.5]}"/>
-    <xacro:property name="j_arm_3_lower" value="${[-2.6, 2.6]}"/>
+    <xacro:property name="j_arm_3_lower" value="${[-2.6, -2.6]}"/>
     <xacro:property name="j_arm_4_lower" value="${[-0.8, -2.4]}"/>
     <xacro:property name="j_arm_5_lower" value="${[-2.8, -2.8]}"/>
     <xacro:property name="j_arm_6_lower" value="${[-2.8, -2.1]}"/>
     <xacro:property name="j_arm_7_lower" value="${[-2.8, -2.8]}"/>
-    <xacro:property name="j_prismatic_upper" value="${[-2]}"/>
+    <xacro:property name="j_prismatic_upper" value="${[2]}"/>
     <xacro:property name="j_torso_upper" value="${[2.6]}"/>
     <xacro:property name="j_arm_1_upper" value="${[2.6, 2.6]}"/>
@@ -20,5 +20,5 @@
     <xacro:property name="j_arm_6_upper" value="${[2.1, 2.8]}"/>
     <xacro:property name="j_arm_7_upper" value="${[2.8, 2.8]}"/>
-    <xacro:property name="j_prismatic_velocity" value="${[-5]}"/>
+    <xacro:property name="j_prismatic_velocity" value="${[5]}"/>
     <xacro:property name="j_torso_velocity" value="${[3.86]}"/>
     <xacro:property name="j_arm_1_velocity" value="${[3.86]}"/>

File: repair_urdf/urdf/repair_arm_macro.urdf.xacro (robot description, xacro)
@@ -162,5 +162,5 @@
             <xacro:insert_block name="origin" />
             <limit lower="${j_arm_1_lower[limit_index]}" upper="${j_arm_1_upper[limit_index]}"
-            effort="${j_arm_1_torque[limit_index]}" velocity="${j_arm_1_velocity[limit_index]}" />
+            effort="${j_arm_1_torque[0]}" velocity="${j_arm_1_velocity[0]}" />
         </joint>
         <!-- shoulder pitch -->
@@ -172,5 +172,5 @@
             rpy="${rot*Shoulder_2_roll} ${Shoulder_2_pitch} ${Shoulder_2_yaw}" />
             <axis xyz="0 0 1" /> <!-- -1 -->
-            <limit lower="${j_arm_2_lower[limit_index]}" upper="${rot*j_arm_2_upper[limit_index]}"
+            <limit lower="${j_arm_2_lower[limit_index]}" upper="${j_arm_2_upper[limit_index]}"
             effort="${j_arm_2_torque[0]}" velocity="${j_arm_2_velocity[0]}" />
         </joint>
