Commit message: changed arm order

File: repair_srdf/srdf/repair.srdf.xacro (robot description, xacro)
@@ -1,26 +1,190 @@
-<?xml version="1.0" encoding="utf-8"?>
-<robot name="repair">
-    <group name="arm">
+<?xml version="1.0" encoding="UTF-8"?>
+<robot name="repair_full">
+    <group name="sliding_guide">
+        <chain base_link="sliding_guide_link" tip_link="torso_1"/>
+    </group>
+    <group name="arm1">
         <chain base_link="torso_1" tip_link="arm_1_tcp"/>
+    </group>
+    <group name="arm2">
         <chain base_link="torso_1" tip_link="arm_2_tcp"/>
     </group>
     <group name="chains">
-        <group name="arm"/>
+        <group name="sliding_guide" />
+        <group name="arm1"/>
+        <group name="arm2"/>
     </group>
-    <group_state group="chains" name="home">
-        <joint name="j_arm_1_1" value="-0.5"/>
-        <joint name="j_arm_1_2" value="-0.5"/>
-        <joint name="j_arm_1_3" value="-1.5"/>
+    <!--GROUP STATES: Purpose: Define a named state for a particular group, in terms of joint values. This is useful to define states like 'folded arms'-->
+    <group_state name="home" group="chains">
+        <joint name="j_arm_1_1" value="0.5"/>
+        <joint name="j_arm_1_2" value="0.5"/>
+        <joint name="j_arm_1_3" value="-0.5"/>
         <joint name="j_arm_1_4" value="1.0"/>
-        <joint name="j_arm_1_5" value="1.5"/>
+        <joint name="j_arm_1_5" value="0.5"/>
         <joint name="j_arm_1_6" value="0.5"/>
-        <joint name="j_arm_1_7" value="0.5"/>
-        <joint name="j_arm_2_1" value="0.5"/>
+        <joint name="j_arm_1_7" value="1.0"/>
+        <joint name="j_arm_2_1" value="-0.5"/>
         <joint name="j_arm_2_2" value="-0.5"/>
-        <joint name="j_arm_2_3" value="1.5"/>
+        <joint name="j_arm_2_3" value="0.5"/>
         <joint name="j_arm_2_4" value="-1.0"/>
-        <joint name="j_arm_2_5" value="-1.5"/>
-        <joint name="j_arm_2_6" value="0.5"/>
-        <joint name="j_arm_2_7" value="0.5"/>
+        <joint name="j_arm_2_5" value="-0.5"/>
+        <joint name="j_arm_2_6" value="-0.5"/>
+        <joint name="j_arm_2_7" value="-1.0"/>
     </group_state>
+    <!-- DISABLE COLLISIONS: By default it is assumed that any link of the robot could potentially come into collision with any other link in the robot. This tag disables collision checking between a specified pair of links. -->
+    <!-- <disable_collisions link1="arm_1_link_1" link2="arm_1_link_2" reason="Adjacent"/>
+    <disable_collisions link1="arm_1_link_1" link2="arm_1_link_3" reason="Never"/>
+    <disable_collisions link1="arm_1_link_1" link2="arm_1_link_4" reason="Never"/>
+    <disable_collisions link1="arm_1_link_1" link2="arm_2_link_1" reason="Adjacent"/>
+    <disable_collisions link1="arm_1_link_1" link2="arm_2_link_2" reason="Never"/>
+    <disable_collisions link1="arm_1_link_1" link2="arm_2_link_3" reason="Never"/>
+    <disable_collisions link1="arm_1_link_1" link2="arm_2_link_4" reason="Never"/>
+    <disable_collisions link1="arm_1_link_1" link2="arm_2_link_5" reason="Never"/>
+    <disable_collisions link1="arm_1_link_1" link2="arm_2_link_7" reason="Never"/>
+    <disable_collisions link1="arm_1_link_2" link2="arm_1_link_3" reason="Adjacent"/>
+    <disable_collisions link1="arm_1_link_2" link2="arm_1_link_4" reason="Never"/>
+    <disable_collisions link1="arm_1_link_2" link2="arm_2_link_1" reason="Never"/>
+    <disable_collisions link1="arm_1_link_2" link2="arm_2_link_2" reason="Never"/>
+    <disable_collisions link1="arm_1_link_2" link2="arm_2_link_3" reason="Never"/>
+    <disable_collisions link1="arm_1_link_2" link2="arm_2_link_4" reason="Never"/>
+    <disable_collisions link1="arm_1_link_2" link2="arm_2_link_5" reason="Never"/>
+    <disable_collisions link1="arm_1_link_2" link2="arm_2_link_6" reason="Never"/>
+    <disable_collisions link1="arm_1_link_2" link2="arm_2_link_7" reason="Never"/>
+    <disable_collisions link1="arm_1_link_3" link2="arm_1_link_4" reason="Adjacent"/>
+    <disable_collisions link1="arm_1_link_3" link2="arm_2_link_1" reason="Never"/>
+    <disable_collisions link1="arm_1_link_3" link2="arm_2_link_2" reason="Never"/>
+    <disable_collisions link1="arm_1_link_3" link2="arm_2_link_3" reason="Never"/>
+    <disable_collisions link1="arm_1_link_3" link2="arm_2_link_4" reason="Never"/>
+    <disable_collisions link1="arm_1_link_4" link2="arm_1_link_5" reason="Adjacent"/>
+    <disable_collisions link1="arm_1_link_4" link2="arm_1_link_6" reason="Never"/>
+    <disable_collisions link1="arm_1_link_4" link2="arm_1_link_7" reason="Never"/>
+    <disable_collisions link1="arm_1_link_4" link2="arm_2_link_1" reason="Never"/>
+    <disable_collisions link1="arm_1_link_4" link2="arm_2_link_2" reason="Never"/>
+    <disable_collisions link1="arm_1_link_4" link2="arm_2_link_3" reason="Never"/>
+    <disable_collisions link1="arm_1_link_4" link2="arm_2_link_4" reason="Never"/>
+    <disable_collisions link1="arm_1_link_5" link2="arm_1_link_6" reason="Adjacent"/>
+    <disable_collisions link1="arm_1_link_5" link2="arm_1_link_7" reason="Never"/>
+    <disable_collisions link1="arm_1_link_5" link2="arm_2_link_1" reason="Never"/>
+    <disable_collisions link1="arm_1_link_5" link2="arm_2_link_2" reason="Never"/>
+    <disable_collisions link1="arm_1_link_6" link2="arm_1_link_7" reason="Adjacent"/>
+    <disable_collisions link1="arm_1_link_6" link2="arm_2_link_2" reason="Never"/>
+    <disable_collisions link1="arm_2_link_1" link2="arm_2_link_2" reason="Adjacent"/>
+    <disable_collisions link1="arm_2_link_1" link2="arm_2_link_4" reason="Never"/>
+    <disable_collisions link1="arm_2_link_4" link2="arm_2_link_5" reason="Adjacent"/>
+    <disable_collisions link1="arm_2_link_4" link2="arm_2_link_6" reason="Never"/>
+    <disable_collisions link1="arm_2_link_4" link2="arm_2_link_7" reason="Never"/>
+    <disable_collisions link1="arm_2_link_5" link2="arm_2_link_6" reason="Adjacent"/>
+    <disable_collisions link1="arm_2_link_5" link2="arm_2_link_7" reason="Never"/>
+    <disable_collisions link1="arm_2_link_5" link2="leg1_link" reason="Never"/>
+    <disable_collisions link1="arm_2_link_5" link2="leg3_link" reason="Never"/>
+    <disable_collisions link1="arm_2_link_5" link2="obar1_link" reason="Never"/>
+    <disable_collisions link1="arm_2_link_5" link2="obar2_link" reason="Never"/>
+    <disable_collisions link1="arm_2_link_5" link2="obar3_link" reason="Never"/>
+    <disable_collisions link1="arm_2_link_5" link2="obar4_link" reason="Never"/>
+    <disable_collisions link1="arm_2_link_5" link2="sliding_guide_link" reason="Never"/>
+    <disable_collisions link1="arm_2_link_5" link2="vbar1_link" reason="Never"/>
+    <disable_collisions link1="arm_2_link_5" link2="vbar3_link" reason="Never"/>
+    <disable_collisions link1="arm_2_link_6" link2="arm_2_link_7" reason="Adjacent"/>
+    <disable_collisions link1="arm_2_link_6" link2="leg1_link" reason="Never"/>
+    <disable_collisions link1="arm_2_link_6" link2="leg3_link" reason="Never"/>
+    <disable_collisions link1="arm_2_link_6" link2="obar3_link" reason="Never"/>
+    <disable_collisions link1="arm_2_link_6" link2="obar4_link" reason="Never"/>
+    <disable_collisions link1="arm_2_link_6" link2="vbar1_link" reason="Never"/>
+    <disable_collisions link1="arm_2_link_6" link2="vbar3_link" reason="Never"/>
+    <disable_collisions link1="arm_2_link_7" link2="leg1_link" reason="Never"/>
+    <disable_collisions link1="arm_2_link_7" link2="leg3_link" reason="Never"/>
+    <disable_collisions link1="arm_2_link_7" link2="obar3_link" reason="Never"/>
+    <disable_collisions link1="arm_2_link_7" link2="vbar1_link" reason="Never"/>
+    <disable_collisions link1="arm_2_link_7" link2="vbar3_link" reason="Never"/>
+    <disable_collisions link1="leg1_link" link2="leg2_link" reason="Never"/>
+    <disable_collisions link1="leg1_link" link2="leg3_link" reason="Never"/>
+    <disable_collisions link1="leg1_link" link2="leg4_link" reason="Never"/>
+    <disable_collisions link1="leg1_link" link2="obar1_link" reason="Never"/>
+    <disable_collisions link1="leg1_link" link2="obar2_link" reason="Never"/>
+    <disable_collisions link1="leg1_link" link2="obar3_link" reason="Never"/>
+    <disable_collisions link1="leg1_link" link2="obar4_link" reason="Never"/>
+    <disable_collisions link1="leg1_link" link2="sliding_guide_link" reason="Never"/>
+    <disable_collisions link1="leg1_link" link2="table_top_link" reason="Adjacent"/>
+    <disable_collisions link1="leg1_link" link2="vbar1_link" reason="Adjacent"/>
+    <disable_collisions link1="leg1_link" link2="vbar2_link" reason="Never"/>
+    <disable_collisions link1="leg1_link" link2="vbar3_link" reason="Never"/>
+    <disable_collisions link1="leg1_link" link2="vbar4_link" reason="Never"/>
+    <disable_collisions link1="leg2_link" link2="leg3_link" reason="Never"/>
+    <disable_collisions link1="leg2_link" link2="leg4_link" reason="Never"/>
+    <disable_collisions link1="leg2_link" link2="obar1_link" reason="Never"/>
+    <disable_collisions link1="leg2_link" link2="obar2_link" reason="Never"/>
+    <disable_collisions link1="leg2_link" link2="obar3_link" reason="Never"/>
+    <disable_collisions link1="leg2_link" link2="obar4_link" reason="Never"/>
+    <disable_collisions link1="leg2_link" link2="sliding_guide_link" reason="Never"/>
+    <disable_collisions link1="leg2_link" link2="table_top_link" reason="Adjacent"/>
+    <disable_collisions link1="leg2_link" link2="vbar1_link" reason="Never"/>
+    <disable_collisions link1="leg2_link" link2="vbar2_link" reason="Adjacent"/>
+    <disable_collisions link1="leg2_link" link2="vbar3_link" reason="Never"/>
+    <disable_collisions link1="leg2_link" link2="vbar4_link" reason="Never"/>
+    <disable_collisions link1="leg3_link" link2="leg4_link" reason="Never"/>
+    <disable_collisions link1="leg3_link" link2="obar1_link" reason="Never"/>
+    <disable_collisions link1="leg3_link" link2="obar2_link" reason="Never"/>
+    <disable_collisions link1="leg3_link" link2="obar3_link" reason="Never"/>
+    <disable_collisions link1="leg3_link" link2="obar4_link" reason="Never"/>
+    <disable_collisions link1="leg3_link" link2="sliding_guide_link" reason="Never"/>
+    <disable_collisions link1="leg3_link" link2="table_top_link" reason="Adjacent"/>
+    <disable_collisions link1="leg3_link" link2="vbar1_link" reason="Never"/>
+    <disable_collisions link1="leg3_link" link2="vbar2_link" reason="Never"/>
+    <disable_collisions link1="leg3_link" link2="vbar3_link" reason="Adjacent"/>
+    <disable_collisions link1="leg3_link" link2="vbar4_link" reason="Never"/>
+    <disable_collisions link1="leg4_link" link2="obar1_link" reason="Never"/>
+    <disable_collisions link1="leg4_link" link2="obar2_link" reason="Never"/>
+    <disable_collisions link1="leg4_link" link2="obar3_link" reason="Never"/>
+    <disable_collisions link1="leg4_link" link2="obar4_link" reason="Never"/>
+    <disable_collisions link1="leg4_link" link2="sliding_guide_link" reason="Never"/>
+    <disable_collisions link1="leg4_link" link2="table_top_link" reason="Adjacent"/>
+    <disable_collisions link1="leg4_link" link2="vbar1_link" reason="Never"/>
+    <disable_collisions link1="leg4_link" link2="vbar2_link" reason="Never"/>
+    <disable_collisions link1="leg4_link" link2="vbar3_link" reason="Never"/>
+    <disable_collisions link1="leg4_link" link2="vbar4_link" reason="Adjacent"/>
+    <disable_collisions link1="obar1_link" link2="obar2_link" reason="Never"/>
+    <disable_collisions link1="obar1_link" link2="obar3_link" reason="Default"/>
+    <disable_collisions link1="obar1_link" link2="obar4_link" reason="Default"/>
+    <disable_collisions link1="obar1_link" link2="sliding_guide_link" reason="Default"/>
+    <disable_collisions link1="obar1_link" link2="table_top_link" reason="Never"/>
+    <disable_collisions link1="obar1_link" link2="vbar1_link" reason="Adjacent"/>
+    <disable_collisions link1="obar1_link" link2="vbar2_link" reason="Default"/>
+    <disable_collisions link1="obar1_link" link2="vbar3_link" reason="Never"/>
+    <disable_collisions link1="obar1_link" link2="vbar4_link" reason="Never"/>
+    <disable_collisions link1="obar2_link" link2="obar3_link" reason="Default"/>
+    <disable_collisions link1="obar2_link" link2="obar4_link" reason="Default"/>
+    <disable_collisions link1="obar2_link" link2="sliding_guide_link" reason="Adjacent"/>
+    <disable_collisions link1="obar2_link" link2="table_top_link" reason="Never"/>
+    <disable_collisions link1="obar2_link" link2="vbar1_link" reason="Never"/>
+    <disable_collisions link1="obar2_link" link2="vbar2_link" reason="Never"/>
+    <disable_collisions link1="obar2_link" link2="vbar3_link" reason="Adjacent"/>
+    <disable_collisions link1="obar2_link" link2="vbar4_link" reason="Default"/>
+    <disable_collisions link1="obar3_link" link2="obar4_link" reason="Never"/>
+    <disable_collisions link1="obar3_link" link2="sliding_guide_link" reason="Never"/>
+    <disable_collisions link1="obar3_link" link2="table_top_link" reason="Never"/>
+    <disable_collisions link1="obar3_link" link2="vbar1_link" reason="Default"/>
+    <disable_collisions link1="obar3_link" link2="vbar2_link" reason="Never"/>
+    <disable_collisions link1="obar3_link" link2="vbar3_link" reason="Adjacent"/>
+    <disable_collisions link1="obar3_link" link2="vbar4_link" reason="Never"/>
+    <disable_collisions link1="obar4_link" link2="sliding_guide_link" reason="Never"/>
+    <disable_collisions link1="obar4_link" link2="table_top_link" reason="Never"/>
+    <disable_collisions link1="obar4_link" link2="vbar1_link" reason="Never"/>
+    <disable_collisions link1="obar4_link" link2="vbar2_link" reason="Default"/>
+    <disable_collisions link1="obar4_link" link2="vbar3_link" reason="Never"/>
+    <disable_collisions link1="obar4_link" link2="vbar4_link" reason="Adjacent"/>
+    <disable_collisions link1="sliding_guide_link" link2="table_top_link" reason="Never"/>
+    <disable_collisions link1="sliding_guide_link" link2="vbar1_link" reason="Never"/>
+    <disable_collisions link1="sliding_guide_link" link2="vbar2_link" reason="Never"/>
+    <disable_collisions link1="sliding_guide_link" link2="vbar3_link" reason="Never"/>
+    <disable_collisions link1="sliding_guide_link" link2="vbar4_link" reason="Never"/>
+    <disable_collisions link1="table_top_link" link2="vbar1_link" reason="Default"/>
+    <disable_collisions link1="table_top_link" link2="vbar2_link" reason="Default"/>
+    <disable_collisions link1="table_top_link" link2="vbar3_link" reason="Default"/>
+    <disable_collisions link1="table_top_link" link2="vbar4_link" reason="Default"/>
+    <disable_collisions link1="vbar1_link" link2="vbar2_link" reason="Never"/>
+    <disable_collisions link1="vbar1_link" link2="vbar3_link" reason="Never"/>
+    <disable_collisions link1="vbar1_link" link2="vbar4_link" reason="Never"/>
+    <disable_collisions link1="vbar2_link" link2="vbar3_link" reason="Never"/>
+    <disable_collisions link1="vbar2_link" link2="vbar4_link" reason="Never"/>
+    <disable_collisions link1="vbar3_link" link2="vbar4_link" reason="Never"/> -->
 </robot>

File: repair_urdf/urdf/kinematics_properties.urdf.xacro (robot description, xacro)
@@ -1,21 +1,4 @@
 <!--<?xml version="1.0"?>-->
 <robot  xmlns:xacro="http://ros.org/wiki/xacro">
-    <xacro:property name="Cage_Ox" value=" 0.0 "/>  <!-- 0.0  -->
-    <xacro:property name="Cage_Oy" value=" 0.0 "/>  <!-- 0.0  -->
-    <xacro:property name="Cage_Oz" value=" 0.5 "/>  <!-- 0.0  -->
-    <!-- <xacro:property name="table_height" value="0.5" />
-    <xacro:property name="cage_width" value="1.5" />
-    <xacro:property name="cage_height" value="1.0"/>
-    <xacro:property name="cage_depth" value="2.5" />
-    <xacro:property name="leg_radius" value="0.02" />
-    <xacro:property name="cage_depth" value="2.5" />
-    <xacro:property name="sliding_guide_width" value="0.2" />
-    <xacro:property name="table_x" value="0.98" />
-    <xacro:property name="table_y" value="0.0" />
-    <xacro:property name="table_z" value="0.0" />
-    <xacro:property name="table_top_thickness" value="0.05"/>
-    <xacro:property name="PI" value="3.14159265359" />
-    <xacro:property name="PI_2" value="1.57079632679" />
-     -->
     <xacro:property name="Cage_x" value="1.5" />
     <xacro:property name="Cage_y" value="2.5" />

File: repair_urdf/urdf/repair_cage_macro.urdf.xacro (robot description, xacro)
@@ -2,11 +2,4 @@
 <robot xmlns:xacro="http://ros.org/wiki/xacro">
   <xacro:macro name="repair_cage" params="parent">
-  <!-- only something to avoid collisions between leg and ground plane when using Gaz. -->
-  <!-- <xacro:if value="$(arg shorten_table_legs_coll)">
-    <xacro:property name="leg_z_offset_gz" value="0.05" />
-  </xacro:if>
-    <xacro:property name="leg_z_offset_gz" value="0.0" />
-  </xacro:unless> -->
-  <xacro:property name="leg_z_offset_gz" value="0.0" />
   <link name="table_top_link">
     <visual>
@@ -42,5 +35,5 @@
     </visual>
     <collision>
-      <origin xyz="0.0 0.0 ${-table_height/2 + leg_z_offset_gz}" rpy="0.0 0.0 0.0" />
+      <origin xyz="0.0 0.0 ${-table_height/2}" rpy="0.0 0.0 0.0" />
       <geometry>
         <cylinder radius="${Cage_leg_radius}" length="${table_height}" />
@@ -82,5 +75,5 @@
     </visual>
     <collision>
-      <origin xyz="0.0 0.0 ${-table_height/2 + leg_z_offset_gz}" rpy="0.0 0.0 0.0" />
+      <origin xyz="0.0 0.0 ${-table_height/2}" rpy="0.0 0.0 0.0" />
       <geometry>
         <cylinder radius="${Cage_leg_radius}" length="${table_height}" />
@@ -122,5 +115,5 @@
     </visual>
     <collision>
-      <origin xyz="0.0 0.0 ${-table_height/2 + leg_z_offset_gz}" rpy="0.0 0.0 0.0" />
+      <origin xyz="0.0 0.0 ${-table_height/2}" rpy="0.0 0.0 0.0" />
       <geometry>
         <cylinder radius="${Cage_leg_radius}" length="${table_height}" />
@@ -162,5 +155,5 @@
     </visual>
     <collision>
-      <origin xyz="0.0 0.0 ${-table_height/2 + leg_z_offset_gz}" rpy="0.0 0.0 0.0" />
+      <origin xyz="0.0 0.0 ${-table_height/2}" rpy="0.0 0.0 0.0" />
       <geometry>
         <cylinder radius="${Cage_leg_radius}" length="${table_height}" />

File: repair_urdf/urdf/repair_full.urdf.xacro (robot description, xacro)
@@ -16,9 +16,9 @@
         <origin xyz="0.0 0.0 0.0" rpy="0.0 0.0 0.0" />
     </xacro:repair_torso>
-    <xacro:repair_arm id="1"  rot="1"  parent="torso_1">
+    <xacro:repair_arm id="2"  rot="1"  parent="torso_1">
       <origin xyz="${Shoulder_1_Ox} ${Shoulder_1_Oy} ${Shoulder_1_Oz}"
               rpy="${Shoulder_1_roll} ${Shoulder_1_pitch} ${Shoulder_1_yaw}" />
     </xacro:repair_arm>
-    <xacro:repair_arm id="2"  rot="-1"  parent="torso_1">
+    <xacro:repair_arm id="1"  rot="-1"  parent="torso_1">
         <origin xyz="${Shoulder_1_Ox} ${-Shoulder_1_Oy} ${Shoulder_1_Oz}"
                 rpy="${-Shoulder_1_roll} ${Shoulder_1_pitch} ${Shoulder_1_yaw}" />
