Commit message: added fixed hand argument to allow xbot2 integration

File: repair_srdf/srdf/repair_full.srdf.xacro (robot description, xacro)
@@ -27,8 +27,8 @@
         <!-- <group name="palm_left"/> -->
         <!-- <group name="thumb_left"/> -->
-        <group name="index_left"/>
+        <!-- <group name="index_left"/>
         <group name="middle_left"/>
         <group name="ring_left"/>
-        <group name="little_left"/>
+        <group name="little_left"/> -->
     </group>
     <group_state name="home" group="chains">

File: repair_urdf/urdf/repair_arm.urdf.xacro (robot description, xacro)
@@ -16,5 +16,5 @@
 <xacro:property name="sm_tau_max" value="200.0" />
 <xacro:include filename="$(find repair_urdf)/urdf/repair_arm_coll_params.urdf.xacro"/>
-<xacro:macro name="repair_arm" params="id base_link is_sliding_wrist gen_coll load_sol use_updated_wrist gz_self_collide" >
+<xacro:macro name="repair_arm" params="id base_link is_sliding_wrist gen_coll load_sol use_updated_wrist gz_self_collide fixed_hands" >
 <xacro:if value="${gen_coll == True}">
     <xacro:include filename="$(find repair_urdf)/urdf/repair_arm_coll.urdf.xacro"/>
@@ -354,5 +354,6 @@
         orientation="0 0 0"
         operation_mode="0"
-        translation="0">
+        translation="0"
+        fixed_hands="${fixed_hands}">
     </xacro:softhands>
 </xacro:if>
@@ -364,5 +365,6 @@
         orientation="0 0 0"
         operation_mode="0"
-        translation="0">
+        translation="0"
+        fixed_hands="${fixed_hands}">
     </xacro:softhands>
 </xacro:unless>

File: repair_urdf/urdf/repair_full.urdf.xacro (robot description, xacro)
@@ -16,4 +16,5 @@
 <xacro:arg name="gz_self_collide" default="true" />
 <xacro:arg name="xbot" default="true" />
+<xacro:arg name="fixed_hands" default="false" />
 <xacro:include filename="$(find repair_urdf)/urdf/repair_arm.urdf.xacro"/>
 <xacro:include filename="$(find repair_urdf)/urdf/repair_cage.urdf.xacro"/>
@@ -154,9 +155,9 @@
 </xacro:unless>
 <xacro:repair_arm base_link="r_arm_mount_frame" id="1" is_sliding_wrist="$(arg is_sliding_wrist)"
-gen_coll="$(arg gen_coll)" load_sol="$(arg load_sol)" use_updated_wrist = "$(arg use_updated_wrist)"
-gz_self_collide = "$(arg gz_self_collide)" />
+gen_coll="$(arg gen_coll)" load_sol="$(arg load_sol)" use_updated_wrist ="$(arg use_updated_wrist)"
+gz_self_collide ="$(arg gz_self_collide)" fixed_hands ="$(arg fixed_hands)" />
 <xacro:repair_arm base_link="l_arm_mount_frame" id="2" is_sliding_wrist="$(arg is_sliding_wrist)"
-gen_coll="$(arg gen_coll)" load_sol="$(arg load_sol)" use_updated_wrist = "$(arg use_updated_wrist)"
-gz_self_collide = "$(arg gz_self_collide)" />
+gen_coll="$(arg gen_coll)" load_sol="$(arg load_sol)" use_updated_wrist ="$(arg use_updated_wrist)"
+gz_self_collide ="$(arg gz_self_collide)" fixed_hands ="$(arg fixed_hands)" />
 <xacro:repair_arm_materials id="1" />
 <xacro:repair_arm_materials id="2" />

File: repair_urdf/urdf/repair_full_xbot.urdf (robot description, URDF)
Before this commit: robot repair_full, 79 links, 78 joints
Joints:
- joint left_hand_v1s_index_distal_joint: type revolute -> fixed
- joint left_hand_v1s_index_knuckle_joint: type revolute -> fixed
- joint left_hand_v1s_index_middle_joint: type revolute -> fixed
- joint left_hand_v1s_index_proximal_joint: type revolute -> fixed
- joint left_hand_v1s_little_distal_joint: type revolute -> fixed
- joint left_hand_v1s_little_knuckle_joint: type revolute -> fixed
- joint left_hand_v1s_little_middle_joint: type revolute -> fixed
- joint left_hand_v1s_little_proximal_joint: type revolute -> fixed
- joint left_hand_v1s_middle_distal_joint: type revolute -> fixed
- joint left_hand_v1s_middle_knuckle_joint: type revolute -> fixed
- joint left_hand_v1s_middle_middle_joint: type revolute -> fixed
- joint left_hand_v1s_middle_proximal_joint: type revolute -> fixed
- joint left_hand_v1s_ring_distal_joint: type revolute -> fixed
- joint left_hand_v1s_ring_knuckle_joint: type revolute -> fixed
- joint left_hand_v1s_ring_middle_joint: type revolute -> fixed
- joint left_hand_v1s_ring_proximal_joint: type revolute -> fixed
- joint left_hand_v1s_thumb_distal_joint: type continuous -> fixed
- joint left_hand_v1s_thumb_knuckle_joint: type continuous -> fixed
- joint left_hand_v1s_thumb_proximal_joint: type continuous -> fixed
- joint right_hand_v1s_index_distal_joint: type revolute -> fixed
- joint right_hand_v1s_index_knuckle_joint: type revolute -> fixed
- joint right_hand_v1s_index_middle_joint: type revolute -> fixed
- joint right_hand_v1s_index_proximal_joint: type revolute -> fixed
- joint right_hand_v1s_little_distal_joint: type revolute -> fixed
- joint right_hand_v1s_little_knuckle_joint: type revolute -> fixed
- joint right_hand_v1s_little_middle_joint: type revolute -> fixed
- joint right_hand_v1s_little_proximal_joint: type revolute -> fixed
- joint right_hand_v1s_middle_distal_joint: type revolute -> fixed
- joint right_hand_v1s_middle_knuckle_joint: type revolute -> fixed
- joint right_hand_v1s_middle_middle_joint: type revolute -> fixed
- joint right_hand_v1s_middle_proximal_joint: type revolute -> fixed
- joint right_hand_v1s_ring_distal_joint: type revolute -> fixed
- joint right_hand_v1s_ring_knuckle_joint: type revolute -> fixed
- joint right_hand_v1s_ring_middle_joint: type revolute -> fixed
- joint right_hand_v1s_ring_proximal_joint: type revolute -> fixed
- joint right_hand_v1s_thumb_distal_joint: type continuous -> fixed
- joint right_hand_v1s_thumb_knuckle_joint: type continuous -> fixed
- joint right_hand_v1s_thumb_proximal_joint: type continuous -> fixed

Commit message: fixed orientation and added reasonable homing

File: repair_srdf/srdf/repair_full.srdf.xacro (robot description, xacro)
@@ -33,18 +33,18 @@
     </group>
     <group_state name="home" group="chains">
-        <joint name="arm_1_joint_1" value="1.5"/>
-        <joint name="arm_1_joint_2" value="1.1"/>
+        <joint name="arm_1_joint_1" value="0.85"/>
+        <joint name="arm_1_joint_2" value="0.72"/>
         <joint name="arm_1_joint_3" value="0.6"/>
         <joint name="arm_1_joint_4" value="-0.9"/>
         <joint name="arm_1_joint_5" value="-0.5"/>
         <joint name="arm_1_joint_6" value="0"/>
-        <joint name="arm_1_joint_7" value="0"/>
-        <joint name="arm_2_joint_1" value="-1.5"/>
-        <joint name="arm_2_joint_2" value="-1.1"/>
+        <joint name="arm_1_joint_7" value="1.0"/>
+        <joint name="arm_2_joint_1" value="-0.85"/>
+        <joint name="arm_2_joint_2" value="-0.72"/>
         <joint name="arm_2_joint_3" value="-0.6"/>
         <joint name="arm_2_joint_4" value="-0.9"/>
         <joint name="arm_2_joint_5" value="0.5"/>
         <joint name="arm_2_joint_6" value="0"/>
-        <joint name="arm_2_joint_7" value="0"/>
+        <joint name="arm_2_joint_7" value="-1.0"/>
         <joint name="x_joint" value="-0.05"/>
         <xacro:softhand_homing side="right" type="v1s"/>

File: repair_urdf/urdf/repair_arm.urdf.xacro (robot description, xacro)
@@ -352,5 +352,5 @@
         parent="arm_${id}_link_7"
         position="0 0 -0.015"
-        orientation="0 0 0"
+        orientation="0 0.0 ${PI}"
         translation="0"
         operation_mode="0"
@@ -362,6 +362,6 @@
         version="v1.0_simple"
         parent="arm_${id}_link_7"
-        position="0 0.013900 -0.015"
-        orientation="0 0.0 ${PI}"
+        position="0 -0.013900 -0.015"
+        orientation="0 0 0"
         translation="0"
         operation_mode="0"

File: repair_urdf/urdf/repair_full.urdf (robot description, URDF)
Before this commit: robot repair_full, 79 links, 78 joints
Joints:
- joint left_hand_base_joint: origin xyz=0 0.013900 -0.015 rpy=0 0.0 3.14159265359 -> xyz=0 -0.013900 -0.015 rpy=0 0 0
- joint right_hand_base_joint: origin xyz=0 0 -0.015 rpy=0 0 0 -> xyz=0 0 -0.015 rpy=0 0.0 3.14159265359

Commit message: corrected hands, new homing position, new cage dimensions

File: repair_srdf/srdf/repair_full.srdf.xacro (robot description, xacro)
@@ -33,17 +33,17 @@
     <group_state name="home" group="chains">
         <joint name="j_arm_1_1" value="-0.5"/>
-        <joint name="j_arm_1_2" value="-0.5"/>
+        <joint name="j_arm_1_2" value="-0.7"/>
         <joint name="j_arm_1_3" value="0.5"/>
-        <joint name="j_arm_1_4" value="-1.0"/>
+        <joint name="j_arm_1_4" value="-1.2"/>
         <joint name="j_arm_1_5" value="-0.5"/>
-        <joint name="j_arm_1_6" value="-0.5"/>
-        <joint name="j_arm_1_7" value="-1.0"/>
+        <joint name="j_arm_1_6" value="0.5"/>
+        <joint name="j_arm_1_7" value="0.5"/>
         <joint name="j_arm_2_1" value="0.5"/>
-        <joint name="j_arm_2_2" value="0.5"/>
+        <joint name="j_arm_2_2" value="0.7"/>
         <joint name="j_arm_2_3" value="-0.5"/>
-        <joint name="j_arm_2_4" value="1.0"/>
+        <joint name="j_arm_2_4" value="1.2"/>
         <joint name="j_arm_2_5" value="0.5"/>
-        <joint name="j_arm_2_6" value="0.5"/>
-        <joint name="j_arm_2_7" value="1.0"/>
+        <joint name="j_arm_2_6" value="-0.5"/>
+        <joint name="j_arm_2_7" value="-0.5"/>
         <!-- <xacro:softhand_homing side="right" type="v1s"/>
         <xacro:softhand_homing side="left" type="v1s"/> -->

File: repair_urdf/urdf/kinematics_properties.urdf.xacro (robot description, xacro)
@@ -4,9 +4,9 @@
     <xacro:property name="Table_y" value="0.0" />
     <xacro:property name="Table_z" value="0.0" /> <!-- w.r.t world  -->
-    <xacro:property name="table_top_thickness" value="0.05"/>
-    <xacro:property name="table_height" value="1.0"/>
+    <xacro:property name="table_top_thickness" value="0.03"/> <!-- w.r.t. top origin of table to down  -->
+    <xacro:property name="table_height" value="0.983"/> <!-- w.r.t. working surface of the table  -->
     <xacro:property name="Cage_x" value="1.0" />
     <xacro:property name="Cage_y" value="2.5" />
-    <xacro:property name="Cage_z" value="0.97"/> <!-- w.r.t table  -->
+    <xacro:property name="Cage_z" value="1.05"/> <!-- w.r.t table  -->
     <xacro:property name="Cage_leg_radius" value="0.02" />
     <xacro:property name="Cage_sliding_guide_x" value="0.0"/> <!-- w.r.t world  -->
@@ -14,5 +14,5 @@
     <xacro:property name="Cage_sliding_guide_z" value="0.0"/> <!-- w.r.t world  -->
     <xacro:property name="Cage_sliding_guide_width" value="0.4"/>
-    <xacro:property name="Torso_Ox" value=" 0.0 "/>
+    <xacro:property name="Torso_Ox" value=" -0.13 "/>
     <xacro:property name="Torso_Oy" value=" 0.0 "/>
     <xacro:property name="Torso_Oz" value=" 0.0 "/>

File: repair_urdf/urdf/repair_full.urdf.xacro (robot description, xacro)
@@ -29,18 +29,18 @@
         version="v1.0_simple"
         parent="arm_1_7"
-        position="0 0 -0.015"
-        orientation="0 0.0 ${PI}"
+        position="0.0 0.0 0.0"
+        orientation="0 0.0 ${PI/2}"
         translation="0"
         operation_mode="0"
-        fixed_hands="false">
+        fixed_hands="true">
     </xacro:softhands>
     <xacro:softhands type="right"
         version="v1.0_simple"
         parent="arm_2_7"
-        position="0 -0.013900 -0.015"
-        orientation="0 0 ${PI}"
+        position="0.0 0.0 0.0"
+        orientation="0.0 0.0 ${-PI/2}"
         translation="0"
         operation_mode="0"
-        fixed_hands="false">
+        fixed_hands="true">
     </xacro:softhands>
     <!-- <gazebo reference="table_top_link">
