Commit message: added file for gazebo simulation

File: repair_urdf/urdf/gazebo/xbot.gazebo.xacro (robot description, xacro)
@@ -4,15 +4,14 @@
     <plugin name="xbot2_joint_driver" filename="libxbot2_gz_joint_server.so">
         <pid>
-            <gain name="lowpwr_mot" p="50"  d="5"/>
+            <gain name="fake_mot"  p="10"  d="1"/>
             <gain name="small_mot"  p="1000"  d="10"/>
-            <gain name="medium_mot" p="4000" d="40"/>
-            <gain name="big_mot"    p="8000" d="50"/>
-            <pid name="j_arm1_1" profile="medium_mot"/>
-            <pid name="j_arm1_2" profile="medium_mot"/>
-            <pid name="j_arm1_3" profile="medium_mot"/>
-            <pid name="j_arm1_4" profile="medium_mot"/>
-            <pid name="j_arm1_5" profile="small_mot"/>
-            <pid name="j_arm1_6" profile="small_mot"/>
-            <pid name="j_arm1_7" profile="small_mot"/>
+            <gain name="medium_mot" p="2000" d="20"/>
+            <pid name="j_arm_1_1" profile="medium_mot"/>
+            <pid name="j_arm_1_2" profile="medium_mot"/>
+            <pid name="j_arm_1_3" profile="medium_mot"/>
+            <pid name="j_arm_1_4" profile="medium_mot"/>
+            <pid name="j_arm_1_5" profile="small_mot"/>
+            <pid name="j_arm_1_6" profile="small_mot"/>
+            <pid name="j_arm_1_7" profile="small_mot"/>
         </pid>
     </plugin>

File: repair_urdf/urdf/inertial_properties.urdf.xacro (robot description, xacro)
@@ -106,14 +106,14 @@
     <!-- WRITST ROLL -->
     <!-- Center of Mass -->
-    <xacro:property name="Wrist_2_x" value="0.0000000e+00"/>
-    <xacro:property name="Wrist_2_y" value="-1.0491951e+00"/>
-    <xacro:property name="Wrist_2_z" value="-1.0307299e+01"/>
+    <xacro:property name="Wrist_2_x" value=" ${0.0000000e+00 *mmTom} "/>
+    <xacro:property name="Wrist_2_y" value=" ${-1.0491951e+00 *mmTom} "/>
+    <xacro:property name="Wrist_2_z" value=" ${-1.0307299e+01 *mmTom} "/>
     <!-- Inertia -->
-    <xacro:property name="Wrist_2_xx" value="6.1479333e+01"/>
-    <xacro:property name="Wrist_2_yy" value="6.4247521e+01"/>
-    <xacro:property name="Wrist_2_zz" value="1.1879744e+02"/>
-    <xacro:property name="Wrist_2_xy" value="-7.4023399e-05"/>
-    <xacro:property name="Wrist_2_xz" value="0.0000000e+00"/>
-    <xacro:property name="Wrist_2_yz" value="4.7786448e-01"/>
+    <xacro:property name="Wrist_2_xx" value=" ${6.1479333e+01 *mm2Tom2} "/>
+    <xacro:property name="Wrist_2_yy" value=" ${6.4247521e+01 *mm2Tom2} "/>
+    <xacro:property name="Wrist_2_zz" value=" ${1.1879744e+02 *mm2Tom2} "/>
+    <xacro:property name="Wrist_2_xy" value=" ${-7.4023399e-05 *mm2Tom2} "/>
+    <xacro:property name="Wrist_2_xz" value=" ${0.0000000e+00 *mm2Tom2} "/>
+    <xacro:property name="Wrist_2_yz" value=" ${4.7786448e-01 *mm2Tom2} "/>
     <!-- Mass -->
     <xacro:property name="Wrist_2_mass" value="1.4163970e-01"/>

File: repair_urdf/urdf/kinematics_properties.urdf.xacro (robot description, xacro)
@@ -44,5 +44,5 @@
     <xacro:property name="Wrist_1_yaw" value=" 0.0 "/>
     <!-- Origin -->
-    <xacro:property name="Wrist_2_Ox" value=" 0.0216503 "/>
+    <xacro:property name="Wrist_2_Ox" value=" 0.00 "/>
     <xacro:property name="Wrist_2_Oy" value=" 0.062877 "/>
     <xacro:property name="Wrist_2_Oz" value=" 0.050 "/>

File: repair_urdf/urdf/repair_arm_macro.urdf.xacro (robot description, xacro)
@@ -130,5 +130,5 @@
                 <inertia ixx="${Wrist_2_xx}" ixy="${rot*Wrist_2_xy}" ixz="${Wrist_2_xz}"
                     iyy="${Wrist_2_yy}" iyz="${rot*Wrist_2_yz}" izz="${Wrist_2_zz}" />
-                </inertial>
+            </inertial>
             <visual>
                 <geometry>
@@ -143,5 +143,11 @@
             </collision>
         </link>
-        <link name="arm_${id}_tcp" />
+        <link name="arm_${id}_tcp">
+            <inertial>
+                <origin xyz="0.0 0.05 0.1" />
+                <mass value="0.5" />
+                <inertia ixx="0.001" ixy="0.0" ixz="0.0" iyy="0.001" iyz="0.0" izz="0.001" />
+            </inertial>
+        </link>
         <!-- JOINTS -->
         <!-- shoulder pitch -->

Commit message: added full system in urdf

File: repair_urdf/urdf/gazebo/xbot.gazebo.xacro (robot description, xacro)
@@ -14,4 +14,11 @@
             <pid name="j_arm_1_6" profile="small_mot"/>
             <pid name="j_arm_1_7" profile="small_mot"/>
+            <!-- <pid name="j_arm_2_1" profile="medium_mot"/>
+            <pid name="j_arm_2_2" profile="medium_mot"/>
+            <pid name="j_arm_2_3" profile="medium_mot"/>
+            <pid name="j_arm_2_4" profile="medium_mot"/>
+            <pid name="j_arm_2_5" profile="small_mot"/>
+            <pid name="j_arm_2_6" profile="small_mot"/>
+            <pid name="j_arm_2_7" profile="small_mot"/> -->
         </pid>
     </plugin>

File: repair_urdf/urdf/inertial_properties.urdf.xacro (robot description, xacro)
@@ -7,4 +7,17 @@
     <xacro:property name="motors_length" value=" 0.100000 "/>
     <xacro:property name="motors_weight" value=" 1.500000 "/>
+    <!-- Center of Mass -->
+    <xacro:property name="Torso_x" value=" ${4.9776510e-01 *mmTom} "/>
+    <xacro:property name="Torso_y" value=" ${-4.2604032e-01*mmTom} "/>
+    <xacro:property name="Torso_z" value=" ${-1.6838189e+02 *mmTom} "/>
+    <!-- Inertia -->
+    <xacro:property name="Torso_xx" value=" ${1.1857829e+05 *mm2Tom2} "/>
+    <xacro:property name="Torso_yy" value=" ${8.0733992e+04 *mm2Tom2} "/>
+    <xacro:property name="Torso_zz" value=" ${5.4100212e+04 *mm2Tom2} "/>
+    <xacro:property name="Torso_xy" value=" ${2.0401988e+01 *mm2Tom2} "/>
+    <xacro:property name="Torso_xz" value=" ${1.2279511e+01 *mm2Tom2} "/>
+    <xacro:property name="Torso_yz" value=" ${7.0011268e+00 *mm2Tom2}"/>
+    <!-- Mass -->
+    <xacro:property name="Torso_mass" value=" 8.7077745e+00 "/>
     <!-- Center of Mass -->
     <xacro:property name="Base_x" value=" ${2.0548930e-01 *mmTom} "/>
@@ -33,5 +46,5 @@
     <xacro:property name="Shoulder_1_yz" value=" ${1.2857051e+03 *mm2Tom2}"/>
     <!-- Mass -->
-    <xacro:property name="Shoulder_1_mass" value="2.4405495"/>
+    <xacro:property name="Shoulder_1_mass" value="2.347"/> <!-- 2.4405495 -->
     <!-- SHOULDER ROLL -->
     <!-- Center of Mass -->
@@ -47,5 +60,5 @@
     <xacro:property name="Shoulder_2_yz" value=" ${-6.6693438e+02 *mm2Tom2}"/>
     <!-- Mass -->
-    <xacro:property name="Shoulder_2_mass" value="7.8724534e-01"/>
+    <xacro:property name="Shoulder_2_mass" value="0.76"/> <!-- 7.8724534e-01 -->
     <!-- SHOULDER YAW -->
     <!-- Center of Mass -->
@@ -61,5 +74,5 @@
     <xacro:property name="Shoulder_3_yz" value=" ${1.8728041e+03 *mm2Tom2}"/>
     <!-- Mass -->
-    <xacro:property name="Shoulder_3_mass" value="2.8848438e+00"/>
+    <xacro:property name="Shoulder_3_mass" value="3.34"/> <!-- 2.8848438e+00-->
     <!-- ELBOW -->
     <!-- Center of Mass -->
@@ -75,33 +88,33 @@
     <xacro:property name="Elbow_yz" value=" ${-3.9531701e+02 *mm2Tom2} "/>
     <!-- Mass -->
-    <xacro:property name="Elbow_mass" value="6.0145584e-01"/>
+    <xacro:property name="Elbow_mass" value="0.55"/> <!-- 6.0145584e-01 -->
     <!-- FOREARM -->
     <!-- Center of Mass -->
-    <xacro:property name="Forearm_x" value=" ${2.0004978e+00 *mmTom} "/>
-    <xacro:property name="Forearm_y" value=" ${-5.9178127e+01 *mmTom} "/>
-    <xacro:property name="Forearm_z" value=" ${-1.5065406e+02 *mmTom} "/>
+    <xacro:property name="Forearm_x" value=" ${9.4711044e-01 *mmTom} "/>
+    <xacro:property name="Forearm_y" value=" ${-4.8009667e+01 *mmTom} "/>
+    <xacro:property name="Forearm_z" value=" ${-1.4331833e+02 *mmTom} "/>
     <!-- Inertia -->
-    <xacro:property name="Forearm_xx" value=" ${9.9022766e+03 *mm2Tom2}"/>
-    <xacro:property name="Forearm_yy" value=" ${7.1759859e+03 *mm2Tom2}"/>
-    <xacro:property name="Forearm_zz" value=" ${4.5802104e+03 *mm2Tom2}"/>
-    <xacro:property name="Forearm_xy" value=" ${4.4500899e+01 *mm2Tom2} "/>
-    <xacro:property name="Forearm_xz" value=" ${1.3354192e+01 *mm2Tom2} "/>
-    <xacro:property name="Forearm_yz" value=" ${-3.1875374e+03 *mm2Tom2}"/>
+    <xacro:property name="Forearm_xx" value=" ${3.0333275e+04 *mm2Tom2}"/>
+    <xacro:property name="Forearm_yy" value=" ${2.5195445e+04 *mm2Tom2}"/>
+    <xacro:property name="Forearm_zz" value=" ${6.9975104e+03 *mm2Tom2}"/>
+    <xacro:property name="Forearm_xy" value=" ${7.3729709e+01 *mm2Tom2} "/>
+    <xacro:property name="Forearm_xz" value=" ${3.2427371e+01 *mm2Tom2} "/>
+    <xacro:property name="Forearm_yz" value=" ${-9.5263763e+03 *mm2Tom2}"/>
     <!-- Mass -->
-    <xacro:property name="Forearm_mass" value="1.3065556e+00"/>
+    <xacro:property name="Forearm_mass" value="2.825"/> <!-- 2.7650803e+00 -->
     <!-- WRITST PITCH -->
     <!-- Center of Mass -->
-    <xacro:property name="Wrist_1_x" value=" ${-5.8850122e+00 *mmTom} "/>
-    <xacro:property name="Wrist_1_y" value=" ${-2.0700011e+01 *mmTom} "/>
-    <xacro:property name="Wrist_1_z" value=" ${4.4606499e+01 *mmTom} "/>
+    <xacro:property name="Wrist_1_x" value=" ${6.8559302e-01 *mmTom} "/>
+    <xacro:property name="Wrist_1_y" value=" ${-5.0299682e+00 *mmTom} "/>
+    <xacro:property name="Wrist_1_z" value=" ${4.6682846e+01 *mmTom} "/>
     <!-- Inertia -->
-    <xacro:property name="Wrist_1_xx" value=" ${3.3129474e+03 *mm2Tom2} "/>
-    <xacro:property name="Wrist_1_yy" value=" ${2.9894708e+03 *mm2Tom2} "/>
-    <xacro:property name="Wrist_1_zz" value=" ${3.6865610e+03 *mm2Tom2} "/>
-    <xacro:property name="Wrist_1_xy" value=" ${-2.2801449e+02 *mm2Tom2} "/>
-    <xacro:property name="Wrist_1_xz" value=" ${-1.1490187e+02 *mm2Tom2} "/>
-    <xacro:property name="Wrist_1_yz" value=" ${-4.9067763e+01 *mm2Tom2} "/>
+    <xacro:property name="Wrist_1_xx" value=" ${4.2406037e+03 *mm2Tom2} "/>
+    <xacro:property name="Wrist_1_yy" value=" ${2.9010806e+03 *mm2Tom2} "/>
+    <xacro:property name="Wrist_1_zz" value=" ${4.4989008e+03 *mm2Tom2} "/>
+    <xacro:property name="Wrist_1_xy" value=" ${-5.5692732e+01 *mm2Tom2} "/>
+    <xacro:property name="Wrist_1_xz" value=" ${-9.0851982e+01 *mm2Tom2} "/>
+    <xacro:property name="Wrist_1_yz" value=" ${-1.8560541e+02 *mm2Tom2} "/>
     <!-- Mass -->
-    <xacro:property name="Wrist_1_mass" value="1.1552856e+00"/>
+    <xacro:property name="Wrist_1_mass" value="1.861"/> <!-- 1.8854765e+00 -->
     <!-- WRITST ROLL -->
     <!-- Center of Mass -->
@@ -117,4 +130,4 @@
     <xacro:property name="Wrist_2_yz" value=" ${4.7786448e-01 *mm2Tom2} "/>
     <!-- Mass -->
-    <xacro:property name="Wrist_2_mass" value="1.4163970e-01"/>
+    <xacro:property name="Wrist_2_mass" value="1.4163970e-01"/> <!-- 2.4405495 -->
     </robot>

File: repair_urdf/urdf/kinematics_properties.urdf.xacro (robot description, xacro)
@@ -1,9 +1,43 @@
 <!--<?xml version="1.0"?>-->
 <robot  xmlns:xacro="http://ros.org/wiki/xacro">
+    <xacro:property name="Cage_Ox" value=" 0.0 "/>  <!-- 0.0  -->
+    <xacro:property name="Cage_Oy" value=" 0.0 "/>  <!-- 0.0  -->
+    <xacro:property name="Cage_Oz" value=" 0.5 "/>  <!-- 0.0  -->
+    <!-- <xacro:property name="table_height" value="0.5" />
+    <xacro:property name="cage_width" value="1.5" />
+    <xacro:property name="cage_height" value="1.0"/>
+    <xacro:property name="cage_depth" value="2.5" />
+    <xacro:property name="leg_radius" value="0.02" />
+    <xacro:property name="cage_depth" value="2.5" />
+    <xacro:property name="sliding_guide_width" value="0.2" />
+    <xacro:property name="table_x" value="0.98" />
+    <xacro:property name="table_y" value="0.0" />
+    <xacro:property name="table_z" value="0.0" />
+    <xacro:property name="table_top_thickness" value="0.05"/>
+    <xacro:property name="PI" value="3.14159265359" />
+    <xacro:property name="PI_2" value="1.57079632679" />
+     -->
+    <xacro:property name="Cage_x" value="1.5" />
+    <xacro:property name="Cage_y" value="2.5" />
+    <xacro:property name="Cage_z" value="1.0"/>
+    <xacro:property name="Cage_leg_radius" value="0.02" />
+    <xacro:property name="Cage_sliding_guide_width" value="0.2" />
+    <xacro:property name="Table_x" value="0.98" />
+    <xacro:property name="Table_y" value="0.0" />
+    <xacro:property name="Table_z" value="0.0" />
+    <xacro:property name="table_top_thickness" value="0.05"/>
+    <xacro:property name="table_height" value="0.5"/>
+    <xacro:property name="sliding_guide_width" value="0.2"/>
+    <xacro:property name="Torso_Ox" value=" 0.0 "/>
+    <xacro:property name="Torso_Oy" value=" 0.0 "/>
+    <xacro:property name="Torso_Oz" value=" 0.0 "/>
+    <xacro:property name="Torso_roll" value=" 0.0 "/>
+    <xacro:property name="Torso_pitch" value=" ${PI/2} "/>
+    <xacro:property name="Torso_yaw" value=" 0.0 "/>
     <!-- Origin -->
     <xacro:property name="Shoulder_1_Ox" value=" 0.0 "/>  <!-- 0.0  -->
-    <xacro:property name="Shoulder_1_Oy" value=" 0.0"/> <!-- 0.13515  -->
-    <xacro:property name="Shoulder_1_Oz" value=" 0.14 "/> <!-- -0.24215  -->
-    <xacro:property name="Shoulder_1_roll" value=" 0.0 "/> <!-- ${PI/2}  -->
+    <xacro:property name="Shoulder_1_Oy" value="  -0.135150"/> <!-- 0.13515  -->
+    <xacro:property name="Shoulder_1_Oz" value=" -0.242150 "/> <!-- -0.24215  -->
+    <xacro:property name="Shoulder_1_roll" value=" ${PI/2} "/> <!-- ${PI/2}  -->
     <xacro:property name="Shoulder_1_pitch" value=" 0.0 "/> <!-- 0.0  -->
     <xacro:property name="Shoulder_1_yaw" value=" 0.0 "/> <!-- 0.0  -->
@@ -20,5 +54,5 @@
     <xacro:property name="Shoulder_3_Oz" value=" -0.06015 "/> <!-- -0.06015  -->
     <xacro:property name="Shoulder_3_roll" value=" ${-PI/2}"/>
-    <xacro:property name="Shoulder_3_pitch" value=" ${-PI/2} "/>
+    <xacro:property name="Shoulder_3_pitch" value=" ${PI/2} "/>
     <xacro:property name="Shoulder_3_yaw" value=" 0.0 "/>
     <!-- Origin -->

File: repair_urdf/urdf/limits.urdf.xacro (robot description, xacro)
@@ -2,4 +2,6 @@
 <robot  xmlns:xacro="http://ros.org/wiki/xacro">
     <!-- Origin -->
+    <xacro:property name="j_prismatic_lower" value="${[2]}"/>
+    <xacro:property name="j_torso_lower" value="${[-2.6]}"/>
     <xacro:property name="j_arm_1_lower" value="${[-2.6]}"/>
     <xacro:property name="j_arm_2_lower" value="${[-2.5]}"/>
@@ -9,4 +11,6 @@
     <xacro:property name="j_arm_6_lower" value="${[-2.8]}"/>
     <xacro:property name="j_arm_7_lower" value="${[-2.8]}"/>
+    <xacro:property name="j_prismatic_upper" value="${[-2]}"/>
+    <xacro:property name="j_torso_upper" value="${[2.6]}"/>
     <xacro:property name="j_arm_1_upper" value="${[2.6]}"/>
     <xacro:property name="j_arm_2_upper" value="${[0.1]}"/>
@@ -16,4 +20,6 @@
     <xacro:property name="j_arm_6_upper" value="${[2.1]}"/>
     <xacro:property name="j_arm_7_upper" value="${[2.8]}"/>
+    <xacro:property name="j_prismatic_velocity" value="${[-5]}"/>
+    <xacro:property name="j_torso_velocity" value="${[3.86]}"/>
     <xacro:property name="j_arm_1_velocity" value="${[3.86]}"/>
     <xacro:property name="j_arm_2_velocity" value="${[3.86]}"/>
@@ -23,4 +29,6 @@
     <xacro:property name="j_arm_6_velocity" value="${[11.72]}"/>
     <xacro:property name="j_arm_7_velocity" value="${[11.72]}"/>
+    <xacro:property name="j_prismatic_torque" value="${[147]}"/>
+    <xacro:property name="j_torso_torque" value="${[147.00]}"/>
     <xacro:property name="j_arm_1_torque" value="${[147.00]}"/>
     <xacro:property name="j_arm_2_torque" value="${[147.00]}"/>

File: repair_urdf/urdf/materials.urdf.xacro (robot description, xacro)
@@ -25,3 +25,9 @@
     <color rgba="0.6 0.6 0.6 1"/>
 </material>
+<material name="wood">
+  <color rgba="0.522 0.369 0.259 0.8"/>
+</material>
+<material name="silver_gray">
+  <color rgba="0.8 0.8 0.8 0.8"/>
+</material>
 </robot>

File: repair_urdf/urdf/repair_arm.urdf (robot description, URDF)
Before this commit: robot repair_arm, 10 links, 9 joints
Links:
- link arm_1_1: mass 2.4405495 -> 2.347
- link arm_1_2: mass 0.78724534 -> 0.76
- link arm_1_3: mass 2.8848438 -> 3.34
- link arm_1_4: mass 0.60145584 -> 0.55
- link arm_1_5: mass 1.3065556 -> 2.825
- link arm_1_6: mass 1.1552856 -> 1.861

File: repair_urdf/urdf/repair_arm_final.urdf.xacro (robot description, xacro)
@@ -14,6 +14,6 @@
     </xacro:repair_base>
     <xacro:repair_arm id="1"  rot="1"  parent="base_link">
-      <origin xyz="${Shoulder_1_Ox} ${Shoulder_1_Oy} ${Shoulder_1_Oz}"
-              rpy="${Shoulder_1_roll} ${Shoulder_1_pitch} ${Shoulder_1_yaw}" />
+      <origin xyz="0.0 0.0 0.14"
+              rpy="0.0 0.0 0.0" />
     </xacro:repair_arm>
 </robot>
