Commit message: added full system in urdf

File: repair_urdf/urdf/repair_cage_macro.urdf.xacro (robot description, xacro)
@@ -1,19 +1,5 @@
 <?xml version="1.0"?>
-<!-- xacro for the cage defining the workspace of the RePair platform -->
-<robot name = "repair_cage" xmlns:xacro="http://ros.org/wiki/xacro">
-  <xacro:include filename="$(find repair_urdf)/urdf/materials.gazebo.xacro"/>
-  <xacro:property name="table_height" value="0.5" />
-  <xacro:property name="cage_width" value="1.5" />
-  <xacro:property name="cage_height" value="1.0"/>
-  <xacro:property name="cage_depth" value="2.5" />
-  <xacro:property name="leg_radius" value="0.02" />
-  <xacro:property name="cage_depth" value="2.5" />
-  <xacro:property name="sliding_guide_width" value="0.2" />
-  <xacro:property name="table_x" value="0.98" />
-  <xacro:property name="table_y" value="0.0" />
-  <xacro:property name="table_z" value="0.0" />
-  <xacro:property name="table_top_thickness" value="0.05"/>
-  <xacro:property name="PI" value="3.14159265359" />
-  <xacro:property name="PI_2" value="1.57079632679" />
+<robot xmlns:xacro="http://ros.org/wiki/xacro">
+  <xacro:macro name="repair_cage" params="parent">
   <!-- only something to avoid collisions between leg and ground plane when using Gaz. -->
   <!-- <xacro:if value="$(arg shorten_table_legs_coll)">
@@ -23,35 +9,26 @@
   </xacro:unless> -->
   <xacro:property name="leg_z_offset_gz" value="0.0" />
-  <material name="wood">
-    <color rgba="0.522 0.369 0.259 0.8"/>
-  </material>
-  <material name="silver_gray">
-    <color rgba="0.8 0.8 0.8 0.8"/>
-  </material>
-  <link name="world">
-  </link>
-  <joint name="world_joint" type="fixed" >
-    <parent link="world" />
-    <origin xyz="0 0 0" rpy="0 0 0" />
+  <link name="table_top_link">
+    <visual>
+      <origin xyz="${Table_x} ${Table_y} ${Table_z+table_height-table_top_thickness/2}" />
+      <geometry>
+        <box size="${Cage_x} ${Cage_y} ${table_top_thickness}" />
+      </geometry>
+      <material name="wood" />
+    </visual>
+    <collision>
+      <origin xyz="${Table_x} ${Table_y} ${Table_z+table_height-table_top_thickness/2}" />
+      <geometry>
+        <box size="${Cage_x} ${Cage_y} ${table_top_thickness}" />
+      </geometry>
+    </collision>
+  </link>
+  <joint name="table_top_link_joint" type="fixed" >
+    <parent link="${parent}" />
     <child link="table_top_link" />
   </joint>
-  <link name="table_top_link">
-    <visual>
-      <origin xyz="${table_x} ${table_y} ${table_z+table_height-table_top_thickness/2}" />
-      <geometry>
-        <box size="${cage_width} ${cage_depth} ${table_top_thickness}" />
-      </geometry>
-      <material name="wood" />
-    </visual>
-    <collision>
-      <origin xyz="${table_x} ${table_y} ${table_z+table_height-table_top_thickness/2}" />
-      <geometry>
-        <box size="${cage_width} ${cage_depth} ${table_top_thickness}" />
-      </geometry>
-    </collision>
-  </link>
   <joint name="leg1_joint" type="fixed" >
     <parent link="table_top_link" />
-    <origin xyz="${table_x+cage_width/2} ${table_y+cage_depth/2} ${table_z+table_height}" rpy="0 0 0" />
+    <origin xyz="${Table_x+Cage_x/2} ${Table_y+Cage_y/2} ${Table_z+table_height}" rpy="0 0 0" />
     <child link="leg1_link" />
   </joint>
@@ -60,5 +37,5 @@
       <origin xyz="0.0 0.0 ${-table_height/2}" rpy="0 0 0" />
       <geometry>
-        <cylinder radius="${leg_radius}" length="${table_height}" />
+        <cylinder radius="${Cage_leg_radius}" length="${table_height}" />
       </geometry>
     <material name="silver_gray" />
@@ -67,5 +44,5 @@
       <origin xyz="0.0 0.0 ${-table_height/2 + leg_z_offset_gz}" rpy="0.0 0.0 0.0" />
       <geometry>
-        <cylinder radius="${leg_radius}" length="${table_height}" />
+        <cylinder radius="${Cage_leg_radius}" length="${table_height}" />
       </geometry>
     </collision>
@@ -73,5 +50,5 @@
   <joint name="vbar1_joint" type="fixed" >
     <parent link="leg1_link" />
-    <origin xyz="0 0 ${cage_height/2}" rpy="0 0 0" />
+    <origin xyz="0 0 ${Cage_z/2}" rpy="0 0 0" />
     <child link="vbar1_link" />
   </joint>
@@ -80,12 +57,12 @@
       <origin xyz="0.0 0.0 0" rpy="0 0 0" />
       <geometry>
-        <cylinder radius="${leg_radius}" length="${cage_height}" />
-      </geometry>
-    <material name="silver_gray" />
-    </visual>
-    <collision>
-      <origin xyz="0.0 0.0 0" rpy="0.0 0.0 0.0" />
-      <geometry>
-        <cylinder radius="${leg_radius}" length="${cage_height}" />
+        <cylinder radius="${Cage_leg_radius}" length="${Cage_z}" />
+      </geometry>
+    <material name="silver_gray" />
+    </visual>
+    <collision>
+      <origin xyz="0.0 0.0 0" rpy="0.0 0.0 0.0" />
+      <geometry>
+        <cylinder radius="${Cage_leg_radius}" length="${Cage_z}" />
       </geometry>
     </collision>
@@ -93,5 +70,5 @@
   <joint name="leg2_joint" type="fixed" >
     <parent link="table_top_link" />
-    <origin xyz="${table_x-cage_width/2} ${table_y+cage_depth/2} ${table_z+table_height}" rpy="0 0 0" />
+    <origin xyz="${Table_x-Cage_x/2} ${Table_y+Cage_y/2} ${Table_z+table_height}" rpy="0 0 0" />
     <child link="leg2_link" />
   </joint>
@@ -100,5 +77,5 @@
       <origin xyz="0.0 0.0 ${-table_height/2}" rpy="0 0 0" />
       <geometry>
-        <cylinder radius="${leg_radius}" length="${table_height}" />
+        <cylinder radius="${Cage_leg_radius}" length="${table_height}" />
       </geometry>
       <material name="silver_gray" />
@@ -107,5 +84,5 @@
       <origin xyz="0.0 0.0 ${-table_height/2 + leg_z_offset_gz}" rpy="0.0 0.0 0.0" />
       <geometry>
-        <cylinder radius="${leg_radius}" length="${table_height}" />
+        <cylinder radius="${Cage_leg_radius}" length="${table_height}" />
       </geometry>
     </collision>
@@ -113,5 +90,5 @@
   <joint name="vbar2_joint" type="fixed" >
     <parent link="leg2_link" />
-    <origin xyz="0 0 ${cage_height/2}" rpy="0 0 0" />
+    <origin xyz="0 0 ${Cage_z/2}" rpy="0 0 0" />
     <child link="vbar2_link" />
   </joint>
@@ -120,12 +97,12 @@
       <origin xyz="0.0 0.0 0" rpy="0 0 0" />
       <geometry>
-        <cylinder radius="${leg_radius}" length="${cage_height}" />
-      </geometry>
-    <material name="silver_gray" />
-    </visual>
-    <collision>
-      <origin xyz="0.0 0.0 0" rpy="0.0 0.0 0.0" />
-      <geometry>
-        <cylinder radius="${leg_radius}" length="${cage_height}" />
+        <cylinder radius="${Cage_leg_radius}" length="${Cage_z}" />
+      </geometry>
+    <material name="silver_gray" />
+    </visual>
+    <collision>
+      <origin xyz="0.0 0.0 0" rpy="0.0 0.0 0.0" />
+      <geometry>
+        <cylinder radius="${Cage_leg_radius}" length="${Cage_z}" />
       </geometry>
     </collision>
@@ -133,5 +110,5 @@
   <joint name="leg3_joint" type="fixed" >
     <parent link="table_top_link" />
-    <origin xyz="${table_x+cage_width/2} ${table_y-cage_depth/2} ${table_z+table_height}" rpy="0 0 0" />
+    <origin xyz="${Table_x+Cage_x/2} ${Table_y-Cage_y/2} ${Table_z+table_height}" rpy="0 0 0" />
     <child link="leg3_link" />
   </joint>
@@ -140,5 +117,5 @@
       <origin xyz="0.0 0.0 ${-table_height/2}" rpy="0 0 0" />
       <geometry>
-        <cylinder radius="${leg_radius}" length="${table_height}" />
+        <cylinder radius="${Cage_leg_radius}" length="${table_height}" />
       </geometry>
       <material name="silver_gray" />
@@ -147,5 +124,5 @@
       <origin xyz="0.0 0.0 ${-table_height/2 + leg_z_offset_gz}" rpy="0.0 0.0 0.0" />
       <geometry>
-        <cylinder radius="${leg_radius}" length="${table_height}" />
+        <cylinder radius="${Cage_leg_radius}" length="${table_height}" />
       </geometry>
     </collision>
@@ -153,5 +130,5 @@
   <joint name="vbar3_joint" type="fixed" >
     <parent link="leg3_link" />
-    <origin xyz="0 0 ${cage_height/2}" rpy="0 0 0" />
+    <origin xyz="0 0 ${Cage_z/2}" rpy="0 0 0" />
     <child link="vbar3_link" />
   </joint>
@@ -160,12 +137,12 @@
       <origin xyz="0.0 0.0 0" rpy="0 0 0" />
       <geometry>
-        <cylinder radius="${leg_radius}" length="${cage_height}" />
-      </geometry>
-    <material name="silver_gray" />
-    </visual>
-    <collision>
-      <origin xyz="0.0 0.0 0" rpy="0.0 0.0 0.0" />
-      <geometry>
-        <cylinder radius="${leg_radius}" length="${cage_height}" />
+        <cylinder radius="${Cage_leg_radius}" length="${Cage_z}" />
+      </geometry>
+    <material name="silver_gray" />
+    </visual>
+    <collision>
+      <origin xyz="0.0 0.0 0" rpy="0.0 0.0 0.0" />
+      <geometry>
+        <cylinder radius="${Cage_leg_radius}" length="${Cage_z}" />
       </geometry>
     </collision>
@@ -173,5 +150,5 @@
   <joint name="leg4_joint" type="fixed" >
     <parent link="table_top_link" />
-    <origin xyz="${table_x-cage_width/2} ${table_y-cage_depth/2} ${table_z+table_height}" rpy="0 0 0" />
+    <origin xyz="${Table_x-Cage_x/2} ${Table_y-Cage_y/2} ${Table_z+table_height}" rpy="0 0 0" />
     <child link="leg4_link" />
   </joint>
@@ -180,5 +157,5 @@
       <origin xyz="0.0 0.0 ${-table_height/2}" rpy="0 0 0" />
       <geometry>
-        <cylinder radius="${leg_radius}" length="${table_height}" />
+        <cylinder radius="${Cage_leg_radius}" length="${table_height}" />
       </geometry>
       <material name="silver_gray" />
@@ -187,5 +164,5 @@
       <origin xyz="0.0 0.0 ${-table_height/2 + leg_z_offset_gz}" rpy="0.0 0.0 0.0" />
       <geometry>
-        <cylinder radius="${leg_radius}" length="${table_height}" />
+        <cylinder radius="${Cage_leg_radius}" length="${table_height}" />
       </geometry>
     </collision>
@@ -193,5 +170,5 @@
   <joint name="vbar4_joint" type="fixed" >
     <parent link="leg4_link" />
-    <origin xyz="0 0 ${cage_height/2}" rpy="0 0 0" />
+    <origin xyz="0 0 ${Cage_z/2}" rpy="0 0 0" />
     <child link="vbar4_link" />
   </joint>
@@ -200,12 +177,12 @@
       <origin xyz="0.0 0.0 0" rpy="0 0 0" />
       <geometry>
-        <cylinder radius="${leg_radius}" length="${cage_height}" />
-      </geometry>
-    <material name="silver_gray" />
-    </visual>
-    <collision>
-      <origin xyz="0.0 0.0 0" rpy="0.0 0.0 0.0" />
-      <geometry>
-        <cylinder radius="${leg_radius}" length="${cage_height}" />
+        <cylinder radius="${Cage_leg_radius}" length="${Cage_z}" />
+      </geometry>
+    <material name="silver_gray" />
+    </visual>
+    <collision>
+      <origin xyz="0.0 0.0 0" rpy="0.0 0.0 0.0" />
+      <geometry>
+        <cylinder radius="${Cage_leg_radius}" length="${Cage_z}" />
       </geometry>
     </collision>
@@ -213,5 +190,5 @@
   <joint name="obar1_joint" type="fixed" >
     <parent link="vbar1_link" />
-    <origin xyz="-${cage_width/2} 0 ${cage_height/2}" rpy="0 -${PI_2} 0" />
+    <origin xyz="-${Cage_x/2} 0 ${Cage_z/2}" rpy="0 -${PI_2} 0" />
     <child link="obar1_link" />
   </joint>
@@ -220,12 +197,12 @@
       <origin xyz="0.0 0.0 0" rpy="0 0 0" />
       <geometry>
-        <cylinder radius="${leg_radius}" length="${cage_width}" />
-      </geometry>
-    <material name="silver_gray" />
-    </visual>
-    <collision>
-      <origin xyz="0.0 0.0 0" rpy="0.0 0.0 0.0" />
-      <geometry>
-        <cylinder radius="${leg_radius}" length="${cage_width}" />
+        <cylinder radius="${Cage_leg_radius}" length="${Cage_x}" />
+      </geometry>
+    <material name="silver_gray" />
+    </visual>
+    <collision>
+      <origin xyz="0.0 0.0 0" rpy="0.0 0.0 0.0" />
+      <geometry>
+        <cylinder radius="${Cage_leg_radius}" length="${Cage_x}" />
       </geometry>
     </collision>
@@ -233,5 +210,5 @@
   <joint name="obar2_joint" type="fixed" >
     <parent link="vbar3_link" />
-    <origin xyz="-${cage_width/2} 0 ${cage_height/2}" rpy="0 -${PI_2} 0" />
+    <origin xyz="-${Cage_x/2} 0 ${Cage_z/2}" rpy="0 -${PI_2} 0" />
     <child link="obar2_link" />
   </joint>
@@ -240,12 +217,12 @@
       <origin xyz="0.0 0.0 0" rpy="0 0 0" />
       <geometry>
-        <cylinder radius="${leg_radius}" length="${cage_width}" />
-      </geometry>
-    <material name="silver_gray" />
-    </visual>
-    <collision>
-      <origin xyz="0.0 0.0 0" rpy="0.0 0.0 0.0" />
-      <geometry>
-        <cylinder radius="${leg_radius}" length="${cage_width}" />
+        <cylinder radius="${Cage_leg_radius}" length="${Cage_x}" />
+      </geometry>
+    <material name="silver_gray" />
+    </visual>
+    <collision>
+      <origin xyz="0.0 0.0 0" rpy="0.0 0.0 0.0" />
+      <geometry>
+        <cylinder radius="${Cage_leg_radius}" length="${Cage_x}" />
       </geometry>
     </collision>
@@ -253,5 +230,5 @@
   <joint name="obar3_joint" type="fixed" >
     <parent link="vbar3_link" />
-    <origin xyz="0 ${cage_depth/2} ${cage_height/2}" rpy="-${PI_2} 0 0" />
+    <origin xyz="0 ${Cage_y/2} ${Cage_z/2}" rpy="-${PI_2} 0 0" />
     <child link="obar3_link" />
   </joint>
@@ -260,12 +237,12 @@
       <origin xyz="0.0 0.0 0" rpy="0 0 0" />
       <geometry>
-        <cylinder radius="${leg_radius}" length="${cage_depth}" />
-      </geometry>
-    <material name="silver_gray" />
-    </visual>
-    <collision>
-      <origin xyz="0.0 0.0 0" rpy="0.0 0.0 0.0" />
-      <geometry>
-        <cylinder radius="${leg_radius}" length="${cage_depth}" />
+        <cylinder radius="${Cage_leg_radius}" length="${Cage_y}" />
+      </geometry>
+    <material name="silver_gray" />
+    </visual>
+    <collision>
+      <origin xyz="0.0 0.0 0" rpy="0.0 0.0 0.0" />
+      <geometry>
+        <cylinder radius="${Cage_leg_radius}" length="${Cage_y}" />
       </geometry>
     </collision>
@@ -273,5 +250,5 @@
   <joint name="obar4_joint" type="fixed" >
     <parent link="vbar4_link" />
-    <origin xyz="0 ${cage_depth/2} ${cage_height/2}" rpy="-${PI_2} 0 0" />
+    <origin xyz="0 ${Cage_y/2} ${Cage_z/2}" rpy="-${PI_2} 0 0" />
     <child link="obar4_link" />
   </joint>
@@ -281,12 +258,12 @@
       <origin xyz="0.0 0.0 0" rpy="0 0 0" />
       <geometry>
-        <cylinder radius="${leg_radius}" length="${cage_depth}" />
-      </geometry>
-    <material name="silver_gray" />
-    </visual>
-    <collision>
-      <origin xyz="0.0 0.0 0" rpy="0.0 0.0 0.0" />
-      <geometry>
-        <cylinder radius="${leg_radius}" length="${cage_depth}" />
+        <cylinder radius="${Cage_leg_radius}" length="${Cage_y}" />
+      </geometry>
+    <material name="silver_gray" />
+    </visual>
+    <collision>
+      <origin xyz="0.0 0.0 0" rpy="0.0 0.0 0.0" />
+      <geometry>
+        <cylinder radius="${Cage_leg_radius}" length="${Cage_y}" />
       </geometry>
     </collision>
@@ -294,5 +271,5 @@
   <joint name="sliding_guide_joint" type="fixed" >
     <parent link="obar2_link" />
-    <origin xyz="0 ${cage_depth/2} 0" rpy="-${PI_2} 0 0" />
+    <origin xyz="0 ${Cage_y/2} 0" rpy="-${PI_2} 0 0" />
     <child link="sliding_guide_link" />
   </joint>
@@ -301,12 +278,12 @@
       <origin xyz="0.0 0.0 0" rpy="0 0 0" />
       <geometry>
-        <box size="0.001 ${sliding_guide_width} ${cage_depth}" />
-      </geometry>
-    <material name="silver_gray" />
-    </visual>
-    <collision>
-      <origin xyz="0.0 0.0 0" rpy="0.0 0.0 0.0" />
-      <geometry>
-        <cylinder radius="${leg_radius}" length="${cage_depth}" />
+        <box size="0.001 ${sliding_guide_width} ${Cage_y}" />
+      </geometry>
+    <material name="silver_gray" />
+    </visual>
+    <collision>
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