Commit message: added full system in urdf

File: repair_urdf/urdf/repair_full.urdf.xacro (robot description, xacro)
@@ -1,167 +1,26 @@
 <?xml version="1.0"?>
-<!-- xacro for generating the full urdf of the RePair platform (cage + bimanual robot) -->
-<!-- is_sliding_wrist: whether to add a sliding joint along the wrist second d.o.f.
-    (true -> yes), everything else -> no. This is used to generate the URDF for the optimization.  -->
-<!-- gen_coll: whether to add the approximate collision  model of the platform -->
-<!-- load_sol: whether to generate the URDF without the additional d.o.f. used by the co-design optimization.
-Setting it to "true", allow to fix the additional d.o.f. to desired values
-(specified in the repair_urdf/config/arm_opt_mount_vals.yaml file) -->
-<!-- use_updated_wrist: visual parameter. if true, we load the latest meshes (which are adapted to the
-results of the optimization), otherwise we go with the old ones (generated for a spherical wrist) -->
-<!-- xbot: if true, we add the gazebo tags necessary to use the URDF with XBot2 framework -->
-<robot name = "repair_full" xmlns:xacro="http://ros.org/wiki/xacro">
-<xacro:arg name="is_sliding_wrist" default="false" />
-<xacro:arg name="gen_coll" default="false" />
-<xacro:arg name="load_sol" default="false" />
-<xacro:arg name="use_updated_wrist" default="false" />
-<xacro:arg name="xbot" default="false" />
-<xacro:include filename="$(find repair_urdf)/urdf/repair_arm.urdf.xacro"/>
-<xacro:include filename="$(find repair_urdf)/urdf/repair_cage.urdf.xacro"/>
-<xacro:include filename="$(find repair_urdf)/urdf/repair_opt_mount_params.urdf.xacro"/>
-<xacro:include filename="$(find repair_urdf)/urdf/materials.gazebo.xacro"/>
-<xacro:if value="$(arg xbot)">
-    <xacro:include filename="$(find repair_urdf)/urdf/xbot2.gazebo.xacro"/>
-</xacro:if>
-<!-- <xacro:if value="$(arg gen_coll)">
-    <xacro:include filename="$(find repair_urdf)/urdf/repair_torso_coll_params.urdf.xacro"/>
-    <xacro:include filename="$(find repair_urdf)/urdf/repair_torso_coll.urdf.xacro"/>
-    <xacro:repair_torso_coll />
-</xacro:if> -->
-<xacro:if value="$(arg load_sol)">
-    <joint name="x_joint" type="prismatic">
-        <origin xyz="0.0 0.0 ${mount_h}" rpy="0.0 0.0 0.0"/>
-        <parent link="working_surface_link"/>
-        <child link="base_link"/>
-        <axis xyz="1 0 0"/>
-        <limit lower="${- cage_depth/2 + x_joint_limit_margin}" upper= "${cage_depth/2 - x_joint_limit_margin}" effort="1000.0" velocity="20.0"/>
-    </joint>
-    <link name="base_link">
-        <!-- torso inertias + stuff attached to the sliding guide -->
-        <inertial>
-          <mass value="${full_torso_mass}" />
-          <origin xyz="0 0 0" />
-          <inertia ixx="0" ixy="0"  ixz="0"
-                  iyy="0" iyz="0"
-                  izz="0" />
-        </inertial>
-        <xacro:if value="$(arg use_updated_wrist)">
-            <visual name="base_link_visual">
-                <geometry>
-                    <mesh filename="package://repair_urdf/meshes/optimized/link_0.stl" scale="${mmTom} ${mmTom} ${mmTom}"/>
-                </geometry>
-                <material name="dark"/>
-            </visual>
-        </xacro:if>
-    </link>
-    <joint name="r_arm_mount_joint" type="fixed">
-        <origin xyz="0.0 ${-should_w} 0.0" rpy="0 0 0"/>
-        <parent link="base_link"/>
-        <child link="dummy_r"/>
-    </joint>
-    <joint name="l_arm_mount_joint" type="fixed">
-        <origin xyz="0.0 ${should_w} 0.0" rpy="0 0 0"/>
-        <parent link="base_link"/>
-        <child link="dummy_l"/>
-    </joint>
-    <link name="dummy_r">
-    </link>
-    <link name="dummy_l">
-    </link>
-    <joint name="roll_r" type="fixed">
-        <origin xyz="0 0.0 0.0" rpy="${roll_mount} 0.0 0.0"/>
-        <parent link="dummy_r"/>
-        <child link="r_arm_mount_frame"/>
-    </joint>
-    <joint name="roll_l" type="fixed">
-        <origin xyz="0 0.0 0.0" rpy="${-roll_mount} 0.0 0.0"/>
-        <parent link="dummy_l"/>
-        <child link="l_arm_mount_frame"/>
-    </joint>
-    <link name="r_arm_mount_frame">
-        <xacro:aux_inertia cutoff_inertia="${gazebo_cutoff_inertia}"/>
-    </link>
-    <link name="l_arm_mount_frame">
-        <xacro:aux_inertia cutoff_inertia="${gazebo_cutoff_inertia}"/>
-    </link>
-</xacro:if>
-<xacro:unless value="$(arg load_sol)">
-    <joint name="x_joint" type="prismatic">
-        <origin xyz="0.0 0.0 0.0" rpy="0.0 0.0 0.0"/>
-        <parent link="working_surface_link"/>
-        <child link="dummy_link"/>
-        <axis xyz="1 0 0"/>
-        <limit lower="${- cage_depth/2 + x_joint_limit_margin}" upper= "${cage_depth/2 - x_joint_limit_margin}" effort="1000.0" velocity="20.0"/>
-    </joint>
-    <link name="dummy_link">
-    </link>
-    <joint name="z_joint" type="prismatic">
-        <origin xyz="0.0 0.0 0.0" rpy="0.0 0.0 0.0"/>
-        <parent link="dummy_link"/>
-        <child link="base_link"/>
-        <axis xyz="0 0 1"/>
-        <limit lower="${z_joint_lb}" upper= "2" effort="1000.0" velocity="20.0"/>
-    </joint>
-    <!-- RePAIR assembly (two arms) -->
-    <link name="base_link">
-        <!-- torso inertias + stuff attached to the sliding guide -->
-        <inertial>
-            <mass value="${full_torso_mass}" />
-            <origin xyz="0 0 0" />
-            <inertia ixx="0" ixy="0"  ixz="0"
-                    iyy="0" iyz="0"
-                    izz="0" />
-          </inertial>
-        <xacro:if value="$(arg use_updated_wrist)">
-            <visual name="base_link_visual">
-                <geometry>
-                    <mesh filename="package://repair_urdf/meshes/optimized/link_0.stl" scale="${mmTom} ${mmTom} ${mmTom}"/>
-                </geometry>
-                <material name="dark"/>
-            </visual>
-        </xacro:if>
-    </link>
-    <link name="dummy_r">
-    </link>
-    <link name="dummy_l">
-    </link>
-    <joint name="r_arm_mount_joint" type="prismatic">
-        <origin xyz="0.0 0.0 0.0" rpy="0 0 0"/>
-        <parent link="base_link"/>
-        <child link="dummy_r"/>
-        <axis xyz="0 -1 0"/>
-        <limit lower="${shoulder_width_lb}" upper= "${shoulder_width_ub}" effort="1000.0" velocity="20.0"/>
-    </joint>
-    <joint name="l_arm_mount_joint" type="prismatic">
-        <origin xyz="0.0 0.0 0.0" rpy="0 0 0"/>
-        <parent link="base_link"/>
-        <child link="dummy_l"/>
-        <axis xyz="0 1 0"/>
-        <limit lower="${shoulder_width_lb}" upper= "${shoulder_width_ub}" effort="1000.0" velocity="20.0"/>
-    </joint>
-    <joint name="roll_r" type="revolute">
-        <origin xyz="0.0 0.0 0.0" rpy="0.0 0.0 0.0"/>
-        <parent link="dummy_r"/>
-        <child link="r_arm_mount_frame"/>
-        <axis xyz="1 0 0"/>
-        <limit lower="${shoulder_roll_lb}" upper="${shoulder_roll_ub}" effort="0.0" velocity="0.0"/>
-    </joint>
-    <joint name="roll_l" type="revolute">
-        <origin xyz="0.0 0.0 0.0" rpy="0.0 0.0 0.0"/>
-        <parent link="dummy_l"/>
-        <child link="l_arm_mount_frame"/>
-        <axis xyz="-1 0 0"/>
-        <limit lower="${shoulder_roll_lb}" upper="${shoulder_roll_ub}" effort="0.0" velocity="0.0"/>
-    </joint>
-    <link name="r_arm_mount_frame">
-    </link>
-    <link name="l_arm_mount_frame">
-    </link>
-</xacro:unless>
-<xacro:repair_arm base_link="r_arm_mount_frame" id="1" is_sliding_wrist="$(arg is_sliding_wrist)"
-gen_coll="$(arg gen_coll)" load_sol="$(arg load_sol)" use_updated_wrist = "$(arg use_updated_wrist)"/>
-<xacro:repair_arm base_link="l_arm_mount_frame" id="2" is_sliding_wrist="$(arg is_sliding_wrist)"
-gen_coll="$(arg gen_coll)" load_sol="$(arg load_sol)" use_updated_wrist = "$(arg use_updated_wrist)"/>
-<xacro:repair_arm_materials id="1" />
-<xacro:repair_arm_materials id="2" />
-<xacro:repair_torso_materials />
+<robot xmlns:xacro="http://ros.org/wiki/xacro" name="repair_full">
+    <xacro:include filename="$(find repair_urdf)/urdf/conversions.urdf.xacro" />
+    <xacro:include filename="$(find repair_urdf)/urdf/materials.urdf.xacro" />
+    <xacro:include filename="$(find repair_urdf)/urdf/repair_arm_macro.urdf.xacro" />
+    <xacro:include filename="$(find repair_urdf)/urdf/repair_torso_macro.urdf.xacro"/>
+    <xacro:include filename="$(find repair_urdf)/urdf/repair_cage_macro.urdf.xacro"/>
+    <xacro:include filename="$(find repair_urdf)/urdf/kinematics_properties.urdf.xacro" />
+    <xacro:include filename="$(find repair_urdf)/urdf/inertial_properties.urdf.xacro" />
+    <xacro:include filename="$(find repair_urdf)/urdf/limits.urdf.xacro" />
+    <xacro:include filename="$(find repair_urdf)/urdf/gazebo/xbot.gazebo.xacro" />
+    <link name="world"/>
+    <xacro:repair_cage parent="world">
+    </xacro:repair_cage>
+    <xacro:repair_torso parent="sliding_guide_link">
+        <origin xyz="0.0 0.0 0.0" rpy="0.0 0.0 0.0" />
+    </xacro:repair_torso>
+    <xacro:repair_arm id="1"  rot="1"  parent="torso_1">
+      <origin xyz="${Shoulder_1_Ox} ${Shoulder_1_Oy} ${Shoulder_1_Oz}"
+              rpy="${Shoulder_1_roll} ${Shoulder_1_pitch} ${Shoulder_1_yaw}" />
+    </xacro:repair_arm>
+    <xacro:repair_arm id="2"  rot="-1"  parent="torso_1">
+        <origin xyz="${Shoulder_1_Ox} ${-Shoulder_1_Oy} ${Shoulder_1_Oz}"
+                rpy="${-Shoulder_1_roll} ${Shoulder_1_pitch} ${Shoulder_1_yaw}" />
+      </xacro:repair_arm>
 </robot>

Commit message: updated model for gazebo

File: repair_urdf/urdf/gazebo/xbot.gazebo.xacro (robot description, xacro)
@@ -7,5 +7,6 @@
             <gain name="small_mot"  p="1000"  d="10"/>
             <gain name="medium_mot" p="2000" d="20"/>
-            <!-- <pid name="j_arm_1_1" profile="medium_mot"/>
+            <pid name="j_torso_1" profile="medium_mot"/>
+            <pid name="j_arm_1_1" profile="medium_mot"/>
             <pid name="j_arm_1_2" profile="medium_mot"/>
             <pid name="j_arm_1_3" profile="medium_mot"/>
@@ -13,5 +14,5 @@
             <pid name="j_arm_1_5" profile="small_mot"/>
             <pid name="j_arm_1_6" profile="small_mot"/>
-            <pid name="j_arm_1_7" profile="small_mot"/> -->
+            <pid name="j_arm_1_7" profile="small_mot"/>
             <pid name="j_arm_2_1" profile="medium_mot"/>
             <pid name="j_arm_2_2" profile="medium_mot"/>

File: repair_urdf/urdf/repair_full.urdf.xacro (robot description, xacro)
@@ -14,5 +14,6 @@
     </xacro:repair_cage>
     <xacro:repair_torso parent="sliding_guide_link">
-        <origin xyz="0.0 0.0 0.0" rpy="0.0 0.0 0.0" />
+    <origin xyz="${Torso_Ox} ${Torso_Oy} ${Torso_Oz}"
+            rpy="${Torso_roll} ${Torso_pitch} ${Torso_yaw}" />
     </xacro:repair_torso>
     <xacro:repair_arm id="2"  rot="1"  parent="torso_1">

File: repair_urdf/urdf/repair_torso_macro.urdf.xacro (robot description, xacro)
@@ -2,5 +2,5 @@
 <robot xmlns:xacro="http://ros.org/wiki/xacro">
     <xacro:macro name="repair_torso" params="parent *origin">
-        <link name="dummy_prismatic_link"/>
+        <!-- <link name="dummy_prismatic_link"/> -->
         <link name="torso_1">
             <inertial>
@@ -22,5 +22,5 @@
             </collision>
         </link>
-        <joint name="j_torso_base" type="prismatic">
+        <!-- <joint name="j_torso_base" type="fixed">
             <xacro:insert_block name="origin" />
             <parent link="${parent}" />
@@ -28,12 +28,11 @@
             <axis xyz="0 0 1"/>
             <limit lower="${j_prismatic_lower[0]/2}" upper= "${j_prismatic_upper[0]/2}" effort="${j_prismatic_torque[0]}" velocity="${j_prismatic_velocity[0]}"/>
-        </joint>
+        </joint> -->
         <!-- torso -->
         <joint name="j_torso_1" type="revolute">
-            <parent link="dummy_prismatic_link" />
+            <parent link="${parent}" />
             <child link="torso_1" />
             <axis xyz="0 0 1" />
-            <origin xyz="${Torso_Ox} ${Torso_Oy} ${Torso_Oz}"
-            rpy="${Torso_roll} ${Torso_pitch} ${Torso_yaw}" />
+            <xacro:insert_block name="origin" />
             <limit lower="${j_torso_lower[0]}" upper="${j_torso_upper[0]}"
             effort="${j_torso_torque[0]}" velocity="${j_torso_velocity[0]}" />

Commit message: added to urdf and simulation softhands

File: repair_urdf/urdf/gazebo/xbot.gazebo.xacro (robot description, xacro)
@@ -2,4 +2,5 @@
 <robot xmlns:xacro="http://ros.org/wiki/xacro">
 <gazebo>
+    <xacro:include filename="$(find repair_urdf)/urdf/gazebo/ignore_joint_softhand.xbot.xacro" />
     <plugin name="xbot2_joint_driver" filename="libxbot2_gz_joint_server.so">
         <pid>
@@ -23,4 +24,8 @@
             <pid name="j_arm_2_7" profile="small_mot"/>
         </pid>
+        <ignore_joints>
+            <xacro:ignore_softhand_jnts side="right" type="v1s"/>
+            <xacro:ignore_softhand_jnts side="left" type="v1s"/>
+        </ignore_joints>
     </plugin>
 </gazebo>

File: repair_urdf/urdf/repair_cage_macro.urdf.xacro (robot description, xacro)
@@ -10,10 +10,10 @@
       <material name="wood" />
     </visual>
-    <collision>
+    <!-- <collision>
       <origin xyz="${Table_x} ${Table_y} ${Table_z+table_height-table_top_thickness/2}" />
       <geometry>
         <box size="${Cage_x} ${Cage_y} ${table_top_thickness}" />
       </geometry>
-    </collision>
+    </collision> -->
   </link>
   <joint name="table_top_link_joint" type="fixed" >

File: repair_urdf/urdf/repair_full.urdf.xacro (robot description, xacro)
@@ -1,4 +1,5 @@
 <?xml version="1.0"?>
 <robot xmlns:xacro="http://ros.org/wiki/xacro" name="repair_full">
+    <xacro:include filename="$(find softhands_description)/urdf/softhands.xacro" />
     <xacro:include filename="$(find repair_urdf)/urdf/conversions.urdf.xacro" />
     <xacro:include filename="$(find repair_urdf)/urdf/materials.urdf.xacro" />
@@ -25,3 +26,24 @@
                 rpy="${-Shoulder_1_roll} ${Shoulder_1_pitch} ${Shoulder_1_yaw}" />
       </xacro:repair_arm>
+    <xacro:softhands type="left"
+        version="v1.0_simple"
+        parent="arm_1_7"
+        position="0 0 -0.015"
+        orientation="0 0.0 ${PI}"
+        translation="0"
+        operation_mode="0"
+        fixed_hands="false">
+    </xacro:softhands>
+    <xacro:softhands type="right"
+        version="v1.0_simple"
+        parent="arm_2_7"
+        position="0 -0.013900 -0.015"
+        orientation="0 0 ${PI}"
+        translation="0"
+        operation_mode="0"
+        fixed_hands="false">
+    </xacro:softhands>
+    <!-- <gazebo reference="table_top_link">
+        <selfCollide> 1 </selfCollide>
+    </gazebo> -->
 </robot>
